Commit message: Updated erratic model

File: wubble/wubble_robots/defs/erratic/erratic.urdf.xacro (robot description, xacro)
@@ -8,5 +8,5 @@
     <include filename="$(find pr2_defs)/calibration/default_cal.xml" />
 <!--    <include filename="$(find pr2_defs)/defs/head/head_defs.urdf.xacro" />-->
-    <include filename="$(find pr2_defs)/defs/head/head_sensor_package_defs.urdf.xacro" />
+    <include filename="$(find wubble_robots)/defs/erratic/head_sensor_package_defs.urdf.xacro" />
     <include filename="$(find pr2_defs)/defs/materials.urdf.xacro" />
     <include filename="$(find wubble_robots)/defs/erratic/erratic_head.xacro" />
@@ -15,5 +15,5 @@
     <property name="base_size_x" value="0.395224" />
     <property name="base_size_y" value="0.367284" />
-    <property name="base_size_z" value="0.155448" />
+    <property name="base_size_z" value="0.135448" />
     <property name="wheel_radius" value="0.0625" />
     <property name="wheel_length" value="0.02" />
@@ -23,5 +23,5 @@
         <inertial>
             <mass value="10" />
-            <origin xyz="-0.1 0 ${base_size_z/2}" />
+            <origin xyz="-0.05 0 ${base_size_z/2}" />
             <inertia ixx="1.0" ixy="0.0" ixz="0.0"
                 iyy="1.0" iyz="0.0"
@@ -212,11 +212,11 @@
   </gazebo>
     <property name="support_radius" value="0.01" />
-    <property name="support_height" value="0.3" />
-    <joint name="laser_support_joint" type="fixed">
-        <origin xyz="0 0 ${(support_height/2)+base_size_z}" />
+    <property name="support_height" value="0.8128" />
+    <joint name="head_support_joint" type="fixed">
+        <origin xyz="-0.0254 0 ${(support_height/2)+base_size_z}" />
         <parent link="base_top_link" />
-        <child link="laser_support_link" />
+        <child link="head_support_link" />
     </joint>
-    <link name="laser_support_link">
+    <link name="head_support_link">
         <inertial>
             <mass value="0.1"/>
@@ -225,5 +225,5 @@
         </inertial>
         <visual>
-            <origin rpy="0 0 ${support_height/2}" xyz="0 0 0.0"/>
+            <origin rpy="0 0 0" xyz="0 0 0"/>
             <geometry>
                 <cylinder radius="${support_radius}" length="${support_height}"/>
@@ -231,5 +231,5 @@
         </visual>
         <collision>
-            <origin rpy="0 0 ${support_height/2}" xyz="0 0 0.0"/>
+            <origin rpy="0 0 0" xyz="0 0 0"/>
             <geometry>
                 <cylinder radius="${support_radius}" length="${support_height}"/>
@@ -237,56 +237,38 @@
         </collision>
     </link>
-<!--  <joint name="base_laser_joint" type="fixed">-->
-<!--    <origin xyz="0.0 0 ${support_height/2}" rpy="0 0 0" />-->
-<!--    <parent link="laser_support_link"/>-->
-<!--    <child link="base_laser_link"/>-->
-<!--  </joint>-->
-<!--  <link name="base_laser_link" type="laser">-->
-<!--    <inertial>-->
-<!--      <mass value="0.1"/>-->
-<!--      <origin xyz="0 0 0.0"/>-->
-<!--      <inertia ixx="0.1" ixy="0" ixz="0" iyy="0.1" iyz="0" izz="0.1"/>-->
-<!--    </inertial>-->
-<!--    -->
-<!--    <visual>-->
-<!--      <origin rpy="0 0 0" xyz="0 0 0.0"/>-->
-<!--      <geometry>-->
-<!--        <cylinder radius=".05" length=".05"/>-->
-<!--      </geometry>-->
-<!--    </visual>-->
-<!--    -->
-<!--    <collision>-->
-<!--      <origin rpy="0 0 0" xyz="0 0 0.0"/>-->
-<!--      <geometry>-->
-<!--        <cylinder radius=".05" length=".05"/>-->
-<!--      </geometry>-->
-<!--    </collision>-->
-<!--    -->
-<!--  </link>-->
-<!--  <gazebo reference="base_laser_link">-->
-<!--    <sensor:ray name="base_laser_link">-->
-<!--      <resRange>0.1</resRange>-->
-<!--      <rayCount>640</rayCount>-->
-<!--      <rangeCount>640</rangeCount>-->
-<!--      <laserCount>1</laserCount>-->
-<!--      <origin>0.0 0.0 0.0</origin>-->
-<!--      <displayRays>false</displayRays>-->
-<!--      -->
-<!--      <minAngle>-100</minAngle> -->
-<!--      <maxAngle>100</maxAngle>-->
-<!--      -->
-<!--      <minRange>0.07</minRange>-->
-<!--      <maxRange>10.0</maxRange>-->
-<!--      <updateRate>20.0</updateRate>-->
-<!--      <controller:gazebo_ros_laser name="gazebo_ros_base_laser_link_controller" plugin="libgazebo_ros_laser.so">-->
-<!--        <gaussianNoise>0.005</gaussianNoise>-->
-<!--        <alwaysOn>true</alwaysOn>-->
-<!--        <updateRate>20.0</updateRate>-->
-<!--        <topicName>base_scan</topicName>-->
-<!--        <frameName>base_laser_link</frameName>-->
-<!--        <interface:laser name="gazebo_ros_base_laser_link_iface"/>-->
-<!--      </controller:gazebo_ros_laser>-->
-<!--    </sensor:ray>-->
-<!--  </gazebo>-->
+    <joint name="head_tilt_joint" type="fixed"><!--type="continuous">-->
+        <origin xyz="0 0 ${support_height/2}" />
+        <axis xyz="0 0 1" />
+<!--        <anchor xyz="0 0 0" />
+        <limit effort="100" velocity="100" />
+        <joint_properties damping="0.0" friction="0.0" /> -->
+        <parent link="head_support_link" />
+        <child link="head_tilt_link" />
+    </joint>
+    <link name="head_tilt_link">
+        <inertial>
+            <mass value="0.01"/>
+            <origin xyz="0 0 0.0"/>
+            <inertia ixx="0.01" ixy="0" ixz="0" iyy="0.01" iyz="0" izz="0.01"/>
+        </inertial>
+        <visual>
+            <origin xyz="0 0 0.0127" rpy="0 0 0"/>
+            <geometry>
+                <box size="${2*support_radius} ${2*support_radius} 0.0254" />
+            </geometry>
+        </visual>
+        <collision>
+            <origin xyz="0 0 0.0127" rpy="0 0 0"/>
+            <geometry>
+                <box size="${2*support_radius} ${2*support_radius} 0.0254" />
+            </geometry>
+        </collision>
+    </link>
+<!--    <joint name="head_pitch_joint" type="fixed">
+       <origin xyz="0 0 ${support_height+base_size_z}" />
+        <parent link="head_support_link" />
+        <child link="stoc_camera_link" />
+    </joint>
+-->
   <gazebo>
     <controller:differential_position2d name="controller1">
@@ -332,7 +314,7 @@
     <!-- attempt to add the pan-tilt laser from the pr2, it should be close enough -->
     <pr2_tilting_laser name="laser_tilt" parent="base_top_link" laser_calib_ref="-0.35">
-        <origin xyz="0.1 0 0.235" rpy="0 0 0" />
+        <origin xyz="0.1 0 ${base_size_z - 0.05}" rpy="0 -1 0" />
     </pr2_tilting_laser>
-    <stoc_camera name="stoc" parent="base_top_link" />
+    <stoc_camera name="stoc" parent="head_tilt_link" />
     <!-- Gazebo materials -->
     <gazebo reference="base_link">
@@ -354,6 +336,12 @@
         <material>Gazebo/Blue</material>
     </gazebo>
-    <gazebo reference="laser_support_link">
+    <gazebo reference="head_support_link">
+	<material>Gazebo/Chrome</material>
+    </gazebo>
+    <gazebo reference="head_tilt_link">
         <material>Gazebo/Black</material>
     </gazebo>
+  <material name="Greyish">
+    <color rgba="0.7 0.7 0.7 1.0"/>
+  </material>
 </robot>

File: wubble/wubble_robots/defs/erratic/erratic_head.xacro (robot description, xacro)
@@ -18,5 +18,5 @@
     <macro name="stoc_eye" params="name parent suffix reflect">
         <joint name="${suffix}_stoc_eye_joint" type="fixed">
-            <origin xyz="${(stoc_depth/2)+(eye_length/2)} ${reflect*eye_offset} 0" rpy="0 ${M_PI/2} 0" />
+            <origin xyz="${(stoc_depth/2)+(eye_length/2)} ${reflect*eye_offset} 0.03" rpy="0 ${M_PI/2} 0" />
             <parent link="${parent}" />
             <child link="${suffix}_stoc_eye_link"/>
@@ -101,9 +101,22 @@
     </macro>
     <macro name="stoc_camera" params="name parent">
-        <joint name="stoc_camera_joint" type="fixed">
-            <origin xyz="0 0 0.5" rpy="0 0 0" />
+<!--        <joint name="stoc_camera_joint" type="fixed">
+            <origin xyz="0 0 ${(stoc_height/2)+0.0254}" rpy="0 0 0" />
             <parent link="${parent}" />
             <child link="stoc_camera_link"/>
         </joint>
+-->
+    <joint name="stoc_camera_joint" type="fixed"><!--revolute"> -->
+      <origin xyz="0 0 ${(stoc_height/2)}" rpy="0 0 0" />
+      <axis xyz="0 1 0" />
+      <limit lower="-0.785" upper="1.57" effort="0.5292" velocity="10.0" />
+      <safety_controller k_position="100" k_velocity="0.05" soft_lower_limit="${-0.785+0.0}" soft_upper_limit="${1.57-0.0}" />
+      <!-- hold both reference_position and upper/lower for tick-tock, remove reference_positiion after verifying upper/lower works with calibration controllers.  if search velocity in pr2_calibration_controllers.yaml is +, the reference_position is rising, if - then it is falling -->
+      <calibration reference_position="-.35}" falling="-.35" />
+      <dynamics damping="0.008" />
+<!--      <insert_block name="origin" /> -->
+      <parent link="${parent}"/>
+      <child link="stoc_camera_link"/>
+    </joint>
         <link name="stoc_camera_link">
             <inertial>
@@ -115,5 +128,5 @@
             </inertial>
             <visual>
-                <origin xyz="0 0 0" rpy="0 0 0" />
+                <origin xyz="0 0 0.03" rpy="0 0 0" />
                 <geometry>
                     <box size="${stoc_depth} ${stoc_width} ${stoc_height}" />
@@ -121,5 +134,5 @@
             </visual>
             <collision>
-                <origin xyz="0 0 0" rpy="0 0 0" />
+                <origin xyz="0 0 0.03" rpy="0 0 0" />
                 <geometry>
                     <box size="${stoc_depth} ${stoc_width} ${stoc_height}" />
@@ -128,5 +141,5 @@
         </link>
         <joint name="stoc_back_joint" type="fixed">
-            <origin xyz="${-(stoc_depth/2)-(back_depth/2)} 0 0" rpy="0 0 0" />
+            <origin xyz="${-(stoc_depth/2)-(back_depth/2)} 0 0.03" rpy="0 0 0" />
             <parent link="stoc_camera_link" />
             <child link="stoc_back_link"/>
@@ -156,5 +169,5 @@
         <stoc_eye name="right_eye" parent="stoc_camera_link" suffix="right" reflect="-1"/>
         <joint name="stoc_optical_frame_joint" type="fixed">
-            <origin xyz="${cal_stereo_x}            ${0.045+cal_stereo_y}   ${.0305+cal_stereo_z}" rpy="${-M_PI/2+cal_stereo_roll} ${0.0+cal_stereo_pitch} ${-M_PI/2+cal_stereo_yaw}" />
+            <origin xyz="${cal_stereo_x}            ${0.045+cal_stereo_y}   ${.0305+cal_stereo_z+0.03}" rpy="${-M_PI/2+cal_stereo_roll} ${0.0+cal_stereo_pitch} ${-M_PI/2+cal_stereo_yaw}" />
             <parent link="stoc_camera_link"/>
             <child link="stoc_optical_frame"/>

Commit message: 

File: wubble/wubble_robots/defs/erratic/erratic.urdf.xacro (robot description, xacro)
@@ -237,5 +237,5 @@
         </collision>
     </link>
-    <joint name="head_tilt_joint" type="fixed"><!--type="continuous">-->
+    <joint name="head_pan_joint" type="fixed"><!--type="continuous">-->
         <origin xyz="0 0 ${support_height/2}" />
         <axis xyz="0 0 1" />
@@ -244,7 +244,7 @@
         <joint_properties damping="0.0" friction="0.0" /> -->
         <parent link="head_support_link" />
-        <child link="head_tilt_link" />
+        <child link="head_pan_link" />
     </joint>
-    <link name="head_tilt_link">
+    <link name="head_pan_link">
         <inertial>
             <mass value="0.01"/>
@@ -265,10 +265,4 @@
         </collision>
     </link>
-<!--    <joint name="head_pitch_joint" type="fixed">
-       <origin xyz="0 0 ${support_height+base_size_z}" />
-        <parent link="head_support_link" />
-        <child link="stoc_camera_link" />
-    </joint>
--->
   <gazebo>
     <controller:differential_position2d name="controller1">
@@ -301,20 +295,10 @@
     </controller:gazebo_ros_controller_manager>
   </gazebo>
-    <!-- PR2-derived things. These will need to be adapted further to match what we have -->
-<!--    <pr2_head name="head" parent="base_top_link">-->
-<!--    <origin xyz="${cal_head_x}    ${cal_head_y}     ${0.3915+cal_head_z}"-->
-<!--            rpy="${cal_head_roll} ${cal_head_pitch} ${cal_head_yaw}" />-->
-<!--    </pr2_head>-->
-    <!-- Camera package: double stereo, prosilica -->
-<!--    <pr2_head_sensor_package name="sensor_mount" hd_name="high_def" -->
-<!--		       stereo_name="double_stereo" -->
-<!--		       parent="head_plate_frame">-->
-<!--    <origin xyz="0.0 0.0 0.0" rpy="0 0 0" />-->
-<!--    </pr2_head_sensor_package>-->
     <!-- attempt to add the pan-tilt laser from the pr2, it should be close enough -->
     <pr2_tilting_laser name="laser_tilt" parent="base_top_link" laser_calib_ref="-0.35">
         <origin xyz="0.1 0 ${base_size_z - 0.05}" rpy="0 -1 0" />
     </pr2_tilting_laser>
-    <stoc_camera name="stoc" parent="head_tilt_link" />
+    <stoc_camera name="stoc" parent="head_pan_link" />
+    <arm name="arm" parent="base_top_link" />
     <!-- Gazebo materials -->
     <gazebo reference="base_link">
@@ -339,9 +323,6 @@
 	<material>Gazebo/Chrome</material>
     </gazebo>
-    <gazebo reference="head_tilt_link">
+    <gazebo reference="head_pan_link">
         <material>Gazebo/Black</material>
     </gazebo>
-  <material name="Greyish">
-    <color rgba="0.7 0.7 0.7 1.0"/>
-  </material>
 </robot>

File: wubble/wubble_robots/defs/overhead_cam/overhead_cam.urdf.xacro (robot description, xacro)
@@ -34,5 +34,5 @@
         <sensor:camera name="overhead_cam_sensor">
             <imageSize>1024 1024</imageSize>
-            <imageFormat>B8G8R8</imageFormat>
+            <imageFormat>RGB8</imageFormat>
             <hfov>90</hfov>
             <nearClip>0.1</nearClip>
