Commit message: Added stub beginning of arm, reworked coordinate system for erratic model from scratch

File: wubble/wubble_robots/defs/erratic/erratic_head.xacro (robot description, xacro)
@@ -107,16 +107,21 @@
         </joint>
 -->
-    <joint name="stoc_camera_joint" type="fixed"><!--revolute"> -->
-      <origin xyz="0 0 ${(stoc_height/2)}" rpy="0 0 0" />
-      <axis xyz="0 1 0" />
-      <limit lower="-0.785" upper="1.57" effort="0.5292" velocity="10.0" />
-      <safety_controller k_position="100" k_velocity="0.05" soft_lower_limit="${-0.785+0.0}" soft_upper_limit="${1.57-0.0}" />
-      <!-- hold both reference_position and upper/lower for tick-tock, remove reference_positiion after verifying upper/lower works with calibration controllers.  if search velocity in pr2_calibration_controllers.yaml is +, the reference_position is rising, if - then it is falling -->
-      <calibration reference_position="-.35}" falling="-.35" />
-      <dynamics damping="0.008" />
-<!--      <insert_block name="origin" /> -->
-      <parent link="${parent}"/>
-      <child link="stoc_camera_link"/>
+    <joint name="stoc_camera_joint" type="revolute">
+        <origin xyz="0 0 ${(stoc_height/2)}" rpy="0 0 0" />
+        <parent link="${parent}"/>
+        <child link="stoc_camera_link"/>
+<!--      <limit lower="-0.785" upper="1.57" effort="0.5292" velocity="10.0" />-->
+        <axis xyz="0 1 0" />
+        <limit lower="0" upper="0" effort="0.5292" velocity="10.0" />
+        <safety_controller k_position="100" k_velocity="0.05" soft_lower_limit="${-0.785+0.0}" soft_upper_limit="${1.57-0.0}" />
+        <!-- hold both reference_position and upper/lower for tick-tock, remove reference_positiion after verifying upper/lower works with calibration controllers.  if search velocity in pr2_calibration_controllers.yaml is +, the reference_position is rising, if - then it is falling -->
+        <calibration reference_position="-.35" falling="-.35" />
+        <dynamics damping="0.008" />
     </joint>
+    <transmission type="SimpleTransmission" name="head_tilt_trans">
+        <actuator name="head_tilt_motor" />
+        <joint name="stoc_camera_joint" />
+        <mechanicalReduction>6.0</mechanicalReduction>
+    </transmission>
         <link name="stoc_camera_link">
             <inertial>
@@ -150,5 +155,6 @@
                 <origin xyz="${back_depth/2} ${back_width/2} ${back_height/2}" />
                 <inertia ixx="1.0" ixy="0.0" ixz="0.0"
-                         iyy="1.0" iyz="0.0" izz="1.0" />
+                         iyy="1.0" iyz="0.0"
+                         izz="1.0" />
                 <!-- Still don't know what that stuff means? -->
             </inertial>
@@ -169,5 +175,6 @@
         <stoc_eye name="right_eye" parent="stoc_camera_link" suffix="right" reflect="-1"/>
         <joint name="stoc_optical_frame_joint" type="fixed">
-            <origin xyz="${cal_stereo_x}            ${0.045+cal_stereo_y}   ${.0305+cal_stereo_z+0.03}" rpy="${-M_PI/2+cal_stereo_roll} ${0.0+cal_stereo_pitch} ${-M_PI/2+cal_stereo_yaw}" />
+            <origin xyz="${cal_stereo_x}  ${0.045+cal_stereo_y}  ${.0305+cal_stereo_z+0.03}"
+                    rpy="${-M_PI/2+cal_stereo_roll} ${0.0+cal_stereo_pitch} ${-M_PI/2+cal_stereo_yaw}" />
             <parent link="stoc_camera_link"/>
             <child link="stoc_optical_frame"/>
@@ -178,26 +185,30 @@
                 <origin xyz="0 0 0" rpy="0 0 0" />
                 <inertia ixx="0.001"  ixy="0.0"  ixz="0.0"
-                     iyy="0.001"  iyz="0.0"
-                     izz="0.001" />
+                         iyy="0.001"  iyz="0.0"
+                         izz="0.001" />
             </inertial>
             <visual name="stoc_optical_frame_visual">
                 <origin xyz="0 0 0" rpy="0 0 0" />
                 <geometry name="stoc_optical_frame_visual_geom">
-                <box size="0.01 0.01 0.01" />
-            </geometry>
-            <material name="Blue" />
+                    <box size="0.01 0.01 0.01" />
+                </geometry>
             </visual>
             <collision name="stoc_optical_frame_collision">
                 <origin xyz="0 0 0" rpy="0 0 0" />
                 <geometry name="stoc_optical_frame_collision_geom">
-                <box size="0.01 0.01 0.01" />
-                </geometry>
-            </collision>
-        </link>
+                    <box size="0.01 0.01 0.01" />
+                </geometry>
+            </collision>
+        </link>
+        <gazebo reference="stoc_optical_frame" >
+            <material name="clearish">
+                <color rgba="0 0 1 0.5"/>
+            </material>
+        </gazebo>
         <gazebo reference="stoc_camera_link" >
-            <material>Gazebo/Red</material>
+            <material>PR2/Red</material>
         </gazebo>
         <gazebo reference="stoc_back_link" >
-            <material>Gazebo/Red</material>
+            <material>PR2/Red</material>
         </gazebo>
     </macro>

Commit message: New erratic top

File: wubble/wubble_robots/defs/erratic/erratic.urdf.xacro (robot description, xacro)
@@ -5,7 +5,5 @@
     xmlns:interface="http://playerstage.sourceforge.net/gazebo/xmlschema/#interface">
     <!-- Included URDF Files -->
-    <!-- Include file with calibration parameters -->
     <include filename="$(find pr2_defs)/calibration/default_cal.xml" />
-<!--    <include filename="$(find pr2_defs)/defs/head/head_defs.urdf.xacro" />-->
     <include filename="$(find wubble_robots)/defs/erratic/head_sensor_package_defs.urdf.xacro" />
     <include filename="$(find pr2_defs)/defs/materials.urdf.xacro" />
@@ -15,18 +13,15 @@
     <!-- Properties (Constants) -->
     <property name="M_PI" value="3.14159"/>
-<!--    <property name="base_size_x" value="0.395224" />-->
-<!--    <property name="base_size_y" value="0.367284" />-->
-<!--    <property name="base_size_z" value="0.135448" />-->
     <property name="base_size_x" value="0.22" />
     <property name="base_size_y" value="0.29" />
     <property name="base_size_z" value="0.135448" /> <!-- 0.14 -->
-    <property name="top_size_x" value="0.394" />
-    <property name="top_size_y" value="0.356" />
-    <property name="top_size_z" value="0.015" />
+    <property name="top_size_x" value="0.3937" />
+    <property name="top_size_y" value="0.3556" />
+    <property name="top_size_z" value="0.0020" />
     <property name="wheel_radius" value="0.0625" />
     <property name="wheel_length" value="0.02" />
     <property name="caster_wheel_offset_y" value="0.17" />
     <property name="caster_support_x" value="0.086" />
-    <property name="caster_support_z" value="0.10" />
+    <property name="caster_support_z" value="0.095" />
     <property name="support_radius" value="0.01" />
     <property name="support_height" value="0.8128" />
@@ -41,5 +36,5 @@
         </inertial>
         <visual>
-            <origin xyz="0 0 0" rpy="0 0 0" />
+            <origin xyz="0.0 0.0 0.0" rpy="0 0 0" />
             <geometry>
                 <box size="${base_size_x} ${base_size_y} ${base_size_z}" />
@@ -47,5 +42,5 @@
         </visual>
         <collision>
-            <origin xyz="0 0 0" rpy="0 0 0" />
+            <origin xyz="0.0 0.0 0.0" rpy="0 0 0" />
             <geometry>
                 <box size="${base_size_x} ${base_size_y} ${base_size_z}" />
@@ -61,52 +56,48 @@
         <inertial>
             <mass value="1.0"/>
+            <origin xyz="-0.00125736 0.0 -0.0032368" />
+            <inertia ixx="0.00995424" ixy="0.0" ixz="0.00000413"
+                     iyy="0.01191941" iyz="0.0" izx="0.00000413"
+                     izz="0.02181097" />
+        </inertial>
+        <visual>
+            <origin xyz="0.0 0.0 0.0" rpy="0 0 0" />
+                <geometry>
+                    <mesh filename="package://wubble_robots/meshes/erratic_top_origin.stl"/>
+                </geometry>
+        </visual>
+        <collision>
+            <origin xyz="0.0 0.0 0.0" rpy="0 0 0" />
+            <geometry>
+                <mesh filename="package://wubble_robots/meshes/erratic_top_origin.stl"/>
+            </geometry>
+        </collision>
+    </link>
+    <joint name="base_caster_box_joint" type="fixed">
+        <origin xyz="-${base_size_x/2 + caster_support_x/2} 0 0.02" rpy="0 0 0" />
+        <parent link="base_link" />
+        <child link="base_caster_box_link"/>
+    </joint>
+    <link name="base_caster_box_link">
+        <inertial>
+            <mass value="0.1"/>
             <origin xyz="0 0 0" />
-            <inertia ixx="0.0652232699207" ixy="0.0" ixz="0.0"
-                     iyy="0.0669473158652" iyz="0.0"
-                     izz="0.0683196351726" />
-        </inertial>
-        <visual>
-            <origin xyz="0 0 0" rpy="0 0 0" />
-<!--        <geometry>-->
-<!--            <mesh filename="package://wubble_robots/meshes/erratic_top_final.stl"/>-->
-<!--            <mesh filename="package://wubble_robots/meshes/erratic_top.stl"-->
-<!--                  scale="${base_size_x/2.0} ${base_size_y/2.0} 0.05">-->
-<!--            </mesh>-->
-<!--        </geometry>-->
-            <geometry>
-                <box size="${top_size_x} ${top_size_y} ${top_size_z}" />
-            </geometry>
-        </visual>
-        <collision>
-            <origin xyz="0 0 0" rpy="0 0 0" />
-            <geometry>
-                <box size="${top_size_x} ${top_size_y} ${top_size_z}" />
-            </geometry>
-        </collision>
-    </link>
-  <joint name="base_caster_box_joint" type="fixed">
-    <origin xyz="-${base_size_x/2 + caster_support_x/2} 0 0.02" rpy="0 0 0" />
-    <parent link="base_link" />
-    <child link="base_caster_box_link"/>
-  </joint>
-  <link name="base_caster_box_link">
-    <inertial>
-      <mass value="0.1"/>
-      <origin xyz="0 0 0" />
-      <inertia ixx="0.01" ixy="0.0" ixz="0.0"
-               iyy="0.01" iyz="0.0"
-               izz="0.01" />
-    </inertial>
-    <visual>
-      <geometry>
-        <box size="${caster_support_x} 0.02 ${caster_support_z}" />
-      </geometry>
-    </visual>
-    <collision>
-      <geometry>
-        <box size="${caster_support_x} 0.02 ${caster_support_z}" />
-      </geometry>
-    </collision>
-  </link>
+            <inertia ixx="0.01" ixy="0.0" ixz="0.0"
+                     iyy="0.01" iyz="0.0"
+                     izz="0.01" />
+        </inertial>
+        <visual>
+            <origin xyz="0.0 0.0 0.0" rpy="0 0 0" />
+            <geometry>
+                <box size="${caster_support_x} 0.02 ${caster_support_z}" />
+            </geometry>
+        </visual>
+        <collision>
+            <origin xyz="0.0 0.0 0.0" rpy="0 0 0" />
+            <geometry>
+                <box size="${caster_support_x} 0.02 ${caster_support_z}" />
+            </geometry>
+        </collision>
+    </link>
     <joint name="base_caster_support_joint" type="continuous">
         <origin xyz="${-caster_support_x/2 + 0.015} 0 ${-caster_support_z/2 - 0.03}" rpy="0 0 0" />
@@ -150,20 +141,21 @@
     <link name="caster_wheel_link">
         <inertial>
-          <mass value="0.1" />
-          <origin xyz=" 0 0 0 " />
-          <inertia  ixx="0.012411765597" ixy="-0.000711733678" ixz="0.00050272983"
-                    iyy="0.015218160428" iyz="-0.000004273467" izz="0.011763977943" />
-        </inertial>
-        <visual>
-          <origin xyz="0 0 0" rpy="${M_PI/2} 0 0" />
-          <geometry>
+            <mass value="0.1" />
+            <origin xyz="0.0 0.0 0.0" rpy="0 0 0" />
+            <inertia  ixx="0.012411765597" ixy="-0.000711733678" ixz="0.00050272983"
+                      iyy="0.015218160428" iyz="-0.000004273467"
+                      izz="0.011763977943" />
+        </inertial>
+        <visual>
+            <origin xyz="0 0 0" rpy="${M_PI/2} 0 0" />
+            <geometry>
+                <cylinder radius="0.03" length="0.01" />
+            </geometry>
+        </visual>
+        <collision>
+        <origin xyz="0 0 0" rpy="${M_PI/2} 0 0" />
+        <geometry>
             <cylinder radius="0.03" length="0.01" />
-          </geometry>
-        </visual>
-        <collision>
-          <origin xyz="0 0 0" rpy="${M_PI/2} 0 0" />
-          <geometry>
-            <cylinder radius="0.03" length="0.01" />
-          </geometry>
+        </geometry>
         </collision>
     </link>
@@ -182,9 +174,9 @@
         <inertial>
             <mass value="0.1"/>
-            <origin xyz="0 0 0.0"/>
+            <origin xyz="0.0 0.0 0.0" rpy="0 0 0" />
             <inertia ixx="0.1" ixy="0" ixz="0" iyy="0.1" iyz="0" izz="0.1"/>
         </inertial>
         <visual>
-            <origin rpy="0 0 0" xyz="0 0 0"/>
+            <origin xyz="0.0 0.0 0.0" rpy="0 0 0" />
             <geometry>
                 <cylinder radius="${support_radius}" length="${support_height}"/>
@@ -192,5 +184,5 @@
         </visual>
         <collision>
-            <origin rpy="0 0 0" xyz="0 0 0"/>
+            <origin xyz="0.0 0.0 0.0" rpy="0 0 0" />
             <geometry>
                 <cylinder radius="${support_radius}" length="${support_height}"/>
@@ -217,5 +209,5 @@
         <inertial>
             <mass value="0.01"/>
-            <origin xyz="0 0 0.0"/>
+            <origin xyz="0.0 0.0 0.0" rpy="0 0 0" />
             <inertia ixx="0.01" ixy="0" ixz="0" iyy="0.01" iyz="0" izz="0.01"/>
         </inertial>
@@ -242,34 +234,34 @@
     <arm parent="base_top_link" />
     <!-- CONTROLLERS -->
-  <gazebo>
-    <controller:differential_position2d name="controller1">
-      <update>100</update>
-      <leftJoint>base_link_right_wheel_joint</leftJoint>
-      <rightJoint>base_link_left_wheel_joint</rightJoint>
-      <wheelSeparation>${caster_wheel_offset_y*2}</wheelSeparation>
-      <wheelDiameter>${wheel_radius*2}</wheelDiameter>
-      <torque>5</torque>
-      <interface:position name="position_iface_0"/>
-    </controller:differential_position2d>
-    <controller:gazebo_ros_p3d name="p3d_base_controller" plugin="libgazebo_ros_p3d.so">
-      <alwaysOn>true</alwaysOn>
-      <updateRate>100.0</updateRate>
-      <bodyName>base_link</bodyName>
-      <topicName>base_pose_ground_truth</topicName>
-      <gaussianNoise>0.01</gaussianNoise>
-      <frameName>map</frameName>
-      <xyzOffsets>0 0 0</xyzOffsets> <!-- initialize odometry for fake localization-->
-      <rpyOffsets>0 0 0</rpyOffsets>
-      <interface:position name="p3d_base_position"/>
-    </controller:gazebo_ros_p3d>
-    <!-- this publishes empty joint_states due to no transmission, but
+    <gazebo>
+        <controller:differential_position2d name="controller1">
+            <update>100</update>
+            <leftJoint>base_link_right_wheel_joint</leftJoint>
+            <rightJoint>base_link_left_wheel_joint</rightJoint>
+            <wheelSeparation>${caster_wheel_offset_y*2}</wheelSeparation>
+            <wheelDiameter>${wheel_radius*2}</wheelDiameter>
+            <torque>5</torque>
+            <interface:position name="position_iface_0"/>
+        </controller:differential_position2d>
+        <controller:gazebo_ros_p3d name="p3d_base_controller" plugin="libgazebo_ros_p3d.so">
+            <alwaysOn>true</alwaysOn>
+            <updateRate>100.0</updateRate>
+            <bodyName>base_link</bodyName>
+            <topicName>base_pose_ground_truth</topicName>
+            <gaussianNoise>0.01</gaussianNoise>
+            <frameName>map</frameName>
+            <xyzOffsets>0 0 0</xyzOffsets> <!-- initialize odometry for fake localization-->
+            <rpyOffsets>0 0 0</rpyOffsets>
+            <interface:position name="p3d_base_position"/>
+        </controller:gazebo_ros_p3d>
+        <!-- this publishes empty joint_states due to no transmission, but
          triggering robot_state_puublisher to publish tf between fixed joints in erratic,
          (e.g. base_laser_link for the base_scan frame) -->
-    <controller:gazebo_ros_controller_manager name="gazebo_ros_controller_manager" plugin="libgazebo_ros_controller_manager.so">
-      <alwaysOn>true</alwaysOn>
-      <updateRate>1000.0</updateRate>
-      <interface:audio name="gazebo_ros_controller_manager_dummy_iface" />
-    </controller:gazebo_ros_controller_manager>
-  </gazebo>
+        <controller:gazebo_ros_controller_manager name="gazebo_ros_controller_manager" plugin="libgazebo_ros_controller_manager.so">
+            <alwaysOn>true</alwaysOn>
+            <updateRate>100.0</updateRate>
+            <interface:audio name="gazebo_ros_controller_manager_dummy_iface" />
+        </controller:gazebo_ros_controller_manager>
+    </gazebo>
     <!-- GAZEBO MATERIALS -->
     <gazebo reference="base_link">
@@ -292,5 +284,5 @@
     </gazebo>
     <gazebo reference="head_support_link">
-	    <material>Gazebo/Chrome</material>
+        <material>Gazebo/Chrome</material>
     </gazebo>
     <gazebo reference="head_pan_link">
