Commit message: Added wheel model and textures for base, camera support and arm. Fixed keyboard teleop.

File: wubble/wubble_robots/defs/erratic/erratic.urdf.xacro (robot description, xacro)
@@ -23,5 +23,5 @@
     <property name="caster_wheel_offset_y" value="0.17" />
     <property name="caster_support_x" value="0.086" />
-    <property name="caster_support_z" value="0.095" />
+    <property name="caster_support_z" value="0.088148" />
     <property name="support_radius" value="0.01" />
     <property name="support_height" value="0.8128" />
@@ -30,5 +30,5 @@
         <inertial>
             <mass value="20" />
-            <origin xyz="0 0 0" />
+            <origin xyz="${-base_size_x/2} 0 ${-base_size_z/2}" />
             <inertia ixx="1.0" ixy="0.0" ixz="0.0"
                      iyy="1.0" iyz="0.0"
@@ -75,5 +75,5 @@
     </link>
     <joint name="base_caster_box_joint" type="fixed">
-        <origin xyz="-${base_size_x/2 + caster_support_x/2} 0 0.02" rpy="0 0 0" />
+        <origin xyz="-${base_size_x/2 + caster_support_x/2} 0 ${base_size_z/2 - caster_support_z/2}" rpy="0 0 0" />
         <parent link="base_link" />
         <child link="base_caster_box_link"/>
@@ -131,5 +131,5 @@
     </link>
     <joint name="caster_wheel_joint" type="continuous">
-        <origin xyz="-0.02 0 -0.02" rpy="0 0 0" />
+        <origin xyz="-0.015 0 -0.03" rpy="0 0 0" />
         <parent link="base_caster_support_link" />
         <child link="caster_wheel_link" />
@@ -150,5 +150,5 @@
             <origin xyz="0 0 0" rpy="${M_PI/2} 0 0" />
             <geometry>
-                <cylinder radius="0.03" length="0.01" />
+                <cylinder radius="0.0381" length="0.01" />
             </geometry>
         </visual>
@@ -156,5 +156,5 @@
         <origin xyz="0 0 0" rpy="${M_PI/2} 0 0" />
         <geometry>
-            <cylinder radius="0.03" length="0.01" />
+            <cylinder radius="0.0381" length="0.01" />
         </geometry>
         </collision>
@@ -266,11 +266,11 @@
     <!-- GAZEBO MATERIALS -->
     <gazebo reference="base_link">
-        <material>PR2/Blue</material>
+        <material>Wubble/BlueBrushedAluminum</material>
     </gazebo>
     <gazebo reference="base_top_link">
-        <material>PR2/Blue</material>
+        <material>Wubble/BlueBrushedAluminum</material>
     </gazebo>
     <gazebo reference="caster_wheel_link">
-        <material>Gazebo/Black</material>
+        <material>PR2/Black</material>
     </gazebo>
     <gazebo reference="base_laser_link">
@@ -278,14 +278,14 @@
     </gazebo>
     <gazebo reference="base_caster_box_link">
-        <material>PR2/Blue</material>
+        <material>PR2/Black</material>
     </gazebo>
     <gazebo reference="base_caster_support_link">
-        <material>PR2/Blue</material>
+        <material>PR2/White</material>
     </gazebo>
     <gazebo reference="head_support_link">
-        <material>Gazebo/Chrome</material>
+        <material>Wubble/BrassShiny</material>
     </gazebo>
     <gazebo reference="head_pan_link">
-        <material>Gazebo/Black</material>
+        <material>PR2/Black</material>
     </gazebo>
 </robot>

File: wubble/wubble_robots/defs/erratic/erratic_arm.xacro (robot description, xacro)
@@ -30,5 +30,5 @@
         </link>
         <gazebo reference="arm_base_link">
-	        <material>PR2/Grey</material>
+            <material>Wubble/GunMetalBrushedAluminum</material>
         </gazebo>
     </macro>

File: wubble/wubble_robots/defs/erratic/erratic_wheel.xacro (robot description, xacro)
@@ -4,46 +4,78 @@
     xmlns:controller="http://playerstage.sourceforge.net/gazebo/xmlschema/#controller"
     xmlns:interface="http://playerstage.sourceforge.net/gazebo/xmlschema/#interface">
+    <property name="M_PI" value="3.14159"/>
     <property name="wheel_radius" value="0.0625" />
     <property name="wheel_length" value="0.02" />
     <property name="caster_wheel_offset_y" value="0.17" />
-    <property name="wheel_offset_z" value="${-0.115+base_size_z/2}" />
-  <macro name="erratic_wheel" params="suffix parent reflect">
-    <joint name="${parent}_${suffix}_wheel_joint" type="continuous">
-      <origin xyz="0.075 ${reflect*caster_wheel_offset_y} ${wheel_offset_z}" rpy="0 0 0" />
-      <axis xyz="0 1 0" />
-      <anchor xyz="0 0 0" />
-      <limit effort="100" velocity="100" />
-      <joint_properties damping="0.0" friction="0.0" />
-      <parent link="${parent}" />
-      <child link="${parent}_${suffix}_wheel_link" />
-    </joint>
-    <link name="${parent}_${suffix}_wheel_link">
-      <inertial>
-        <mass value="0.1" /> <!-- check jmh 20081205 -->
-        <origin xyz=" 0 0 0 " />
-        <inertia  ixx="0.012411765597" ixy="0.0" ixz="0.0"
-                  iyy="0.015218160428" iyz="0.0"
-                  izz="0.011763977943" />
-      </inertial>
-      <visual>
-        <origin xyz="0 0 0" rpy="${M_PI/2} 0 0" />
-        <geometry>
-          <cylinder radius="${wheel_radius}" length="${wheel_length}" />
-        </geometry>
-      </visual>
-      <collision>
-        <origin xyz="0 0 0" rpy="${M_PI/2} 0 0" />
-        <geometry>
-          <cylinder radius="${wheel_radius}" length="${wheel_length}" />
-        </geometry>
-      </collision>
-    </link>
-    <gazebo reference="${parent}_${suffix}_wheel_link" >
-      <elem key="mu1" value="50.0" />
-      <elem key="mu2" value="50.0" />
-      <elem key="kp"  value="100000000.0" />
-      <elem key="kd"  value="1.0" />
-      <material>Gazebo/Black</material> <!-- Had to add this here because it's a macro -->
-    </gazebo>
-  </macro>
+    <property name="wheel_offset_z" value="${-base_size_z/2 + 0.0236}" />
+    <macro name="erratic_wheel" params="suffix parent reflect">
+        <joint name="${parent}_${suffix}_motor_joint" type="fixed">
+            <origin xyz="0.075 ${reflect*base_size_y/2} ${wheel_offset_z}" rpy="0 0 0" />
+            <parent link="${parent}" />
+            <child link="${parent}_${suffix}_motor_link" />
+        </joint>
+        <link name="${parent}_${suffix}_motor_link">
+            <inertial>
+                <mass value="0.1" />
+                <origin xyz=" 0 ${reflect*0.0125} 0 " />
+                <inertia  ixx="0.012411765597" ixy="0.0" ixz="0.0"
+                          iyy="0.015218160428" iyz="0.0"
+                          izz="0.011763977943" />
+            </inertial>
+            <visual>
+                <origin xyz="0 ${reflect*0.0125} 0" rpy="${M_PI/2} 0 0" />
+                <geometry>
+                    <cylinder radius="0.0127" length="0.025" />
+                </geometry>
+            </visual>
+            <collision>
+                <origin xyz="$0 ${reflect*0.0125} 0" rpy="{M_PI/2} 0 0" />
+                <geometry>
+                    <cylinder radius="0.0127" length="0.025" />
+                </geometry>
+            </collision>
+        </link>
+        <joint name="${parent}_${suffix}_wheel_joint" type="continuous">
+            <origin xyz="0 ${reflect*0.025} 0" rpy="0 0 0" />
+            <axis xyz="0 1 0" />
+            <anchor xyz="0 0 0" />
+            <limit effort="100" velocity="100" />
+            <joint_properties damping="0.0" friction="0.0" />
+            <parent link="${parent}_${suffix}_motor_link" />
+            <child link="${parent}_${suffix}_wheel_link" />
+        </joint>
+        <link name="${parent}_${suffix}_wheel_link">
+            <inertial>
+                <mass value="0.1" />
+                <origin xyz=" 0 0 0 " />
+                <inertia  ixx="0.012411765597" ixy="0.0" ixz="0.0"
+                          iyy="0.015218160428" iyz="0.0"
+                          izz="0.011763977943" />
+            </inertial>
+            <visual>
+                <origin xyz="0 0 0" rpy="0 0 ${M_PI/2}" />
+                <geometry>
+                    <mesh filename="package://wubble_robots/meshes/erratic_wheel.stl"/>
+<!--                    <cylinder radius="${wheel_radius}" length="${wheel_length}" />-->
+                </geometry>
+            </visual>
+            <collision>
+                <origin xyz="0 0 0" rpy="$0 0 ${M_PI/2}" />
+                <geometry>
+                    <mesh filename="package://wubble_robots/meshes/erratic_wheel.stl"/>
+<!--                    <cylinder radius="${wheel_radius}" length="${wheel_length}" />-->
+                </geometry>
+            </collision>
+        </link>
+        <gazebo reference="${parent}_${suffix}_wheel_link" >
+            <elem key="mu1" value="50.0" />
+            <elem key="mu2" value="50.0" />
+            <elem key="kp"  value="100000000.0" />
+            <elem key="kd"  value="1.0" />
+            <material>PR2/Grey</material>
+        </gazebo>
+        <gazebo reference="${parent}_${suffix}_motor_link" >
+            <material>PR2/White</material>
+        </gazebo>
+    </macro>
 </robot>

Commit message: Modified erratic model to have a base_footprint link like PR2, removed static tf publisher hack, switched to local diffdrive plugin which removes debug message and publishes correct transform, modified rviz files to work better, etc.

File: wubble/wubble_robots/defs/erratic/erratic.urdf.xacro (robot description, xacro)
@@ -26,4 +26,35 @@
     <property name="support_radius" value="0.01" />
     <property name="support_height" value="0.8128" />
+    <!-- base_footprint is a fictitious link(frame) that is on the ground right below base_link origin,
+         navigation stack dedpends on this frame -->
+    <link name="base_footprint">
+        <inertial>
+            <mass value="1.0" />
+            <origin xyz="0 0 0" />
+            <inertia ixx="0.01" ixy="0.0" ixz="0.0"
+                     iyy="0.01" iyz="0.0"
+                     izz="0.01" />
+        </inertial>
+        <visual>
+            <origin xyz="0 0 0" rpy="0 0 0" />
+            <geometry>
+                <box size="0.01 0.01 0.01" />
+            </geometry>
+            <material name="Green" />
+        </visual>
+        <collision>
+            <!-- represent base collision with a simple rectangular model, positioned by base_size_z s.t. top
+                 surface of the collision box matches the top surface of the PR2 base -->
+            <origin xyz="0 0 0" rpy="0 0 0" />
+            <geometry>
+              <box size="0.001 0.001 0.001" />
+            </geometry>
+        </collision>
+    </link>
+    <joint name="base_footprint_joint" type="fixed">
+        <origin xyz="0 0 0" rpy="0 0 0" />
+        <parent link="base_footprint"/>
+        <child link="base_link" />
+    </joint>
     <!-- Links and Joints (i.e., the robot) -->
     <link name="base_link">
@@ -40,4 +71,5 @@
                 <box size="${base_size_x} ${base_size_y} ${base_size_z}" />
             </geometry>
+            <material name="Blue" />
         </visual>
         <collision>
@@ -63,7 +95,8 @@
         <visual>
             <origin xyz="0.0 0.0 0.0" rpy="0 0 0" />
-                <geometry>
-                    <mesh filename="package://wubble_robots/meshes/erratic_top_origin.stl"/>
-                </geometry>
+            <geometry>
+                <mesh filename="package://wubble_robots/meshes/erratic_top_origin.stl"/>
+            </geometry>
+            <material name="Blue" />
         </visual>
         <collision>
@@ -92,4 +125,5 @@
                 <box size="${caster_support_x} 0.02 ${caster_support_z}" />
             </geometry>
+            <material name="Blue" />
         </visual>
         <collision>
@@ -109,4 +143,9 @@
         <joint_properties damping="0.0" friction="0.0" />
     </joint>
+    <transmission type="SimpleTransmission" name="base_caster_support_trans">
+        <actuator name="base_caster_support_motor" />
+        <joint name="base_caster_support_joint" />
+        <mechanicalReduction>1.0</mechanicalReduction>
+    </transmission>
     <link name="base_caster_support_link">
         <inertial>
@@ -139,4 +178,9 @@
         <joint_properties damping="0.0" friction="0.0" />
     </joint>
+    <transmission type="SimpleTransmission" name="caster_wheel_trans">
+        <actuator name="caster_wheel_motor" />
+        <joint name="caster_wheel_joint" />
+        <mechanicalReduction>1.0</mechanicalReduction>
+    </transmission>
     <link name="caster_wheel_link">
         <inertial>
@@ -152,4 +196,5 @@
                 <cylinder radius="0.0381" length="0.01" />
             </geometry>
+            <material name="Black"/>
         </visual>
         <collision>
@@ -255,6 +300,7 @@
             <interface:position name="p3d_base_position"/>
         </controller:gazebo_ros_p3d>
+        <canonicalBody>base_footprint</canonicalBody>
         <!-- this publishes empty joint_states due to no transmission, but
-         triggering robot_state_puublisher to publish tf between fixed joints in erratic,
+         triggering robot_state_publisher to publish tf between fixed joints in erratic,
          (e.g. base_laser_link for the base_scan frame) -->
         <controller:gazebo_ros_controller_manager name="gazebo_ros_controller_manager" plugin="libgazebo_ros_controller_manager.so">
@@ -265,4 +311,7 @@
     </gazebo>
     <!-- GAZEBO MATERIALS -->
+    <material name="Black">
+        <color rgba="0.0 0.0 0.0 1.0"/>
+    </material>
     <gazebo reference="base_link">
         <material>Wubble/BlueBrushedAluminum</material>

File: wubble/wubble_robots/defs/erratic/erratic_arm.xacro (robot description, xacro)
@@ -42,4 +42,9 @@
                     velocity="2.33" />
         </joint>
+        <transmission type="SimpleTransmission" name="arm_base_shoulder_trans">
+            <actuator name="arm_base_shoulder_motor" />
+            <joint name="arm_base_shoulder_joint" />
+            <mechanicalReduction>1.0</mechanicalReduction>
+        </transmission>
         <link name="arm_shoulder_pan_link">
             <inertial>

File: wubble/wubble_robots/defs/erratic/erratic_head.xacro (robot description, xacro)
@@ -107,11 +107,10 @@
         </joint>
 -->
-    <joint name="stoc_camera_joint" type="revolute">
+    <joint name="head_tilt_joint" type="revolute">
         <origin xyz="0 0 ${(stoc_height/2)}" rpy="0 0 0" />
         <parent link="${parent}"/>
         <child link="stoc_camera_link"/>
-<!--      <limit lower="-0.785" upper="1.57" effort="0.5292" velocity="10.0" />-->
         <axis xyz="0 1 0" />
-        <limit lower="0" upper="0" effort="0.5292" velocity="10.0" />
+        <limit lower="-0.5" upper="1.00" effort="100" velocity="2.00" />
         <safety_controller k_position="100" k_velocity="0.05" soft_lower_limit="${-0.785+0.0}" soft_upper_limit="${1.57-0.0}" />
         <!-- hold both reference_position and upper/lower for tick-tock, remove reference_positiion after verifying upper/lower works with calibration controllers.  if search velocity in pr2_calibration_controllers.yaml is +, the reference_position is rising, if - then it is falling -->
@@ -121,6 +120,6 @@
     <transmission type="SimpleTransmission" name="head_tilt_trans">
         <actuator name="head_tilt_motor" />
-        <joint name="stoc_camera_joint" />
-        <mechanicalReduction>6.0</mechanicalReduction>
+        <joint name="head_tilt_joint" />
+        <mechanicalReduction>3.0</mechanicalReduction>
     </transmission>
         <link name="stoc_camera_link">

File: wubble/wubble_robots/defs/erratic/erratic_wheel.xacro (robot description, xacro)
@@ -5,5 +5,5 @@
     xmlns:interface="http://playerstage.sourceforge.net/gazebo/xmlschema/#interface">
     <property name="M_PI" value="3.14159"/>
-    <property name="wheel_radius" value="0.0625" />
+    <property name="wheel_radius" value="0.0762" />
     <property name="wheel_length" value="0.02" />
     <property name="caster_wheel_offset_y" value="0.17" />
@@ -57,6 +57,6 @@
                 <geometry>
                     <mesh filename="package://wubble_robots/meshes/erratic_wheel.stl"/>
-<!--                    <cylinder radius="${wheel_radius}" length="${wheel_length}" />-->
                 </geometry>
+                <material name="Black" />
             </visual>
             <collision>
@@ -78,4 +78,9 @@
             <material>PR2/White</material>
         </gazebo>
+        <transmission type="SimpleTransmission" name="${parent}_${suffix}_wheel_trans">
+            <actuator name="${parent}_${suffix}_wheel_motor" />
+            <joint name="${parent}_${suffix}_wheel_joint" />
+            <mechanicalReduction>1.0</mechanicalReduction>
+        </transmission>
     </macro>
 </robot>

Commit message: Added shoulder_tilt link for the arm, changed texture on camera support to something less shiny.

File: wubble/wubble_robots/defs/erratic/erratic.urdf.xacro (robot description, xacro)
@@ -333,5 +333,5 @@
     </gazebo>
     <gazebo reference="head_support_link">
-        <material>Wubble/BrassShiny</material>
+        <material>Wubble/BrassScratched</material>
     </gazebo>
     <gazebo reference="head_pan_link">

File: wubble/wubble_robots/defs/erratic/erratic_arm.xacro (robot description, xacro)
@@ -49,5 +49,5 @@
         <link name="arm_shoulder_pan_link">
             <inertial>
-                <mass value="0.1" />
+                <mass value="0.3" />
                 <origin xyz="0.0 0.0 0.0" rpy="0 0 0" />
                 <inertia ixx="1.0" ixy="0.0" ixz="0.0"
@@ -68,4 +68,40 @@
             </collision>
         </link>
+        <joint name="arm_shoulder_pan_tilt_joint" type="revolute">
+            <origin xyz="0.08995 0 0.0450" rpy="0 0 0" />
+            <parent link="arm_shoulder_pan_link"/>
+            <child link="arm_shoulder_tilt_link" />
+            <axis xyz="0 1 0"/>
+            <limit  lower="-1.972222"
+                    upper="1.04719755"
+                    effort="100"
+                    velocity="2.33" />
+        </joint>
+        <link name="arm_shoulder_tilt_link">
+            <inertial>
+                <mass value="0.18" />
+                <origin xyz="0.0 0.017 0.0" rpy="0 0 0" />
+                <inertia ixx="1.0" ixy="0.0" ixz="0.0"
+                         iyy="1.0" iyz="0.0"
+                         izz="1.0" />
+            </inertial>
+            <visual>
+                <origin xyz="0.0 0.0 0.0" rpy="0 0 0" />
+                <geometry>
+                    <mesh filename="package://wubble_robots/meshes/arm_shoulder_tilt.stl"/>
+                </geometry>
+            </visual>
+            <collision>
+                <origin xyz="0.0 0.0 0.0" rpy="0 0 0" />
+                <geometry>
+                    <mesh filename="package://wubble_robots/meshes/arm_shoulder_tilt.stl"/>
+                </geometry>
+            </collision>
+        </link>
+        <transmission type="SimpleTransmission" name="arm_base_shoulder_tilt_trans">
+            <actuator name="arm_base_shoulder_tilt_motor" />
+            <joint name="arm_shoulder_pan_tilt_joint" />
+            <mechanicalReduction>1.0</mechanicalReduction>
+        </transmission>
         <gazebo reference="arm_base_link">
             <material>Wubble/GunMetalBrushedAluminum</material>
@@ -74,4 +110,7 @@
             <material>Wubble/GunMetalBrushedAluminum</material>
         </gazebo>
+        <gazebo reference="arm_shoulder_tilt_link">
+            <material>Wubble/GunMetalBrushedAluminum</material>
+        </gazebo>
     </macro>
 </robot>

Commit message: Updated laser model so it should match robot better, and sensor should be upside-down, also fixed other model problems with footprint

File: wubble/wubble_robots/defs/erratic/erratic.urdf.xacro (robot description, xacro)
@@ -5,5 +5,5 @@
     xmlns:interface="http://playerstage.sourceforge.net/gazebo/xmlschema/#interface">
     <!-- Included URDF Files -->
-    <include filename="$(find pr2_defs)/calibration/default_cal.xml" />
+    <include filename="$(find wubble_robots)/calibration/default_cal.xml" />
     <include filename="$(find wubble_robots)/defs/erratic/head_sensor_package_defs.urdf.xacro" />
     <include filename="$(find pr2_defs)/defs/materials.urdf.xacro" />
@@ -37,4 +37,5 @@
         </inertial>
         <visual>
+            <!-- Hiding the base_footprint at the center of the body -->
             <origin xyz="0 0 0" rpy="0 0 0" />
             <geometry>
@@ -44,7 +45,5 @@
         </visual>
         <collision>
-            <!-- represent base collision with a simple rectangular model, positioned by base_size_z s.t. top
-                 surface of the collision box matches the top surface of the PR2 base -->
-            <origin xyz="0 0 0" rpy="0 0 0" />
+            <origin xyz="0 0 ${base_size_z/2 + 0.051}" rpy="0 0 0" />
             <geometry>
               <box size="0.001 0.001 0.001" />
@@ -53,5 +52,7 @@
     </link>
     <joint name="base_footprint_joint" type="fixed">
-        <origin xyz="0 0 0" rpy="0 0 0" />
+        <!-- NB: While you would think this would make it go up, it is oddly reversed.
+             This moves the joint to 0,0,0 where we want it for rviz, etc. -->
+        <origin xyz="0 0 ${base_size_z/2 + 0.051}" rpy="0 0 0" />
         <parent link="base_footprint"/>
         <child link="base_link" />
@@ -273,7 +274,7 @@
     <erratic_wheel suffix="left" parent="base_link" reflect="1"/>
     <erratic_wheel suffix="right" parent="base_link" reflect="-1"/>
-    <pr2_tilting_laser name="laser_tilt" parent="base_top_link" laser_calib_ref="-0.35">
-        <origin xyz="0.15 0 ${-top_size_z - 0.05}" rpy="0 -1 0" />
-    </pr2_tilting_laser>
+    <tilting_hokuyo parent="base_top_link">
+        <origin xyz="0.15 0 ${-top_size_z - 0.05}" rpy="${M_PI} 0 0" />
+    </tilting_hokuyo>
     <stoc_camera name="stoc" parent="head_pan_link" />
     <arm parent="base_top_link" />
