Commit message: Added new arm base and arm shoulder links

File: wubble/wubble_robots/defs/erratic/erratic_arm.xacro (robot description, xacro)
@@ -13,5 +13,5 @@
             <inertial>
                 <mass value="0.1" />
-                <origin xyz="0 0 0" />
+                <origin xyz="0.0 0.0 0.0" rpy="0 0 0" />
                 <inertia ixx="1.0" ixy="0.0" ixz="0.0"
                          iyy="1.0" iyz="0.0"
@@ -19,11 +19,40 @@
             </inertial>
             <visual>
+                <origin xyz="0.0 0.0 0.0" rpy="0 0 0" />
+                <geometry>
+<!--                    <box size="${0.0575*2} ${0.0575*2} ${0.025*2}" />-->
+                    <mesh filename="package://wubble_robots/meshes/arm_base.stl"/>
+                </geometry>
+            </visual>
+            <collision>
+                <origin xyz="0.0 0.0 0.0" rpy="0 0 0" />
                 <geometry>
                     <box size="${0.0575*2} ${0.0575*2} ${0.025*2}" />
                 </geometry>
+            </collision>
+        </link>
+        <joint name="arm_base_shoulder_joint" type="fixed" >
+            <origin xyz="-0.0075 0 0.025" rpy="0 0 0" />
+            <parent link="arm_base_link" />
+            <child link="arm_shoulder_pan_link"/>
+        </joint>
+        <link name="arm_shoulder_pan_link">
+            <inertial>
+                <mass value="0.1" />
+                <origin xyz="0.0 0.0 0.0" rpy="0 0 0" />
+                <inertia ixx="1.0" ixy="0.0" ixz="0.0"
+                         iyy="1.0" iyz="0.0"
+                         izz="1.0" />
+            </inertial>
+            <visual>
+                <origin xyz="0.0 0.0 0.005" rpy="0 0 0" />
+                <geometry>
+                    <mesh filename="package://wubble_robots/meshes/arm_shoulder.stl"/>
+                </geometry>
             </visual>
             <collision>
+                <origin xyz="0.0 0.0 0.0" rpy="0 0 0" />
                 <geometry>
-                    <box size="${0.0575*2} ${0.0575*2} ${0.025*2}" />
+                    <mesh filename="package://wubble_robots/meshes/arm_shoulder.stl"/>
                 </geometry>
             </collision>
@@ -32,4 +61,7 @@
             <material>Wubble/GunMetalBrushedAluminum</material>
         </gazebo>
+        <gazebo reference="arm_shoulder_pan_link">
+            <material>Wubble/GunMetalBrushedAluminum</material>
+        </gazebo>
     </macro>
 </robot>

Commit message: Added revolute joint and limits to arm shoulder.

File: wubble/wubble_robots/defs/erratic/erratic_arm.xacro (robot description, xacro)
@@ -32,8 +32,13 @@
             </collision>
         </link>
-        <joint name="arm_base_shoulder_joint" type="fixed" >
+        <joint name="arm_base_shoulder_joint" type="revolute" >
             <origin xyz="-0.0075 0 0.025" rpy="0 0 0" />
             <parent link="arm_base_link" />
             <child link="arm_shoulder_pan_link"/>
+            <axis xyz="0 0 1"/>
+            <limit  lower="-1.22"
+                    upper="1.22"
+                    effort="100"
+                    velocity="2.33" />
         </joint>
         <link name="arm_shoulder_pan_link">

Commit message: Added elbow tilt and wrist rotate joints and links to arm model. Some tweaks to joint locations.

File: wubble/wubble_robots/defs/erratic/erratic_arm.xacro (robot description, xacro)
@@ -68,6 +68,7 @@
             </collision>
         </link>
+        <!-- Shoulder tilt joint and link -->
         <joint name="arm_shoulder_pan_tilt_joint" type="revolute">
-            <origin xyz="0.08995 0 0.0450" rpy="0 0 0" />
+            <origin xyz="${0.105 - 0.01 - 0.03085/2} 0 ${0.01 + 0.05 - 0.031/2}" rpy="0 0 0" />
             <parent link="arm_shoulder_pan_link"/>
             <child link="arm_shoulder_tilt_link" />
@@ -81,5 +82,5 @@
             <inertial>
                 <mass value="0.18" />
-                <origin xyz="0.0 0.017 0.0" rpy="0 0 0" />
+                <origin xyz="0.0 0.17 0.0" rpy="0 0 0" />
                 <inertia ixx="1.0" ixy="0.0" ixz="0.0"
                          iyy="1.0" iyz="0.0"
@@ -104,4 +105,80 @@
             <mechanicalReduction>1.0</mechanicalReduction>
         </transmission>
+        <!-- Elbow tilt joint and link -->
+        <joint name="arm_shoulder_tilt_elbow_tilt_joint" type="revolute">
+            <origin xyz="${0.04 - 0.01 + 0.0015 + 0.105 + 0.055 - 0.01} 0 0" rpy="0 0 0" />
+            <parent link="arm_shoulder_tilt_link"/>
+            <child link="arm_elbow_tilt_link" />
+            <axis xyz="0 1 0"/>
+            <!-- From -113 to 108 degrees -->
+            <limit  lower="-1.972222"
+                    upper="1.8849556"
+                    effort="100"
+                    velocity="2.33" />
+        </joint>
+        <link name="arm_elbow_tilt_link">
+            <inertial>
+                <mass value="0.15" />
+                <origin xyz="0.0 0.07 0.0" rpy="0 0 0" />
+                <inertia ixx="1.0" ixy="0.0" ixz="0.0"
+                         iyy="1.0" iyz="0.0"
+                         izz="1.0" />
+            </inertial>
+            <visual>
+                <origin xyz="0.0 0.0 0.0" rpy="0 0 0" />
+                <geometry>
+                    <mesh filename="package://wubble_robots/meshes/arm_elbow_tilt.stl"/>
+                </geometry>
+            </visual>
+            <collision>
+                <origin xyz="0.0 0.0 0.0" rpy="0 0 0" />
+                <geometry>
+                    <mesh filename="package://wubble_robots/meshes/arm_elbow_tilt.stl"/>
+                </geometry>
+            </collision>
+        </link>
+        <transmission type="SimpleTransmission" name="arm_elbow_tilt_trans">
+            <actuator name="arm_elbow_tilt_motor" />
+            <joint name="arm_shoulder_tilt_elbow_tilt_joint" />
+            <mechanicalReduction>1.0</mechanicalReduction>
+        </transmission>
+        <!-- Wrist rotate joint and link -->
+        <joint name="arm_elbow_tilt_wrist_rotate_joint" type="revolute">
+            <origin xyz="${0.08 - 0.01} 0 ${0.05 - 0.0115 - 0.0155}" rpy="0 0 0" />
+            <parent link="arm_elbow_tilt_link"/>
+            <child link="arm_wrist_rotate_link" />
+            <axis xyz="1 0 0"/>
+            <!-- From -150 to 150 degrees -->
+            <limit  lower="-2.6179939"
+                    upper="2.6179939"
+                    effort="100"
+                    velocity="2.33" />
+        </joint>
+        <link name="arm_wrist_rotate_link">
+            <inertial>
+                <mass value="0.12" />
+                <origin xyz="0.0 0.05 0.0" rpy="0 0 0" />
+                <inertia ixx="1.0" ixy="0.0" ixz="0.0"
+                         iyy="1.0" iyz="0.0"
+                         izz="1.0" />
+            </inertial>
+            <visual>
+                <origin xyz="0.0 0.0 0.0" rpy="0 0 0" />
+                <geometry>
+                    <mesh filename="package://wubble_robots/meshes/arm_wrist_rotate.stl"/>
+                </geometry>
+            </visual>
+            <collision>
+                <origin xyz="0.0 0.0 0.0" rpy="0 0 0" />
+                <geometry>
+                    <mesh filename="package://wubble_robots/meshes/arm_wrist_rotate.stl"/>
+                </geometry>
+            </collision>
+        </link>
+        <transmission type="SimpleTransmission" name="arm_wrist_rotate_trans">
+            <actuator name="arm_wrist_rotate_motor" />
+            <joint name="arm_elbow_tilt_wrist_rotate_joint" />
+            <mechanicalReduction>1.0</mechanicalReduction>
+        </transmission>
         <gazebo reference="arm_base_link">
             <material>Wubble/GunMetalBrushedAluminum</material>
@@ -113,4 +190,10 @@
             <material>Wubble/GunMetalBrushedAluminum</material>
         </gazebo>
+        <gazebo reference="arm_elbow_tilt_link">
+            <material>Wubble/GunMetalBrushedAluminum</material>
+        </gazebo>
+        <gazebo reference="arm_wrist_rotate_link">
+            <material>Wubble/GunMetalBrushedAluminum</material>
+        </gazebo>
     </macro>
 </robot>

Commit message: Added gripper's right finger.

File: wubble/wubble_robots/defs/erratic/erratic_arm.xacro (robot description, xacro)
@@ -181,4 +181,42 @@
             <mechanicalReduction>1.0</mechanicalReduction>
         </transmission>
+        <!-- Gripper right finger joint and link -->
+        <joint name="arm_wrist_rotate_right_finger_joint" type="revolute">
+            <origin xyz="${0.0015 + 0.05 - 0.01} ${-0.035/2} 0" rpy="0 0 0" />
+            <parent link="arm_wrist_rotate_link"/>
+            <child link="arm_right_finger_link" />
+            <axis xyz="0 0 1"/>
+            <!-- From -20 to 20 degrees -->
+            <limit  lower="-0.3490658"
+                    upper="0.3490658"
+                    effort="100"
+                    velocity="2.33" />
+        </joint>
+        <link name="arm_right_finger_link">
+            <inertial>
+                <mass value="0.01" />
+                <origin xyz="0.0 0.0 0.0" rpy="0 0 0" />
+                <inertia ixx="1.0" ixy="0.0" ixz="0.0"
+                         iyy="1.0" iyz="0.0"
+                         izz="1.0" />
+            </inertial>
+            <visual>
+                <origin xyz="0.0 0.0 0.0" rpy="0 0 0" />
+                <geometry>
+                    <mesh filename="package://wubble_robots/meshes/arm_right_finger.stl"/>
+                </geometry>
+            </visual>
+            <collision>
+                <origin xyz="0.0 0.0 0.0" rpy="0 0 0" />
+                <geometry>
+                    <mesh filename="package://wubble_robots/meshes/arm_right_finger.stl"/>
+                </geometry>
+            </collision>
+        </link>
+        <transmission type="SimpleTransmission" name="arm_right_finger_trans">
+            <actuator name="arm_right_finger_motor" />
+            <joint name="arm_wrist_rotate_right_finger_joint" />
+            <mechanicalReduction>1.0</mechanicalReduction>
+        </transmission>
         <gazebo reference="arm_base_link">
             <material>Wubble/GunMetalBrushedAluminum</material>
@@ -194,4 +232,7 @@
         </gazebo>
         <gazebo reference="arm_wrist_rotate_link">
+            <material>Wubble/GunMetalBrushedAluminum</material>
+        </gazebo>
+        <gazebo reference="arm_right_finger_link">
             <material>Wubble/GunMetalBrushedAluminum</material>
         </gazebo>

Commit message: Added gripper's left finger.

File: wubble/wubble_robots/defs/erratic/erratic_arm.xacro (robot description, xacro)
@@ -219,4 +219,42 @@
             <mechanicalReduction>1.0</mechanicalReduction>
         </transmission>
+        <!-- Gripper left finger joint and link -->
+        <joint name="arm_wrist_rotate_left_finger_joint" type="revolute">
+            <origin xyz="${0.0015 + 0.05 - 0.01} ${0.035/2} 0" rpy="0 0 0" />
+            <parent link="arm_wrist_rotate_link"/>
+            <child link="arm_left_finger_link" />
+            <axis xyz="0 0 1"/>
+            <!-- From -20 to 20 degrees -->
+            <limit  lower="-0.3490658"
+                    upper="0.3490658"
+                    effort="100"
+                    velocity="2.33" />
+        </joint>
+        <link name="arm_left_finger_link">
+            <inertial>
+                <mass value="0.01" />
+                <origin xyz="0.0 0.0 0.0" rpy="0 0 0" />
+                <inertia ixx="1.0" ixy="0.0" ixz="0.0"
+                         iyy="1.0" iyz="0.0"
+                         izz="1.0" />
+            </inertial>
+            <visual>
+                <origin xyz="0.0 0.0 0.0" rpy="0 0 0" />
+                <geometry>
+                    <mesh filename="package://wubble_robots/meshes/arm_left_finger.stl"/>
+                </geometry>
+            </visual>
+            <collision>
+                <origin xyz="0.0 0.0 0.0" rpy="0 0 0" />
+                <geometry>
+                    <mesh filename="package://wubble_robots/meshes/arm_left_finger.stl"/>
+                </geometry>
+            </collision>
+        </link>
+        <transmission type="SimpleTransmission" name="arm_left_finger_trans">
+            <actuator name="arm_left_finger_motor" />
+            <joint name="arm_wrist_rotate_left_finger_joint" />
+            <mechanicalReduction>1.0</mechanicalReduction>
+        </transmission>
         <gazebo reference="arm_base_link">
             <material>Wubble/GunMetalBrushedAluminum</material>
@@ -235,4 +273,7 @@
         </gazebo>
         <gazebo reference="arm_right_finger_link">
+            <material>Wubble/GunMetalBrushedAluminum</material>
+        </gazebo>
+        <gazebo reference="arm_left_finger_link">
             <material>Wubble/GunMetalBrushedAluminum</material>
         </gazebo>

Commit message: Fix joint states publisher

File: wubble/wubble_robots/defs/erratic/erratic_arm.xacro (robot description, xacro)
@@ -32,5 +32,6 @@
             </collision>
         </link>
-        <joint name="arm_base_shoulder_joint" type="revolute" >
+        <!-- Shoulder pan joint and link -->
+        <joint name="shoulder_pan_joint" type="revolute" >
             <origin xyz="-0.0075 0 0.025" rpy="0 0 0" />
             <parent link="arm_base_link" />
@@ -44,5 +45,5 @@
         <transmission type="SimpleTransmission" name="arm_base_shoulder_trans">
             <actuator name="arm_base_shoulder_motor" />
-            <joint name="arm_base_shoulder_joint" />
+            <joint name="shoulder_pan_joint" />
             <mechanicalReduction>1.0</mechanicalReduction>
         </transmission>
@@ -69,5 +70,5 @@
         </link>
         <!-- Shoulder tilt joint and link -->
-        <joint name="arm_shoulder_pan_tilt_joint" type="revolute">
+        <joint name="shoulder_tilt_joint" type="revolute">
             <origin xyz="${0.105 - 0.01 - 0.03085/2} 0 ${0.01 + 0.05 - 0.031/2}" rpy="0 0 0" />
             <parent link="arm_shoulder_pan_link"/>
@@ -102,9 +103,9 @@
         <transmission type="SimpleTransmission" name="arm_base_shoulder_tilt_trans">
             <actuator name="arm_base_shoulder_tilt_motor" />
-            <joint name="arm_shoulder_pan_tilt_joint" />
+            <joint name="shoulder_tilt_joint" />
             <mechanicalReduction>1.0</mechanicalReduction>
         </transmission>
         <!-- Elbow tilt joint and link -->
-        <joint name="arm_shoulder_tilt_elbow_tilt_joint" type="revolute">
+        <joint name="elbow_tilt_joint" type="revolute">
             <origin xyz="${0.04 - 0.01 + 0.0015 + 0.105 + 0.055 - 0.01} 0 0" rpy="0 0 0" />
             <parent link="arm_shoulder_tilt_link"/>
@@ -140,9 +141,9 @@
         <transmission type="SimpleTransmission" name="arm_elbow_tilt_trans">
             <actuator name="arm_elbow_tilt_motor" />
-            <joint name="arm_shoulder_tilt_elbow_tilt_joint" />
+            <joint name="elbow_tilt_joint" />
             <mechanicalReduction>1.0</mechanicalReduction>
         </transmission>
         <!-- Wrist rotate joint and link -->
-        <joint name="arm_elbow_tilt_wrist_rotate_joint" type="revolute">
+        <joint name="wrist_rotate_joint" type="revolute">
             <origin xyz="${0.08 - 0.01} 0 ${0.05 - 0.0115 - 0.0155}" rpy="0 0 0" />
             <parent link="arm_elbow_tilt_link"/>
@@ -178,9 +179,9 @@
         <transmission type="SimpleTransmission" name="arm_wrist_rotate_trans">
             <actuator name="arm_wrist_rotate_motor" />
-            <joint name="arm_elbow_tilt_wrist_rotate_joint" />
+            <joint name="wrist_rotate_joint" />
             <mechanicalReduction>1.0</mechanicalReduction>
         </transmission>
         <!-- Gripper right finger joint and link -->
-        <joint name="arm_wrist_rotate_right_finger_joint" type="revolute">
+        <joint name="finger_right_joint" type="revolute">
             <origin xyz="${0.0015 + 0.05 - 0.01} ${-0.035/2} 0" rpy="0 0 0" />
             <parent link="arm_wrist_rotate_link"/>
@@ -216,9 +217,9 @@
         <transmission type="SimpleTransmission" name="arm_right_finger_trans">
             <actuator name="arm_right_finger_motor" />
-            <joint name="arm_wrist_rotate_right_finger_joint" />
+            <joint name="finger_right_joint" />
             <mechanicalReduction>1.0</mechanicalReduction>
         </transmission>
         <!-- Gripper left finger joint and link -->
-        <joint name="arm_wrist_rotate_left_finger_joint" type="revolute">
+        <joint name="finger_left_joint" type="revolute">
             <origin xyz="${0.0015 + 0.05 - 0.01} ${0.035/2} 0" rpy="0 0 0" />
             <parent link="arm_wrist_rotate_link"/>
@@ -254,5 +255,5 @@
         <transmission type="SimpleTransmission" name="arm_left_finger_trans">
             <actuator name="arm_left_finger_motor" />
-            <joint name="arm_wrist_rotate_left_finger_joint" />
+            <joint name="finger_left_joint" />
             <mechanicalReduction>1.0</mechanicalReduction>
         </transmission>
