Commit message: Move camera mount joint inside camera's urdf and pass in orging from calling urdf.

File: arrg/ua_robots/videre_stoc_description/urdf/videre_stoc.xacro (robot description, xacro)
@@ -27,6 +27,6 @@
                 <origin xyz="0 0 0" />
                 <inertia ixx="1.0" ixy="0.0" ixz="0.0"
-                         iyy="1.0" iyz="0.0" izz="1.0" />
-                <!-- Still don't know what that stuff means? -->
+                         iyy="1.0" iyz="0.0"
+                         izz="1.0" />
             </inertial>
             <visual>
@@ -100,15 +100,20 @@
         </gazebo>
     </macro>
-    <macro name="stoc_camera" params="name parent">
+    <macro name="stoc_camera" params="name parent *origin">
+        <joint name="camera_mount_joint" type="fixed">
+            <insert_block name="origin" />
+            <parent link="${parent}"/>
+            <child link="stoc_camera_link"/>
+        </joint>
         <link name="stoc_camera_link">
             <inertial>
                 <mass value="0.1" />
-                <origin xyz="${stoc_depth/2} ${stoc_width/2} ${stoc_height/2}" />
+                <origin xyz="0 0 ${stoc_height/2}" rpy="0 0 0" />
                 <inertia ixx="1.0" ixy="0.0" ixz="0.0"
-                         iyy="1.0" iyz="0.0" izz="1.0" />
-                <!-- Still don't know what that stuff means? -->
+                         iyy="1.0" iyz="0.0"
+                         izz="1.0" />
             </inertial>
             <visual>
-                <origin xyz="0 0 0.0215" rpy="0 0 0" />
+                <origin xyz="0 0 ${stoc_height/2}" rpy="0 0 0" />
                 <geometry>
                     <box size="${stoc_depth} ${stoc_width} ${stoc_height}" />
@@ -116,5 +121,5 @@
             </visual>
             <collision>
-                <origin xyz="0 0 0.0215" rpy="0 0 0" />
+                <origin xyz="0 0 ${stoc_height/2}" rpy="0 0 0" />
                 <geometry>
                     <box size="${stoc_depth} ${stoc_width} ${stoc_height}" />
@@ -134,5 +139,4 @@
                          iyy="1.0" iyz="0.0"
                          izz="1.0" />
-                <!-- Still don't know what that stuff means? -->
             </inertial>
             <visual>

File: arrg/ua_robots/wubble_description/urdf/wubble.urdf.xacro (robot description, xacro)
@@ -10,5 +10,4 @@
     <include filename="$(find videre_stoc_description)/urdf/videre_stoc.xacro" />
     <include filename="$(find pr2_defs)/calibration/default_cal.xml" />
-<!--    <include filename="$(find pr2_defs)/defs/materials.urdf.xacro" />    -->
     <!-- Properties (Constants) -->
     <property name="M_PI" value="3.14159"/>
@@ -146,10 +145,7 @@
         </collision>
     </link>
-    <joint name="head_mount_joint" type="fixed">
+    <stoc_camera name="stoc" parent="head_mount_link" >
         <origin xyz="0 0 0.023" rpy="0 0 0" />
-        <parent link="head_mount_link"/>
-        <child link="stoc_camera_link"/>
-    </joint>
-    <stoc_camera name="stoc" parent="head_mount_link" />
+    </stoc_camera>
     <!-- GAZEBO MATERIALS -->
     <gazebo reference="head_support_link">

Commit message: Move camera joints around a little.

File: arrg/ua_robots/videre_stoc_description/urdf/videre_stoc.xacro (robot description, xacro)
@@ -7,16 +7,16 @@
     <include filename="$(find pr2_defs)/calibration/default_cal.xml" />
     <property name="M_PI" value="3.14159"/>
-    <property name="stoc_depth" value="0.018" />
-    <property name="stoc_width" value="0.132" />
-    <property name="stoc_height" value="0.043" />
-    <property name="back_depth" value="0.022" />
-    <property name="back_width" value="0.069" />
-    <property name="back_height" value="0.043" />
-    <property name="eye_offset" value="0.048" />
-    <property name="eye_radius" value="0.006" />
+    <property name="stoc_depth" value="0.018542" />
+    <property name="stoc_width" value="0.13208" />
+    <property name="stoc_height" value="0.04318" />
+    <property name="back_depth" value="0.022225" />
+    <property name="back_width" value="0.0691134" />
+    <property name="back_height" value="0.04318" />
+    <property name="eye_radius" value="0.0072" />
     <property name="eye_length" value="0.010" />
+    <property name="eye_offset" value="0.045" />    <!-- 9cm baseline -->
     <macro name="stoc_eye" params="name parent suffix reflect">
         <joint name="${suffix}_stoc_eye_joint" type="fixed">
-            <origin xyz="${(stoc_depth/2)+(eye_length/2)} ${reflect*eye_offset} 0.03" rpy="0 ${M_PI/2} 0" />
+            <origin xyz="${stoc_depth/2} ${reflect*eye_offset} ${stoc_height/2}" rpy="0 ${M_PI/2} 0" />
             <parent link="${parent}" />
             <child link="${suffix}_stoc_eye_link"/>
@@ -24,6 +24,6 @@
         <link name="${suffix}_stoc_eye_link">
             <inertial>
-                <mass value="0.0001" />
-                <origin xyz="0 0 0" />
+                <mass value="0.01" />
+                <origin xyz="0 0 ${eye_length/2}" rpy="0 0 0" />
                 <inertia ixx="1.0" ixy="0.0" ixz="0.0"
                          iyy="1.0" iyz="0.0"
@@ -31,5 +31,5 @@
             </inertial>
             <visual>
-                <origin xyz="0 0 0" rpy="0 0 0" />
+                <origin xyz="0 0 ${eye_length/2}" rpy="0 0 0" />
                 <geometry>
                     <cylinder radius="${eye_radius}" length="${eye_length}" />
@@ -37,5 +37,5 @@
             </visual>
             <collision>
-                <origin xyz="0 0 0" rpy="0 0 0" />
+                <origin xyz="0 0 ${eye_length/2}" rpy="0 0 0" />
                 <geometry>
                     <cylinder radius="${eye_radius}" length="${eye_length}" />
@@ -128,5 +128,5 @@
         </link>
         <joint name="stoc_back_joint" type="fixed">
-            <origin xyz="${-(stoc_depth/2)-(back_depth/2)} 0 0.0215" rpy="0 0 0" />
+            <origin xyz="-${stoc_depth/2} 0 ${stoc_height/2}" rpy="0 0 0" />
             <parent link="stoc_camera_link" />
             <child link="stoc_back_link"/>
@@ -135,5 +135,5 @@
             <inertial>
                 <mass value="0.1" />
-                <origin xyz="${back_depth/2} ${back_width/2} ${back_height/2}" />
+                <origin xyz="-${back_depth/2} 0 0" />
                 <inertia ixx="1.0" ixy="0.0" ixz="0.0"
                          iyy="1.0" iyz="0.0"
@@ -141,5 +141,5 @@
             </inertial>
             <visual>
-                <origin xyz="0 0 0" rpy="0 0 0" />
+                <origin xyz="-${back_depth/2} 0 0" />
                 <geometry>
                     <box size="${back_depth} ${back_width} ${back_height}" />
@@ -147,5 +147,5 @@
             </visual>
             <collision>
-                <origin xyz="0 0 0" rpy="0 0 0" />
+                <origin xyz="-${back_depth/2} 0 0" />
                 <geometry>
                     <box size="${back_depth} ${back_width} ${back_height}" />
@@ -153,4 +153,5 @@
             </collision>
         </link>
+        <!-- MACRO INSTANTIATION -->
         <stoc_eye name="left_eye" parent="stoc_camera_link" suffix="left" reflect="1"/>
         <stoc_eye name="right_eye" parent="stoc_camera_link" suffix="right" reflect="-1"/>

Commit message: Fix stereo camera in simulation.

File: arrg/ua_robots/videre_stoc_description/urdf/videre_stoc.xacro (robot description, xacro)
@@ -4,6 +4,5 @@
     xmlns:controller="http://playerstage.sourceforge.net/gazebo/xmlschema/#controller"
     xmlns:interface="http://playerstage.sourceforge.net/gazebo/xmlschema/#interface">
-    <!-- Include file with calibration parameters -->
-    <include filename="$(find pr2_defs)/calibration/default_cal.xml" />
+    <include filename="$(find pr2_description)/urdf/sensors/stereo_camera.urdf.xacro" />
     <property name="M_PI" value="3.14159"/>
     <property name="stoc_depth" value="0.018542" />
@@ -16,11 +15,11 @@
     <property name="eye_length" value="0.010" />
     <property name="eye_offset" value="0.045" />    <!-- 9cm baseline -->
-    <macro name="stoc_eye" params="name parent suffix reflect">
-        <joint name="${suffix}_stoc_eye_joint" type="fixed">
+    <macro name="stoc_eye" params="name parent reflect">
+        <joint name="${name}_stoc_eye_joint" type="fixed">
             <origin xyz="${stoc_depth/2} ${reflect*eye_offset} ${stoc_height/2}" rpy="0 ${M_PI/2} 0" />
             <parent link="${parent}" />
-            <child link="${suffix}_stoc_eye_link"/>
+            <child link="${name}_stoc_eye_link"/>
         </joint>
-        <link name="${suffix}_stoc_eye_link">
+        <link name="${name}_stoc_eye_link">
             <inertial>
                 <mass value="0.01" />
@@ -43,10 +42,10 @@
             </collision>
         </link>
-        <joint name="${suffix}_stoc_eye_frame_joint" type="fixed">
+        <joint name="${name}_stoc_eye_frame_joint" type="fixed">
             <origin xyz="0 0 0" rpy="0 ${-M_PI/2} 0" />
-            <parent link="${suffix}_stoc_eye_link" />
-            <child link="${suffix}_stoc_eye_frame"/>
+            <parent link="${name}_stoc_eye_link" />
+            <child link="${name}_stoc_eye_frame"/>
         </joint>
-        <link name="${suffix}_stoc_eye_frame">
+        <link name="${name}_stoc_eye_frame">
             <inertial>
                 <mass value="0.0001" />
@@ -54,5 +53,4 @@
                 <inertia ixx="1.0" ixy="0.0" ixz="0.0"
                          iyy="1.0" iyz="0.0" izz="1.0" />
-                <!-- Still don't know what that stuff means? -->
             </inertial>
             <visual>
@@ -69,33 +67,6 @@
             </collision>
         </link>
-        <gazebo reference="${suffix}_stoc_eye_link">
+        <gazebo reference="${name}_stoc_eye_link">
             <material>Gazebo/Black</material>
-        </gazebo>
-        <gazebo reference="${suffix}_stoc_eye_frame">
-            <sensor:camera name="${suffix}_eye_sensor">
-                <imageSize>640 480</imageSize>
-                <imageFormat>BAYER_BGGR8</imageFormat>
-                <hfov>90</hfov>
-                <nearClip>0.1</nearClip>
-                <farClip>100</farClip>
-                <updateRate>30.0</updateRate>
-                <controller:gazebo_ros_camera name="${suffix}_eye_controller" plugin="libgazebo_ros_camera.so">
-                    <alwaysOn>true</alwaysOn>
-                    <updateRate>30.0</updateRate>
-                    <imageTopicName>stereo/${suffix}/image_raw</imageTopicName>
-                    <cameraInfoTopicName>stereo/${suffix}/camera_info</cameraInfoTopicName>
-                    <frameName>${suffix}_stoc_eye_frame</frameName>
-                    <CxPrime>320.5</CxPrime>
-                    <Cx>320.5</Cx>
-                    <Cy>240.5</Cy>
-                    <focal_length>320</focal_length>
-                    <distortion_k1>0</distortion_k1>
-                    <distortion_k2>0</distortion_k2>
-                    <distortion_k3>0</distortion_k3>
-                    <distortion_t1>0</distortion_t1>
-                    <distortion_t2>0</distortion_t2>
-                    <interface:camera name="${suffix}_eye_iface" />
-                </controller:gazebo_ros_camera>
-            </sensor:camera>
         </gazebo>
     </macro>
@@ -154,38 +125,9 @@
         </link>
         <!-- MACRO INSTANTIATION -->
-        <stoc_eye name="left_eye" parent="stoc_camera_link" suffix="left" reflect="1"/>
-        <stoc_eye name="right_eye" parent="stoc_camera_link" suffix="right" reflect="-1"/>
-        <joint name="stoc_optical_frame_joint" type="fixed">
-            <origin xyz="${cal_stereo_x}  ${0.045+cal_stereo_y}  ${.0305+cal_stereo_z+0.03}"
-                    rpy="${-M_PI/2+cal_stereo_roll} ${0.0+cal_stereo_pitch} ${-M_PI/2+cal_stereo_yaw}" />
-            <parent link="stoc_camera_link"/>
-            <child link="stoc_optical_frame"/>
-        </joint>
-        <link name="stoc_optical_frame" type="camera">
-            <inertial>
-                <mass value="0.01" />
-                <origin xyz="0 0 0" rpy="0 0 0" />
-                <inertia ixx="0.001"  ixy="0.0"  ixz="0.0"
-                         iyy="0.001"  iyz="0.0"
-                         izz="0.001" />
-            </inertial>
-            <visual name="stoc_optical_frame_visual">
-                <origin xyz="0 0 0" rpy="0 0 0" />
-                <geometry name="stoc_optical_frame_visual_geom">
-                    <box size="0.01 0.01 0.01" />
-                </geometry>
-            </visual>
-            <collision name="stoc_optical_frame_collision">
-                <origin xyz="0 0 0" rpy="0 0 0" />
-                <geometry name="stoc_optical_frame_collision_geom">
-                    <box size="0.01 0.01 0.01" />
-                </geometry>
-            </collision>
-        </link>
-        <gazebo reference="stoc_optical_frame" >
-            <material name="clearish">
-                <color rgba="0 0 1 0.5"/>
-            </material>
-        </gazebo>
+        <stoc_eye name="left" parent="stoc_camera_link" reflect="1"/>
+        <stoc_eye name="right" parent="stoc_camera_link" reflect="-1"/>
+        <stereo_camera_v0 parent="left_stoc_eye_link" name="stereo" focal_length="772.55" hfov="45" image_format="BAYER_BGGR8" image_width="640" image_height="480" >
+            <origin xyz="0 0 0" rpy="0 -${M_PI/2} 0" />
+        </stereo_camera_v0>
         <gazebo reference="stoc_camera_link" >
             <material>PR2/Red</material>

Commit message: Move in all stereo related urdf files and modify params to match our camera and installed lenses.

File: arrg/ua_robots/videre_stoc_description/urdf/videre_stoc.xacro (robot description, xacro)
@@ -4,13 +4,13 @@
     xmlns:controller="http://playerstage.sourceforge.net/gazebo/xmlschema/#controller"
     xmlns:interface="http://playerstage.sourceforge.net/gazebo/xmlschema/#interface">
-    <include filename="$(find pr2_description)/urdf/sensors/stereo_camera.urdf.xacro" />
+    <include filename="$(find videre_stoc_description)/urdf/stereo_camera.urdf.xacro" />
     <property name="M_PI" value="3.14159"/>
-    <property name="stoc_depth" value="0.018542" />
-    <property name="stoc_width" value="0.13208" />
-    <property name="stoc_height" value="0.04318" />
-    <property name="back_depth" value="0.022225" />
-    <property name="back_width" value="0.0691134" />
-    <property name="back_height" value="0.04318" />
-    <property name="eye_radius" value="0.0072" />
+    <property name="stoc_depth"  value="0.019" />
+    <property name="stoc_width"  value="0.132" />
+    <property name="stoc_height" value="0.043" />
+    <property name="back_depth"  value="0.022" />
+    <property name="back_width"  value="0.069" />
+    <property name="back_height" value="0.043" />
+    <property name="eye_radius" value="0.006" />
     <property name="eye_length" value="0.010" />
     <property name="eye_offset" value="0.045" />    <!-- 9cm baseline -->
@@ -23,5 +23,5 @@
         <link name="${name}_stoc_eye_link">
             <inertial>
-                <mass value="0.01" />
+                <mass value="0.004" />
                 <origin xyz="0 0 ${eye_length/2}" rpy="0 0 0" />
                 <inertia ixx="1.0" ixy="0.0" ixz="0.0"
@@ -127,7 +127,9 @@
         <stoc_eye name="left" parent="stoc_camera_link" reflect="1"/>
         <stoc_eye name="right" parent="stoc_camera_link" reflect="-1"/>
-        <stereo_camera_v0 parent="left_stoc_eye_link" name="stereo" focal_length="772.55" hfov="45" image_format="BAYER_BGGR8" image_width="640" image_height="480" >
-            <origin xyz="0 0 0" rpy="0 -${M_PI/2} 0" />
-        </stereo_camera_v0>
+        <stereo_camera_9cm_baseline parent="left_stoc_eye_link" name="stereo"
+                                    focal_length="698.94" hfov="49.2" image_format="BAYER_BGGR8"
+                                    image_width="640" image_height="480" >
+            <origin xyz="0 0 -0.0042" rpy="0 -${M_PI/2} 0" />
+        </stereo_camera_9cm_baseline>
         <gazebo reference="stoc_camera_link" >
             <material>PR2/Red</material>
