Commit message: Little tweaks to size of camera frames, so they don't stick out of the camera.

File: arrg/ua_robots/videre_stoc_description/urdf/stereo_camera.urdf.xacro (robot description, xacro)
@@ -23,5 +23,5 @@
         <link name="${name}_link">
             <inertial>
-                <mass value="0.001" />
+                <mass value="0.0001" />
                 <origin xyz="0 0 0" rpy="0 0 0" />
                 <inertia ixx="0.01"  ixy="0"  ixz="0"
@@ -32,5 +32,5 @@
                 <origin xyz="0 0 0" rpy="0 0 0" />
                 <geometry>
-                    <box size="0.001 0.001 0.001" />
+                    <box size="0.0001 0.0001 0.0001" />
                 </geometry>
                 <material name="Blue" />
@@ -39,5 +39,5 @@
                 <origin xyz="0 0 0" rpy="0 0 0" />
                 <geometry>
-                    <box size="0.001 0.001 0.001" />
+                    <box size="0.0001 0.0001 0.0001" />
                 </geometry>
             </collision>

File: arrg/ua_robots/videre_stoc_description/urdf/videre_stoc.xacro (robot description, xacro)
@@ -130,5 +130,5 @@
                                     focal_length="698.94" hfov="49.2" image_format="BAYER_BGGR8"
                                     image_width="640" image_height="480" >
-            <origin xyz="0 0 -0.0042" rpy="0 -${M_PI/2} 0" />
+            <origin xyz="0 0 -0.0058" rpy="0 -${M_PI/2} 0" />
         </stereo_camera_9cm_baseline>
         <gazebo reference="stoc_camera_link" >

File: arrg/ua_robots/videre_stoc_description/urdf/videre_stoc_camera.urdf.xacro (robot description, xacro)
@@ -25,5 +25,5 @@
                 <origin xyz="0 0 0" rpy="0 0 0" />
                 <geometry>
-                    <box size="0.01 0.01 0.01" />
+                    <box size="0.001 0.001 0.001" />
                 </geometry>
             </visual>
@@ -31,5 +31,5 @@
                 <origin xyz="0 0 0" rpy="0 0 0"/>
                 <geometry>
-                    <box size="0.01 0.01 0.01" />
+                    <box size="0.001 0.001 0.001" />
                 </geometry>
             </collision>

Commit message: Add 6cm baseline stereo camera urdf.

File: arrg/ua_robots/videre_stoc_description/urdf/stereo_camera.urdf.xacro (robot description, xacro)
@@ -8,5 +8,4 @@
     <include filename="$(find videre_stoc_description)/urdf/stereo_camera.gazebo.xacro" />
     <property name="stereo_dx" value="0.00" />
-    <property name="stereo_dy" value="-0.09" /> <!-- +y to the left -->
     <property name="stereo_dz" value="0.00" />
     <property name="stereo_rx" value="0.00" />
@@ -14,5 +13,5 @@
     <property name="stereo_rz" value="0.00" />
     <!-- this macro is used for creating wide and narrow double stereo camera links -->
-    <xacro:macro name="stereo_camera_9cm_baseline" params="name parent focal_length hfov image_format image_width image_height *origin">
+    <xacro:macro name="stereo_camera" params="name parent stereo_dy focal_length hfov image_format image_width image_height *origin">
         <joint name="${name}_frame_joint" type="fixed">
             <insert_block name="origin" />
@@ -63,7 +62,7 @@
                                   camera_info_topic_name="${name}/right/camera_info" parent="${name}_gazebo_l_stereo_camera_frame"
                                   hfov="${hfov}" focal_length="${focal_length}"
-                                  frame_id="${name}_optical_frame" hack_baseline="${-stereo_dy}"
+                                  frame_id="${name}_optical_frame" hack_baseline="${stereo_dy}"
                                   image_width="${image_width}" image_height="${image_height}">
-            <origin xyz="${stereo_dx} ${stereo_dy} ${stereo_dz}" rpy="${stereo_rx} ${stereo_ry} ${stereo_rz}" />
+            <origin xyz="${stereo_dx} ${-stereo_dy} ${stereo_dz}" rpy="${stereo_rx} ${stereo_ry} ${stereo_rz}" />
         </xacro:videre_stoc_camera>
         <!-- extensions -->

File: arrg/ua_robots/videre_stoc_description/urdf/videre_stereo_9cm.xacro (robot description, xacro)
@@ -71,5 +71,5 @@
         </gazebo>
     </macro>
-    <macro name="stoc_camera" params="name parent *origin">
+    <macro name="videre_stereo_9cm" params="name parent *origin">
         <joint name="camera_mount_joint" type="fixed">
             <insert_block name="origin" />
@@ -127,9 +127,10 @@
         <stoc_eye name="left" parent="stoc_camera_link" reflect="1"/>
         <stoc_eye name="right" parent="stoc_camera_link" reflect="-1"/>
-        <stereo_camera_9cm_baseline parent="left_stoc_eye_link" name="stereo"
-                                    focal_length="698.94" hfov="49.2" image_format="BAYER_BGGR8"
-                                    image_width="640" image_height="480" >
+        <!-- stereo_dy parameter is the stereo camera baseline -->
+        <stereo_camera parent="left_stoc_eye_link" name="stereo"
+                       stereo_dy="${eye_offset*2}" focal_length="698.94" hfov="49.2"
+                       image_format="BAYER_BGGR8" image_width="640" image_height="480" >
             <origin xyz="0 0 -0.0058" rpy="0 -${M_PI/2} 0" />
-        </stereo_camera_9cm_baseline>
+        </stereo_camera>
         <gazebo reference="stoc_camera_link" >
             <material>Erratic/Red</material>

File: arrg/ua_robots/wubble_description/urdf/wubble.urdf.xacro (robot description, xacro)
@@ -8,5 +8,5 @@
     <include filename="$(find smart_arm_description)/urdf/smart_arm.xacro" />
     <include filename="$(find hokuyo_urg_description)/urdf/hokuyo_urg.xacro" />
-    <include filename="$(find videre_stoc_description)/urdf/videre_stoc.xacro" />
+    <include filename="$(find videre_stoc_description)/urdf/videre_stereo_6cm.xacro" />
     <include filename="$(find chr_6dm_imu_description)/urdf/chrobotics_chr_6dm_imu.urdf.xacro" />
     <!-- Properties (Constants) -->
@@ -212,7 +212,7 @@
         </collision>
     </link>
-    <stoc_camera name="stoc" parent="head_mount_link" >
+    <videre_stereo_6cm name="stoc" parent="head_mount_link" >
         <origin xyz="0 0 0.023" rpy="0 0 0" />
-    </stoc_camera>
+    </videre_stereo_6cm>
     <!-- GAZEBO MATERIALS -->
     <gazebo reference="head_support_link">
