Commit message: Fixed dependencies of wubble_mapping, changed laser so by default it sits still

File: arrg/ua_robots/hokuyo_urg_description/urdf/tilting_hokuyo.xacro (robot description, xacro)
@@ -10,8 +10,8 @@
             <axis xyz="0 1 0" />
 <!--           Original effort: 0.5292-->
-            <limit lower="0.00" upper="${M_PI/3}" effort="2.0" velocity="4.0" />
-<!--            <safety_controller k_position="100" k_velocity="0.05" soft_lower_limit="${-0.785+0.0}" soft_upper_limit="${1.57-0.0}" />-->
+            <limit lower="-0.1" upper="${M_PI/2}" effort="100" velocity="4" />
+            <safety_controller k_position="100" k_velocity="4" soft_lower_limit="${-0.1+0.1}" soft_upper_limit="${M_PI/3}" />-->
 <!--            <calibration reference_position="${laser_calib_ref}" falling="${laser_calib_ref}" />-->
-            <dynamics damping="0.008" />
+            <dynamics damping="50" friction="1" />
             <insert_block name="origin" />
         </joint>
@@ -21,5 +21,5 @@
             <actuator name="hokuyo_tilt_motor" />
             <joint name="hokuyo_tilt_joint" />
-            <mechanicalReduction>6.0</mechanicalReduction>
+            <mechanicalReduction>1.0</mechanicalReduction>
         </transmission>
     </macro>
