Commit message: Add meshes to laser tilting motor. Change controller to position controller until we figure out how to use trajectory controller.

File: arrg/ua_robots/hokuyo_urg_description/urdf/hokuyo_urg.xacro (robot description, xacro)
@@ -3,5 +3,10 @@
        xmlns:controller="http://playerstage.sourceforge.net/gazebo/xmlschema/#controller"
        xmlns:interface="http://playerstage.sourceforge.net/gazebo/xmlschema/#interface">
-    <macro name="hokuyo_urg">
+    <macro name="hokuyo_urg" params="parent *origin" >
+        <joint name="hokuyo_mount_joint" type="fixed">
+            <insert_block name="origin" />
+            <parent link="${parent}"/>
+            <child link="hokuyo_link"/>
+        </joint>
         <link name="hokuyo_link">
             <inertial>

File: arrg/ua_robots/wubble_description/urdf/wubble.urdf.xacro (robot description, xacro)
@@ -14,12 +14,76 @@
     <property name="support_radius" value="0.0065" />
     <property name="support_height" value="0.7556" />
-    <!-- MACRO INSTANTIATION -->
+    <!-- VIDERE ERRATIC MOBILE BASE -->
     <erratic />
+    <!-- CRUST CRAWLER SMART ARM ATTACHMENT -->
     <smart_arm parent="base_top_link" >
         <origin xyz="${top_size_x/2 - 0.0575} 0 ${top_size_z/2 + 0.025}"/>
     </smart_arm>
-    <tilting_hokuyo parent="base_top_link">
-        <origin xyz="0.15 0 ${-top_size_z - 0.05}" rpy="${M_PI} 0 0" />
-    </tilting_hokuyo>
+    <!-- HOKUYO LASER ATTACHMENT -->
+    <joint name="laser_support_joint" type="fixed">
+        <origin xyz="${top_size_x/2 - 0.016} 0 -${top_size_z/2}" rpy="${M_PI} 0 0" />
+        <parent link="base_top_link"/>
+        <child link="hokuyo_tilt_link"/>
+    </joint>
+    <link name="hokuyo_tilt_link">
+        <inertial>
+            <mass value="0.1"/>
+            <origin xyz="0 0 0" rpy="0 0 0" />
+            <inertia ixx="0.01" ixy="0" ixz="0"
+                     iyy="0.01" iyz="0"
+                     izz="0.01"/>
+        </inertial>
+        <visual>
+            <origin xyz="0 0 0" rpy="0 0 0"/>
+            <geometry>
+                <mesh filename="package://wubble_description/meshes/camera_tilt.stl"/>
+            </geometry>
+        </visual>
+        <collision>
+            <origin xyz="0 0 0" rpy="0 0 0"/>
+            <geometry>
+                <mesh filename="package://wubble_description/meshes/camera_tilt.stl"/>
+            </geometry>
+        </collision>
+    </link>
+    <joint name="hokuyo_tilt_joint" type="revolute">
+        <origin xyz="-0.019 0 0.043" />
+        <parent link="hokuyo_tilt_link" />
+        <child link="hokuyo_mount_link" />
+        <axis xyz="0 1 0" />
+        <limit lower="-0.1" upper="${M_PI/2}" effort="100" velocity="12.0" />
+        <safety_controller k_position="100" k_velocity="12.0" soft_lower_limit="${-0.1+0.1}" soft_upper_limit="${M_PI/3}" />-->
+        <dynamics damping="50" friction="1"/>
+    </joint>
+    <transmission type="SimpleTransmission" name="hokuyo_tilt_trans">
+        <actuator name="hokuyo_tilt_motor" />
+        <joint name="hokuyo_tilt_joint" />
+        <mechanicalReduction>1.0</mechanicalReduction>
+    </transmission>
+    <link name="hokuyo_mount_link">
+        <inertial>
+            <mass value="0.01"/>
+            <origin xyz="0 0 0" rpy="0 0 0" />
+            <inertia ixx="0.01" ixy="0" ixz="0"
+                     iyy="0.01" iyz="0"
+                     izz="0.01"/>
+        </inertial>
+        <visual>
+            <origin xyz="0 0 0" rpy="0 0 0"/>
+            <geometry>
+                <mesh filename="package://wubble_description/meshes/camera_mount.stl"/>
+            </geometry>
+        </visual>
+        <collision>
+            <origin xyz="0 0 0" rpy="0 0 0"/>
+            <geometry>
+                <mesh filename="package://wubble_description/meshes/camera_mount.stl"/>
+            </geometry>
+        </collision>
+    </link>
+    <hokuyo_urg parent="hokuyo_mount_link">
+        <origin xyz="0 0 0.023" rpy="0 0 0" />
+    </hokuyo_urg>
+    <!-- VIDERE STOC STEREO CAMERA ATTACHMENT -->
     <joint name="head_support_joint" type="fixed">
         <origin xyz="${top_size_x/2 - 0.16} 0 ${top_size_z/2}" />
@@ -160,3 +224,9 @@
         <material>PR2/White</material>
     </gazebo>
+    <gazebo reference="hokuyo_tilt_link">
+        <material>PR2/Black</material>
+    </gazebo>
+    <gazebo reference="hokuyo_mount_link">
+        <material>SmartArm/GunMetalBrushedAluminum</material>
+    </gazebo>
 </robot>

Commit message: More launch file reorg.

File: arrg/ua_robots/hokuyo_urg_description/urdf/hokuyo_urg.xacro (robot description, xacro)
@@ -58,5 +58,5 @@
         </link>
         <gazebo reference="hokuyo_link">
-            <material value="PR2/Black" />
+            <material value="Erratic/Black" />
         </gazebo>
         <gazebo reference="hokuyo_link">

File: arrg/ua_robots/videre_stoc_description/urdf/videre_stoc.xacro (robot description, xacro)
@@ -133,8 +133,8 @@
         </stereo_camera_9cm_baseline>
         <gazebo reference="stoc_camera_link" >
-            <material>PR2/Red</material>
+            <material>Erratic/Red</material>
         </gazebo>
         <gazebo reference="stoc_back_link" >
-            <material>PR2/Red</material>
+            <material>Erratic/Red</material>
         </gazebo>
     </macro>

File: arrg/ua_robots/wubble_description/urdf/wubble_base.urdf.xacro (robot description, xacro)
@@ -80,5 +80,5 @@
     <!-- GAZEBO MATERIALS -->
     <gazebo reference="hokuyo_tilt_link">
-        <material>PR2/Black</material>
+        <material>Erratic/Black</material>
     </gazebo>
     <gazebo reference="hokuyo_mount_link">

Commit message: Add stereo camera with pan tilt and neck laser on tilting base to new wubble urdf. Modify how laser xacro works, need to provide a unique name now to be able to have multiple lasers on the robot.

File: arrg/ua_robots/hokuyo_urg_description/urdf/hokuyo_urg.xacro (robot description, xacro)
@@ -3,11 +3,11 @@
        xmlns:controller="http://playerstage.sourceforge.net/gazebo/xmlschema/#controller"
        xmlns:interface="http://playerstage.sourceforge.net/gazebo/xmlschema/#interface">
-    <macro name="hokuyo_urg" params="parent *origin" >
-        <joint name="hokuyo_mount_joint" type="fixed">
+    <macro name="hokuyo_urg" params="name parent *origin" >
+        <joint name="${name}_mount_joint" type="fixed">
             <insert_block name="origin" />
             <parent link="${parent}"/>
-            <child link="hokuyo_link"/>
+            <child link="${name}_mount_link"/>
         </joint>
-        <link name="hokuyo_link">
+        <link name="${name}_mount_link">
             <inertial>
                 <mass value="0.160" />
@@ -30,10 +30,10 @@
             </collision>
         </link>
-        <joint name="laser_joint" type="fixed">
+        <joint name="${name}_joint" type="fixed">
             <origin xyz="0 0 0.06" rpy="0 0 0" />
-            <parent link="hokuyo_link" />
-            <child link="laser_link" />
+            <parent link="${name}_mount_link" />
+            <child link="${name}_link" />
         </joint>
-        <link name="laser_link" type="laser">
+        <link name="${name}_link" type="laser">
             <inertial>
                 <mass value="0.001" />
@@ -57,8 +57,11 @@
             </collision>
         </link>
-        <gazebo reference="hokuyo_link">
+        <gazebo reference="${name}_mount_link">
             <material value="Erratic/Black" />
         </gazebo>
-        <gazebo reference="hokuyo_link">
+        <gazebo reference="${name}_link">
+            <material value="Erratic/Black" />
+        </gazebo>
+        <gazebo reference="${name}_link">
             <sensor:ray name="laser">
                 <rayCount>683</rayCount>
@@ -73,12 +76,12 @@
                 <resRange>0.001</resRange>
                 <updateRate>10.0</updateRate>
-                <controller:gazebo_ros_laser name="gazebo_ros_laser_controller" plugin="libgazebo_ros_laser.so">
+                <controller:gazebo_ros_laser name="gazebo_ros_${name}_laser_controller" plugin="libgazebo_ros_laser.so">
                     <gaussianNoise>0.005</gaussianNoise>
                     <alwaysOn>true</alwaysOn>
                     <updateRate>10.0</updateRate>
-                    <topicName>tilt_laser/scan</topicName>
-                    <deprecatedTopicName>tilt_scan</deprecatedTopicName>
-                    <frameName>laser_link</frameName>
-                    <interface:laser name="gazebo_ros_laser_iface" />
+                    <topicName>${name}/scan</topicName>
+                    <deprecatedTopicName>${name}_scan</deprecatedTopicName>
+                    <frameName>${name}_link</frameName>
+                    <interface:laser name="gazebo_ros_${name}_laser_iface" />
                 </controller:gazebo_ros_laser>
             </sensor:ray>

File: arrg/ua_robots/wubble_description/urdf/wubble.urdf.xacro (robot description, xacro)
@@ -86,5 +86,5 @@
         </collision>
     </link>
-    <hokuyo_urg parent="hokuyo_mount_link">
+    <hokuyo_urg name="tilt_laser" parent="hokuyo_mount_link">
         <origin xyz="0 0 0.023" rpy="0 0 0" />
     </hokuyo_urg>

File: arrg/ua_robots/wubble_description/urdf/wubble2.urdf.xacro (robot description, xacro)
@@ -8,4 +8,5 @@
     <include filename="$(find hokuyo_urg_description)/urdf/hokuyo_urg.xacro" />
     <include filename="$(find wubble_arm_description)/urdf/wubble_arm.xacro" />
+    <include filename="$(find videre_stoc_description)/urdf/videre_stereo_6cm.xacro" />
     <!-- Properties (Constants) -->
     <property name="M_PI" value="3.14159"/>
@@ -39,8 +40,174 @@
         </collision>
     </link>
+    <!-- WUBBLE HEAD ATTACHMENT -->
+    <joint name="head_base_joint" type="fixed">
+        <origin xyz="0.0254 0 0.8001" rpy="0 0 0" />
+        <parent link="platform_link"/>
+        <child link="head_base_link"/>
+    </joint>
+    <joint name="head_pan_joint" type="revolute">
+        <origin xyz="0.0415 0 0.004" rpy="0 0 0" />
+        <parent link="head_base_link"/>
+        <child link="head_pan_link"/>
+        <axis xyz="0 0 1" />
+        <limit lower="-1.57" upper="1.57" effort="100" velocity="12.0" />
+        <safety_controller k_position="100" k_velocity="15.0" soft_lower_limit="${-1.57}" soft_upper_limit="${1.57}" />
+        <dynamics damping="50" friction="1"/>
+    </joint>
+    <joint name="head_tilt_joint" type="revolute">
+        <origin xyz="0 0 0.0415" rpy="0 0 0" />
+        <parent link="head_pan_link"/>
+        <child link="head_tilt_link"/>
+        <axis xyz="0 1 0" />
+        <limit lower="-1.57" upper="1.57" effort="100" velocity="12.0" />
+        <safety_controller k_position="100" k_velocity="15.0" soft_lower_limit="${-1.57}" soft_upper_limit="${1.57}" />
+        <dynamics damping="50" friction="1"/>
+    </joint>
+    <link name="head_base_link">
+        <inertial>
+            <mass value="0.05"/>
+            <origin xyz="0 0 0" rpy="0 0 0" />
+            <inertia ixx="0.1" ixy="0" ixz="0"
+                     iyy="0.1" iyz="0"
+                     izz="0.1"/>
+        </inertial>
+        <visual>
+            <origin xyz="0 0 0" rpy="0 0 0"/>
+            <geometry>
+                <mesh filename="package://wubble_description/meshes/head_base_link.stl"/>
+            </geometry>
+        </visual>
+        <collision>
+            <origin xyz="0 0 0" rpy="0 0 0"/>
+            <geometry>
+                <mesh filename="package://wubble_description/meshes/head_base_link.stl"/>
+            </geometry>
+        </collision>
+    </link>
+    <link name="head_pan_link">
+        <inertial>
+            <mass value="0.05"/>
+            <origin xyz="0 0 0" rpy="0 0 0" />
+            <inertia ixx="0.1" ixy="0" ixz="0"
+                     iyy="0.1" iyz="0"
+                     izz="0.1"/>
+        </inertial>
+        <visual>
+            <origin xyz="0 0 0" rpy="0 0 0"/>
+            <geometry>
+                <mesh filename="package://wubble_description/meshes/head_pan_link.stl"/>
+            </geometry>
+        </visual>
+        <collision>
+            <origin xyz="0 0 0" rpy="0 0 0"/>
+            <geometry>
+                <mesh filename="package://wubble_description/meshes/head_pan_link.stl"/>
+            </geometry>
+        </collision>
+    </link>
+    <link name="head_tilt_link">
+        <inertial>
+            <mass value="0.05"/>
+            <origin xyz="0 0 0" rpy="0 0 0" />
+            <inertia ixx="0.1" ixy="0" ixz="0"
+                     iyy="0.1" iyz="0"
+                     izz="0.1"/>
+        </inertial>
+        <visual>
+            <origin xyz="0 0 0" rpy="0 0 0"/>
+            <geometry>
+                <mesh filename="package://wubble_description/meshes/head_tilt_link.stl"/>
+            </geometry>
+        </visual>
+        <collision>
+            <origin xyz="0 0 0" rpy="0 0 0"/>
+            <geometry>
+                <mesh filename="package://wubble_description/meshes/head_tilt_link.stl"/>
+            </geometry>
+        </collision>
+    </link>
+    <transmission type="pr2_mechanism_model/SimpleTransmission" name="head_pan_trans">
+        <actuator name="head_pan_motor" />
+        <joint name="head_pan_joint" />
+        <mechanicalReduction>1.0</mechanicalReduction>
+    </transmission>
+    <transmission type="pr2_mechanism_model/SimpleTransmission" name="head_tilt_trans">
+        <actuator name="head_tilt_motor" />
+        <joint name="head_tilt_joint" />
+        <mechanicalReduction>1.0</mechanicalReduction>
+    </transmission>
+    <!-- VIDERE STEREO CAMERA ATTACHMENT -->
+    <videre_stereo_6cm name="stoc" parent="head_tilt_link" >
+        <origin xyz="0.01148 0 0.02635" rpy="0 0 0" />
+    </videre_stereo_6cm>
     <!-- WUBBLE ARM ATTACHMENT -->
     <wubble_arm parent="base_top_link" >
         <origin xyz="0.16281 0.0825 ${top_size_z/2 + 0.109}" rpy="0 0 0"/>
     </wubble_arm>
+    <!-- NECK TILTING LASER ATTACHMENT -->
+    <joint name="neck_support_joint" type="fixed">
+        <origin xyz="0.0254 0 0.6001" rpy="0 0 0" />
+        <parent link="platform_link"/>
+        <child link="neck_support_link"/>
+    </joint>
+    <joint name="neck_tilt_joint" type="revolute">
+        <origin xyz="0.0415 0 0.016" rpy="0 0 0" />
+        <parent link="neck_support_link"/>
+        <child link="neck_tilt_link"/>
+        <axis xyz="0 1 0" />
+        <limit lower="0" upper="1.57" effort="100" velocity="12.0" />
+        <safety_controller k_position="100" k_velocity="15.0" soft_lower_limit="${0}" soft_upper_limit="${1.57}" />
+        <dynamics damping="50" friction="1"/>
+    </joint>
+    <link name="neck_support_link">
+        <inertial>
+            <mass value="0.05"/>
+            <origin xyz="0 0 0" rpy="0 0 0" />
+            <inertia ixx="0.1" ixy="0" ixz="0"
+                     iyy="0.1" iyz="0"
+                     izz="0.1"/>
+        </inertial>
+        <visual>
+            <origin xyz="0 0 0" rpy="0 0 0"/>
+            <geometry>
+                <mesh filename="package://wubble_description/meshes/neck_laser_support_link.stl"/>
+            </geometry>
+        </visual>
+        <collision>
+            <origin xyz="0 0 0" rpy="0 0 0"/>
+            <geometry>
+                <mesh filename="package://wubble_description/meshes/neck_laser_support_link.stl"/>
+            </geometry>
+        </collision>
+    </link>
+    <link name="neck_tilt_link">
+        <inertial>
+            <mass value="0.05"/>
+            <origin xyz="0 0 0" rpy="0 0 0" />
+            <inertia ixx="0.1" ixy="0" ixz="0"
+                     iyy="0.1" iyz="0"
+                     izz="0.1"/>
+        </inertial>
+        <visual>
+            <origin xyz="0 0 0" rpy="0 0 0"/>
+            <geometry>
+                <mesh filename="package://wubble_description/meshes/head_tilt_link.stl"/>
+            </geometry>
+        </visual>
+        <collision>
+            <origin xyz="0 0 0" rpy="0 0 0"/>
+            <geometry>
+                <mesh filename="package://wubble_description/meshes/head_tilt_link.stl"/>
+            </geometry>
+        </collision>
+    </link>
+    <transmission type="pr2_mechanism_model/SimpleTransmission" name="neck_tilt_trans">
+        <actuator name="neck_tilt_motor" />
+        <joint name="neck_tilt_joint" />
+        <mechanicalReduction>1.0</mechanicalReduction>
+    </transmission>
+    <hokuyo_urg name="neck_scan" parent="neck_tilt_link">
+        <origin xyz="0.01148 0 0.02635" rpy="0 0 0" />
+    </hokuyo_urg>
     <!-- HOKUYO LASER ATTACHMENT -->
     <joint name="laser_support_joint" type="fixed">
@@ -105,8 +272,23 @@
         </collision>
     </link>
-    <hokuyo_urg parent="hokuyo_mount_link">
+    <hokuyo_urg name="base_scan" parent="hokuyo_mount_link">
         <origin xyz="0 0 0.023" rpy="0 0 0" />
     </hokuyo_urg>
     <!-- GAZEBO MATERIALS -->
+    <gazebo reference="head_base_link">
+        <material>SmartArm/GunMetalBrushedAluminum</material>
+    </gazebo>
+    <gazebo reference="head_pan_link">
+        <material>SmartArm/GunMetalBrushedAluminum</material>
+    </gazebo>
+    <gazebo reference="head_tilt_link">
+        <material>SmartArm/GunMetalBrushedAluminum</material>
+    </gazebo>
+    <gazebo reference="neck_support_link">
+        <material>SmartArm/GunMetalBrushedAluminum</material>
+    </gazebo>
+    <gazebo reference="neck_tilt_link">
+        <material>SmartArm/GunMetalBrushedAluminum</material>
+    </gazebo>
     <gazebo reference="hokuyo_tilt_link">
         <material>Erratic/Black</material>

Commit message: Added navigation and laser filters for Wubble2.

File: arrg/ua_robots/hokuyo_urg_description/urdf/hokuyo_urg.xacro (robot description, xacro)
@@ -81,5 +81,4 @@
                     <updateRate>10.0</updateRate>
                     <topicName>${name}/scan</topicName>
-                    <deprecatedTopicName>${name}_scan</deprecatedTopicName>
                     <frameName>${name}_link</frameName>
                     <interface:laser name="gazebo_ros_${name}_laser_iface" />

File: arrg/ua_robots/wubble_description/urdf/wubble2.urdf.xacro (robot description, xacro)
@@ -242,6 +242,6 @@
         <child link="hokuyo_mount_link" />
         <axis xyz="0 1 0" />
-        <limit lower="-0.1" upper="0.785398164" effort="100" velocity="12.0" />
-        <safety_controller k_position="100" k_velocity="15.0" soft_lower_limit="${-0.1+0.1}" soft_upper_limit="${0.785398164-0.1}" />
+        <limit lower="-0.6" upper="0.785398164" effort="100" velocity="12.0" />
+        <safety_controller k_position="100" k_velocity="15.0" soft_lower_limit="${-0.6+0.1}" soft_upper_limit="${0.785398164-0.1}" />
         <dynamics damping="50" friction="1"/>
     </joint>
