Commit message: New head meshes and description.

File: arrg/ua_robots/hokuyo_urg_description/urdf/hokuyo_urg.xacro (robot description, xacro)
@@ -22,4 +22,5 @@
                     <mesh filename="package://hokuyo_urg_description/meshes/hokuyo_urg.stl"/>
                 </geometry>
+                <material name="Black" />
             </visual>
             <collision>

File: arrg/ua_robots/videre_stoc_description/urdf/videre_stereo_6cm.xacro (robot description, xacro)
@@ -34,4 +34,5 @@
                     <cylinder radius="${eye_radius}" length="${eye_length}" />
                 </geometry>
+                <material name="Black" />
             </visual>
             <collision>

File: arrg/ua_robots/videre_stoc_description/urdf/videre_stereo_9cm.xacro (robot description, xacro)
@@ -34,4 +34,5 @@
                     <cylinder radius="${eye_radius}" length="${eye_length}" />
                 </geometry>
+                <material name="Black" />
             </visual>
             <collision>

File: arrg/ua_robots/wubble_description/urdf/wubble2.urdf.xacro (robot description, xacro)
@@ -44,19 +44,19 @@
     <!-- WUBBLE HEAD ATTACHMENT -->
     <joint name="head_base_joint" type="fixed">
-        <origin xyz="0.0254 0 ${0.8001-0.019}" rpy="0 0 0" />
+        <origin xyz="0.0264 0 0.7811" rpy="0 0 0" />
         <parent link="platform_link"/>
         <child link="head_base_link"/>
     </joint>
     <joint name="head_pan_joint" type="revolute">
-        <origin xyz="0.0545 0 0.026" rpy="0 0 0" />
+        <origin xyz="0.052 0 0.025" rpy="0 0 0" />
         <parent link="head_base_link"/>
         <child link="head_pan_link"/>
         <axis xyz="0 0 1" />
-        <limit lower="-1.57" upper="1.57" effort="100" velocity="12.0" />
-        <safety_controller k_position="100" k_velocity="15.0" soft_lower_limit="${-1.57}" soft_upper_limit="${1.57}" />
+        <limit lower="-2.61" upper="2.61" effort="100" velocity="12.0" />
+        <safety_controller k_position="100" k_velocity="15.0" soft_lower_limit="${-2.61}" soft_upper_limit="${2.61}" />
         <dynamics damping="50" friction="1"/>
     </joint>
     <joint name="head_tilt_joint" type="revolute">
-        <origin xyz="0.06506 0 0.06147" rpy="0 0 0" />
+        <origin xyz="0.02899 0 0.03458" rpy="0 0 0" />
         <parent link="head_pan_link"/>
         <child link="head_tilt_link"/>
@@ -68,4 +68,26 @@
     <link name="head_base_link">
         <inertial>
+            <mass value="0.13"/>
+            <origin xyz="0 0 0" rpy="0 0 0" />
+            <inertia ixx="0.1" ixy="0" ixz="0"
+                     iyy="0.1" iyz="0"
+                     izz="0.1"/>
+        </inertial>
+        <visual>
+            <origin xyz="0 0 0" rpy="0 0 0"/>
+            <geometry>
+                <mesh filename="package://wubble_description/meshes/head_base_link.stl"/>
+            </geometry>
+            <material name="GunMetalBrushedAluminum" />
+        </visual>
+        <collision>
+            <origin xyz="0 0 0" rpy="0 0 0"/>
+            <geometry>
+                <mesh filename="package://wubble_description/meshes/head_base_link.stl"/>
+            </geometry>
+        </collision>
+    </link>
+    <link name="head_pan_link">
+        <inertial>
             <mass value="0.05"/>
             <origin xyz="0 0 0" rpy="0 0 0" />
@@ -77,26 +99,4 @@
             <origin xyz="0 0 0" rpy="0 0 0"/>
             <geometry>
-                <mesh filename="package://wubble_description/meshes/head_base_link.stl"/>
-            </geometry>
-            <material name="GunMetalBrushedAluminum" />
-        </visual>
-        <collision>
-            <origin xyz="0 0 0" rpy="0 0 0"/>
-            <geometry>
-                <mesh filename="package://wubble_description/meshes/head_base_link.stl"/>
-            </geometry>
-        </collision>
-    </link>
-    <link name="head_pan_link">
-        <inertial>
-            <mass value="0.05"/>
-            <origin xyz="0 0 0" rpy="0 0 0" />
-            <inertia ixx="0.1" ixy="0" ixz="0"
-                     iyy="0.1" iyz="0"
-                     izz="0.1"/>
-        </inertial>
-        <visual>
-            <origin xyz="0 0 0" rpy="0 0 0"/>
-            <geometry>
                 <mesh filename="package://wubble_description/meshes/head_pan_link.stl"/>
             </geometry>
@@ -112,5 +112,5 @@
     <link name="head_tilt_link">
         <inertial>
-            <mass value="0.05"/>
+            <mass value="0.25"/>
             <origin xyz="0 0 0" rpy="0 0 0" />
             <inertia ixx="0.1" ixy="0" ixz="0"
@@ -144,9 +144,9 @@
     <!-- SWISSRANGER CAMERA ATTACHMENT -->
     <swissranger_camera name="swissranger" parent="head_tilt_link">
-        <origin xyz="0.0125 0 ${0.036-0.003}" rpy="${M_PI} 0 0" />
+        <origin xyz="0.0195 -0.004 0.1235" rpy="${M_PI} 0 0" />
     </swissranger_camera>
     <!-- VIDERE STEREO CAMERA ATTACHMENT -->
     <videre_stereo_6cm name="stoc" parent="head_tilt_link" >
-        <origin xyz="0.03 0 ${0.036 + 0.016}" rpy="0 0 0" />
+        <origin xyz="0.0375 0 0.142" rpy="0 0 0" />
     </videre_stereo_6cm>
     <!-- WUBBLE ARM ATTACHMENT -->
@@ -228,19 +228,25 @@
     <gazebo reference="head_base_link">
         <material>SmartArm/GunMetalBrushedAluminum</material>
+        <turnGravityOff>true</turnGravityOff>
     </gazebo>
     <gazebo reference="head_pan_link">
         <material>SmartArm/GunMetalBrushedAluminum</material>
+        <turnGravityOff>true</turnGravityOff>
     </gazebo>
     <gazebo reference="head_tilt_link">
         <material>SmartArm/GunMetalBrushedAluminum</material>
+        <turnGravityOff>true</turnGravityOff>
     </gazebo>
     <gazebo reference="neck_support_link">
         <material>SmartArm/GunMetalBrushedAluminum</material>
+        <turnGravityOff>true</turnGravityOff>
     </gazebo>
     <gazebo reference="neck_tilt_link">
         <material>SmartArm/GunMetalBrushedAluminum</material>
+        <turnGravityOff>true</turnGravityOff>
     </gazebo>
     <gazebo reference="platform_link">
         <material>Erratic/White</material>
+        <turnGravityOff>true</turnGravityOff>
     </gazebo>
 </robot>

Commit message: Add all meshes in collada format, make all urdf's point to them instead of stls and add a collada description of the whole wubble2 robot.

File: arrg/ua_robots/hokuyo_urg_description/urdf/hokuyo_urg.xacro (robot description, xacro)
@@ -20,5 +20,5 @@
                 <origin xyz="0.0 0.0 0.0" rpy="${M_PI/2} 0 ${M_PI/2}" />
                 <geometry>
-                    <mesh filename="package://hokuyo_urg_description/meshes/hokuyo_urg.stl"/>
+                    <mesh filename="package://hokuyo_urg_description/meshes/collada/hokuyo_urg.dae"/>
                 </geometry>
                 <material name="Black" />
@@ -27,5 +27,5 @@
                 <origin xyz="0.0 0.0 0.0" rpy="${M_PI/2} 0 ${M_PI/2}" />
                 <geometry>
-                    <mesh filename="package://hokuyo_urg_description/meshes/convex/hokuyo_urg_convex.stlb"/>
+                    <mesh filename="package://hokuyo_urg_description/meshes/collada/hokuyo_urg.dae"/>
                 </geometry>
             </collision>

File: arrg/ua_robots/swissranger_camera_description/urdf/swissranger_camera.xacro (robot description, xacro)
@@ -20,5 +20,5 @@
                 <origin xyz="0 0 0" rpy="0 0 0" />
                 <geometry>
-                    <mesh filename="package://swissranger_camera_description/meshes/SR4000.stl"/>
+                    <mesh filename="package://swissranger_camera_description/meshes/collada/SR4000.dae"/>
                 </geometry>
             </visual>
@@ -26,5 +26,5 @@
                 <origin xyz="0 0 0" rpy="0 0 0" />
                 <geometry>
-                    <mesh filename="package://swissranger_camera_description/meshes/convex/SR4000_convex.stlb"/>
+                    <mesh filename="package://swissranger_camera_description/meshes/collada/SR4000.dae"/>
                 </geometry>
             </collision>

File: arrg/ua_robots/wubble_arm_description/urdf/wubble_arm.xacro (robot description, xacro)
@@ -147,12 +147,12 @@
                 <origin xyz="0 0 0" rpy="0 0 0" />
                 <geometry>
-                    <mesh filename="package://wubble_arm_description/meshes/L0_base_link.stl"/>
-                </geometry>
-                <material name="GunMetalBrushedAluminum" />
-            </visual>
-            <collision>
-                <origin xyz="0 0 0" rpy="0 0 0" />
-                <geometry>
-                    <mesh filename="package://wubble_arm_description/meshes/L0_base_link.stl"/>
+                    <mesh filename="package://wubble_arm_description/meshes/collada/L0_base_link.dae"/>
+                </geometry>
+                <material name="GunMetalBrushedAluminum" />
+            </visual>
+            <collision>
+                <origin xyz="0 0 0" rpy="0 0 0" />
+                <geometry>
+                    <mesh filename="package://wubble_arm_description/meshes/collada/L0_base_link.dae"/>
                 </geometry>
             </collision>
@@ -169,12 +169,12 @@
                 <origin xyz="0 0 0" rpy="0 0 0" />
                 <geometry>
-                    <mesh filename="package://wubble_arm_description/meshes/L1_shoulder_pitch_link.stl"/>
-                </geometry>
-                <material name="GunMetalBrushedAluminum" />
-            </visual>
-            <collision>
-                <origin xyz="0 0 0" rpy="0 0 0" />
-                <geometry>
-                    <mesh filename="package://wubble_arm_description/meshes/L1_shoulder_pitch_link.stl"/>
+                    <mesh filename="package://wubble_arm_description/meshes/collada/L1_shoulder_pitch_link.dae"/>
+                </geometry>
+                <material name="GunMetalBrushedAluminum" />
+            </visual>
+            <collision>
+                <origin xyz="0 0 0" rpy="0 0 0" />
+                <geometry>
+                    <mesh filename="package://wubble_arm_description/meshes/collada/L1_shoulder_pitch_link.dae"/>
                 </geometry>
             </collision>
@@ -191,5 +191,5 @@
                 <origin xyz="0 0.055 0" rpy="0 0 0" />
                 <geometry>
-                    <mesh filename="package://wubble_arm_description/meshes/L2_shoulder_yaw_link.stl"/>
+                    <mesh filename="package://wubble_arm_description/meshes/collada/L2_shoulder_yaw_link.dae"/>
                 </geometry>
                 <material name="GunMetalBrushedAluminum" />
@@ -198,5 +198,5 @@
                 <origin xyz="0 0.0545 0" rpy="0 0 0" />
                 <geometry>
-                    <mesh filename="package://wubble_arm_description/meshes/L2_shoulder_yaw_link.stl"/>
+                    <mesh filename="package://wubble_arm_description/meshes/collada/L2_shoulder_yaw_link.dae"/>
                 </geometry>
             </collision>
@@ -213,12 +213,12 @@
                 <origin xyz="0 0 0" rpy="0 0 0" />
                 <geometry>
-                    <mesh filename="package://wubble_arm_description/meshes/L3_shoulder_roll_link.stl"/>
-                </geometry>
-                <material name="GunMetalBrushedAluminum" />
-            </visual>
-            <collision>
-                <origin xyz="0 0 0" rpy="0 0 0" />
-                <geometry>
-                    <mesh filename="package://wubble_arm_description/meshes/L3_shoulder_roll_link.stl"/>
+                    <mesh filename="package://wubble_arm_description/meshes/collada/L3_shoulder_roll_link.dae"/>
+                </geometry>
+                <material name="GunMetalBrushedAluminum" />
+            </visual>
+            <collision>
+                <origin xyz="0 0 0" rpy="0 0 0" />
+                <geometry>
+                    <mesh filename="package://wubble_arm_description/meshes/collada/L3_shoulder_roll_link.dae"/>
                 </geometry>
             </collision>
@@ -235,5 +235,5 @@
                 <origin xyz="0.035 0.044 0.026" rpy="0 0 0" />
                 <geometry>
-                    <mesh filename="package://wubble_arm_description/meshes/L4_elbow_pitch_link.stl"/>
+                    <mesh filename="package://wubble_arm_description/meshes/collada/L4_elbow_pitch_link.dae"/>
                 </geometry>
                 <material name="GunMetalBrushedAluminum" />
@@ -242,5 +242,5 @@
                 <origin xyz="0.035 0.044 0.026" rpy="0 0 0" />
                 <geometry>
-                    <mesh filename="package://wubble_arm_description/meshes/L4_elbow_pitch_link.stl"/>
+                    <mesh filename="package://wubble_arm_description/meshes/collada/L4_elbow_pitch_link.dae"/>
                 </geometry>
             </collision>
@@ -257,5 +257,5 @@
                 <origin xyz="0.025 0 0" rpy="0 0 0" />
                 <geometry>
-                    <mesh filename="package://wubble_arm_description/meshes/L5_wrist_roll_link.stl"/>
+                    <mesh filename="package://wubble_arm_description/meshes/collada/L5_wrist_roll_link.dae"/>
                 </geometry>
                 <material name="GunMetalBrushedAluminum" />
@@ -264,5 +264,5 @@
                 <origin xyz="0.025 0 0" rpy="0 0 0" />
                 <geometry>
-                    <mesh filename="package://wubble_arm_description/meshes/L5_wrist_roll_link.stl"/>
+                    <mesh filename="package://wubble_arm_description/meshes/collada/L5_wrist_roll_link.dae"/>
                 </geometry>
             </collision>
@@ -279,12 +279,12 @@
                 <origin xyz="0 0 0" rpy="0 0 0" />
                 <geometry>
-                    <mesh filename="package://wubble_arm_description/meshes/L6_wrist_pitch_link.stl"/>
-                </geometry>
-                <material name="GunMetalBrushedAluminum" />
-            </visual>
-            <collision>
-                <origin xyz="0 0 0" rpy="0 0 0" />
-                <geometry>
-                    <mesh filename="package://wubble_arm_description/meshes/L6_wrist_pitch_link.stl"/>
+                    <mesh filename="package://wubble_arm_description/meshes/collada/L6_wrist_pitch_link.dae"/>
+                </geometry>
+                <material name="GunMetalBrushedAluminum" />
+            </visual>
+            <collision>
+                <origin xyz="0 0 0" rpy="0 0 0" />
+                <geometry>
+                    <mesh filename="package://wubble_arm_description/meshes/collada/L6_wrist_pitch_link.dae"/>
                 </geometry>
             </collision>
@@ -301,5 +301,5 @@
                 <origin xyz="0.091 0 0" rpy="0 0 0" />
                 <geometry>
-                    <mesh filename="package://wubble_arm_description/meshes/L7_wrist_yaw_link.stl"/>
+                    <mesh filename="package://wubble_arm_description/meshes/collada/L7_wrist_yaw_link.dae"/>
                 </geometry>
                 <material name="GunMetalBrushedAluminum" />
@@ -308,5 +308,5 @@
                 <origin xyz="0.091 0 0" rpy="0 0 0" />
                 <geometry>
-                    <mesh filename="package://wubble_arm_description/meshes/L7_wrist_yaw_link.stl"/>
+                    <mesh filename="package://wubble_arm_description/meshes/collada/L7_wrist_yaw_link.dae"/>
                 </geometry>
             </collision>
@@ -323,12 +323,12 @@
                 <origin xyz="0 0 0" rpy="0 0 0" />
                 <geometry>
-                    <mesh filename="package://wubble_arm_description/meshes/L8_gripper_left_finger.stl"/>
-                </geometry>
-                <material name="GunMetalBrushedAluminum" />
-            </visual>
-            <collision>
-                <origin xyz="0 0 0" rpy="0 0 0" />
-                <geometry>
-                    <mesh filename="package://wubble_arm_description/meshes/L8_gripper_left_finger.stl"/>
+                    <mesh filename="package://wubble_arm_description/meshes/collada/L8_gripper_left_finger.dae"/>
+                </geometry>
+                <material name="GunMetalBrushedAluminum" />
+            </visual>
+            <collision>
+                <origin xyz="0 0 0" rpy="0 0 0" />
+                <geometry>
+                    <mesh filename="package://wubble_arm_description/meshes/collada/L8_gripper_left_finger.dae"/>
                 </geometry>
             </collision>
@@ -345,12 +345,12 @@
                 <origin xyz="0 0 0" rpy="0 0 0" />
                 <geometry>
-                    <mesh filename="package://wubble_arm_description/meshes/L9_gripper_right_finger.stl"/>
-                </geometry>
-                <material name="GunMetalBrushedAluminum" />
-            </visual>
-            <collision>
-                <origin xyz="0 0 0" rpy="0 0 0" />
-                <geometry>
-                    <mesh filename="package://wubble_arm_description/meshes/L9_gripper_right_finger.stl"/>
+                    <mesh filename="package://wubble_arm_description/meshes/collada/L9_gripper_right_finger.dae"/>
+                </geometry>
+                <material name="GunMetalBrushedAluminum" />
+            </visual>
+            <collision>
+                <origin xyz="0 0 0" rpy="0 0 0" />
+                <geometry>
+                    <mesh filename="package://wubble_arm_description/meshes/collada/L9_gripper_right_finger.dae"/>
                 </geometry>
             </collision>

File: arrg/ua_robots/wubble_description/urdf/wubble2.urdf.xacro (robot description, xacro)
@@ -31,5 +31,5 @@
             <origin xyz="0 0 0" rpy="0 0 0"/>
             <geometry>
-                <mesh filename="package://wubble_description/meshes/wubble2_platform.stl"/>
+                <mesh filename="package://wubble_description/meshes/collada/wubble2_platform.dae"/>
             </geometry>
             <material name="White" />
@@ -38,5 +38,5 @@
             <origin xyz="0 0 0" rpy="0 0 0"/>
             <geometry>
-                <mesh filename="package://wubble_description/meshes/wubble2_platform.stl"/>
+                <mesh filename="package://wubble_description/meshes/collada/wubble2_platform.dae"/>
             </geometry>
         </collision>
@@ -77,12 +77,12 @@
             <origin xyz="0 0 0" rpy="0 0 0"/>
             <geometry>
-                <mesh filename="package://wubble_description/meshes/head_base_link.stl"/>
-            </geometry>
-            <material name="GunMetalBrushedAluminum" />
-        </visual>
-        <collision>
-            <origin xyz="0 0 0" rpy="0 0 0"/>
-            <geometry>
-                <mesh filename="package://wubble_description/meshes/head_base_link.stl"/>
+                <mesh filename="package://wubble_description/meshes/collada/head_base_link.dae"/>
+            </geometry>
+            <material name="GunMetalBrushedAluminum" />
+        </visual>
+        <collision>
+            <origin xyz="0 0 0" rpy="0 0 0"/>
+            <geometry>
+                <mesh filename="package://wubble_description/meshes/collada/head_base_link.dae"/>
             </geometry>
         </collision>
@@ -99,12 +99,12 @@
             <origin xyz="0 0 0" rpy="0 0 0"/>
             <geometry>
-                <mesh filename="package://wubble_description/meshes/head_pan_link.stl"/>
-            </geometry>
-            <material name="GunMetalBrushedAluminum" />
-        </visual>
-        <collision>
-            <origin xyz="0 0 0" rpy="0 0 0"/>
-            <geometry>
-                <mesh filename="package://wubble_description/meshes/head_pan_link.stl"/>
+                <mesh filename="package://wubble_description/meshes/collada/head_pan_link.dae"/>
+            </geometry>
+            <material name="GunMetalBrushedAluminum" />
+        </visual>
+        <collision>
+            <origin xyz="0 0 0" rpy="0 0 0"/>
+            <geometry>
+                <mesh filename="package://wubble_description/meshes/collada/head_pan_link.dae"/>
             </geometry>
         </collision>
@@ -121,12 +121,12 @@
             <origin xyz="0 0 0" rpy="0 0 0"/>
             <geometry>
-                <mesh filename="package://wubble_description/meshes/head_tilt_link.stl"/>
-            </geometry>
-            <material name="GunMetalBrushedAluminum" />
-        </visual>
-        <collision>
-            <origin xyz="0 0 0" rpy="0 0 0"/>
-            <geometry>
-                <mesh filename="package://wubble_description/meshes/head_tilt_link.stl"/>
+                <mesh filename="package://wubble_description/meshes/collada/head_tilt_link.dae"/>
+            </geometry>
+            <material name="GunMetalBrushedAluminum" />
+        </visual>
+        <collision>
+            <origin xyz="0 0 0" rpy="0 0 0"/>
+            <geometry>
+                <mesh filename="package://wubble_description/meshes/collada/head_tilt_link.dae"/>
             </geometry>
         </collision>
@@ -180,12 +180,12 @@
             <origin xyz="0 0 0" rpy="0 0 0"/>
             <geometry>
-                <mesh filename="package://wubble_description/meshes/neck_laser_support_link.stl"/>
-            </geometry>
-            <material name="GunMetalBrushedAluminum" />
-        </visual>
-        <collision>
-            <origin xyz="0 0 0" rpy="0 0 0"/>
-            <geometry>
-                <mesh filename="package://wubble_description/meshes/neck_laser_support_link.stl"/>
+                <mesh filename="package://wubble_description/meshes/collada/neck_laser_support_link.dae"/>
+            </geometry>
+            <material name="GunMetalBrushedAluminum" />
+        </visual>
+        <collision>
+            <origin xyz="0 0 0" rpy="0 0 0"/>
+            <geometry>
+                <mesh filename="package://wubble_description/meshes/collada/neck_laser_support_link.dae"/>
             </geometry>
         </collision>
@@ -202,12 +202,12 @@
             <origin xyz="0 0 0" rpy="0 0 0"/>
             <geometry>
-                <mesh filename="package://wubble_description/meshes/ax12_45_bracket.stl"/>
-            </geometry>
-            <material name="GunMetalBrushedAluminum" />
-        </visual>
-        <collision>
-            <origin xyz="0 0 0" rpy="0 0 0"/>
-            <geometry>
-                <mesh filename="package://wubble_description/meshes/ax12_45_bracket.stl"/>
+                <mesh filename="package://wubble_description/meshes/collada/ax12_45_bracket.dae"/>
+            </geometry>
+            <material name="GunMetalBrushedAluminum" />
+        </visual>
+        <collision>
+            <origin xyz="0 0 0" rpy="0 0 0"/>
+            <geometry>
+                <mesh filename="package://wubble_description/meshes/collada/ax12_45_bracket.dae"/>
             </geometry>
         </collision>
