Commit message: dae to stl

File: arrg/ua_robots/hokuyo_urg_description/urdf/hokuyo_urg.xacro (robot description, xacro)
@@ -20,5 +20,5 @@
                 <origin xyz="0.0 0.0 0.0" rpy="${M_PI/2} 0 ${M_PI/2}" />
                 <geometry>
-                    <mesh filename="package://hokuyo_urg_description/meshes/collada/hokuyo_urg.dae"/>
+                    <mesh filename="package://hokuyo_urg_description/meshes/hokuyo_urg.stl"/>
                 </geometry>
                 <material name="Black" />
@@ -27,5 +27,5 @@
                 <origin xyz="0.0 0.0 0.0" rpy="${M_PI/2} 0 ${M_PI/2}" />
                 <geometry>
-                    <mesh filename="package://hokuyo_urg_description/meshes/collada/hokuyo_urg.dae"/>
+                    <mesh filename="package://hokuyo_urg_description/meshes/hokuyo_urg.stl"/>
                 </geometry>
             </collision>

File: arrg/ua_robots/swissranger_camera_description/urdf/swissranger_camera.xacro (robot description, xacro)
@@ -20,5 +20,5 @@
                 <origin xyz="0 0 0" rpy="0 0 0" />
                 <geometry>
-                    <mesh filename="package://swissranger_camera_description/meshes/collada/SR4000.dae"/>
+                    <mesh filename="package://swissranger_camera_description/meshes/SR4000.stl"/>
                 </geometry>
             </visual>
@@ -26,5 +26,5 @@
                 <origin xyz="0 0 0" rpy="0 0 0" />
                 <geometry>
-                    <mesh filename="package://swissranger_camera_description/meshes/collada/SR4000.dae"/>
+                    <mesh filename="package://swissranger_camera_description/meshes/SR4000.stl"/>
                 </geometry>
             </collision>

Commit message: Update all urdfs to use collada dae files for collision meshes, update ompl configuration to work with Diamondback

File: arrg/ua_robots/hokuyo_urg_description/urdf/hokuyo_urg.xacro (robot description, xacro)
@@ -27,5 +27,5 @@
                 <origin xyz="0.0 0.0 0.0" rpy="${M_PI/2} 0 ${M_PI/2}" />
                 <geometry>
-                    <mesh filename="package://hokuyo_urg_description/meshes/hokuyo_urg.stl"/>
+                    <mesh filename="package://hokuyo_urg_description/meshes/collada/hokuyo_urg.dae"/>
                 </geometry>
             </collision>

File: arrg/ua_robots/swissranger_camera_description/urdf/swissranger_camera.xacro (robot description, xacro)
@@ -26,5 +26,5 @@
                 <origin xyz="0 0 0" rpy="0 0 0" />
                 <geometry>
-                    <mesh filename="package://swissranger_camera_description/meshes/SR4000.stl"/>
+                    <mesh filename="package://swissranger_camera_description/meshes/collada/SR4000.dae"/>
                 </geometry>
             </collision>

File: arrg/ua_robots/wubble_arm_description/urdf/wubble_arm.xacro (robot description, xacro)
@@ -166,5 +166,5 @@
                 <origin xyz="0 0 0" rpy="0 0 0" />
                 <geometry>
-                    <mesh filename="package://wubble_arm_description/meshes/L0_base_link.stl"/>
+                    <mesh filename="package://wubble_arm_description/meshes/collada/L0_base_link.dae"/>
                 </geometry>
             </collision>
@@ -188,5 +188,5 @@
                 <origin xyz="0 0 0" rpy="0 0 0" />
                 <geometry>
-                    <mesh filename="package://wubble_arm_description/meshes/L1_shoulder_pitch_link.stl"/>
+                    <mesh filename="package://wubble_arm_description/meshes/collada/L1_shoulder_pitch_link.dae"/>
                 </geometry>
             </collision>
@@ -210,5 +210,5 @@
                 <origin xyz="0 0.0545 0" rpy="0 0 0" />
                 <geometry>
-                    <mesh filename="package://wubble_arm_description/meshes/L2_shoulder_pan_link.stl"/>
+                    <mesh filename="package://wubble_arm_description/meshes/collada/L2_shoulder_pan_link.dae"/>
                 </geometry>
             </collision>
@@ -232,5 +232,5 @@
                 <origin xyz="0 0 0" rpy="0 0 0" />
                 <geometry>
-                    <mesh filename="package://wubble_arm_description/meshes/L3_upperarm_roll_link.stl"/>
+                    <mesh filename="package://wubble_arm_description/meshes/collada/L3_upperarm_roll_link.dae"/>
                 </geometry>
             </collision>
@@ -254,5 +254,5 @@
                 <origin xyz="0.035 0.044 0.026" rpy="0 0 0" />
                 <geometry>
-                    <mesh filename="package://wubble_arm_description/meshes/L4_elbow_flex_link.stl"/>
+                    <mesh filename="package://wubble_arm_description/meshes/collada/L4_elbow_flex_link.dae"/>
                 </geometry>
             </collision>
@@ -276,5 +276,5 @@
                 <origin xyz="0.025 0 0" rpy="0 0 0" />
                 <geometry>
-                    <mesh filename="package://wubble_arm_description/meshes/L5_forearm_roll_link.stl"/>
+                    <mesh filename="package://wubble_arm_description/meshes/collada/L5_forearm_roll_link.dae"/>
                 </geometry>
             </collision>
@@ -298,5 +298,5 @@
                 <origin xyz="0 0 0" rpy="0 0 0" />
                 <geometry>
-                    <mesh filename="package://wubble_arm_description/meshes/L6_wrist_pitch_link.stl"/>
+                    <mesh filename="package://wubble_arm_description/meshes/collada/L6_wrist_pitch_link.dae"/>
                 </geometry>
             </collision>
@@ -320,5 +320,5 @@
                 <origin xyz="0.0541 0 0" rpy="0 0 0" />
                 <geometry>
-                    <mesh filename="package://wubble_arm_description/meshes/L7_wrist_roll_link.stl"/>
+                    <mesh filename="package://wubble_arm_description/meshes/collada/L7_wrist_roll_link.dae"/>
                 </geometry>
             </collision>
@@ -342,5 +342,5 @@
                 <origin xyz="0 0 0" rpy="0 0 0" />
                 <geometry>
-                    <mesh filename="package://wubble_arm_description/meshes/L8_gripper_left_finger.stl"/>
+                    <mesh filename="package://wubble_arm_description/meshes/collada/L8_gripper_left_finger.dae"/>
                 </geometry>
             </collision>
@@ -364,5 +364,5 @@
                 <origin xyz="0 0 0" rpy="0 0 0" />
                 <geometry>
-                    <mesh filename="package://wubble_arm_description/meshes/L9_gripper_right_finger.stl"/>
+                    <mesh filename="package://wubble_arm_description/meshes/collada/L9_gripper_right_finger.dae"/>
                 </geometry>
             </collision>

File: arrg/ua_robots/wubble_description/urdf/wubble2.urdf.xacro (robot description, xacro)
@@ -39,5 +39,5 @@
             <origin xyz="0 0 0" rpy="0 0 0"/>
             <geometry>
-                <mesh filename="package://wubble_description/meshes/wubble2_platform.stl"/>
+                <mesh filename="package://wubble_description/meshes/collada/wubble2_platform.dae"/>
             </geometry>
         </collision>
@@ -89,5 +89,5 @@
             <origin xyz="0 0 0" rpy="0 0 0"/>
             <geometry>
-                <mesh filename="package://wubble_description/meshes/head_base_link.stl"/>
+                <mesh filename="package://wubble_description/meshes/collada/head_base_link.dae"/>
             </geometry>
         </collision>
@@ -111,5 +111,5 @@
             <origin xyz="0 0 0" rpy="0 0 0"/>
             <geometry>
-                <mesh filename="package://wubble_description/meshes/head_pan_link.stl"/>
+                <mesh filename="package://wubble_description/meshes/collada/head_pan_link.dae"/>
             </geometry>
         </collision>
@@ -133,5 +133,5 @@
             <origin xyz="0 0 0" rpy="0 0 0"/>
             <geometry>
-                <mesh filename="package://wubble_description/meshes/head_tilt_link.stl"/>
+                <mesh filename="package://wubble_description/meshes/collada/head_tilt_link.dae"/>
             </geometry>
         </collision>
@@ -192,5 +192,5 @@
             <origin xyz="0 0 0" rpy="0 0 0"/>
             <geometry>
-                <mesh filename="package://wubble_description/meshes/neck_laser_support_link.stl"/>
+                <mesh filename="package://wubble_description/meshes/collada/neck_laser_support_link.dae"/>
             </geometry>
         </collision>
@@ -214,5 +214,5 @@
             <origin xyz="0 0 0" rpy="0 0 0"/>
             <geometry>
-                <mesh filename="package://wubble_description/meshes/ax12_45_bracket.stl"/>
+                <mesh filename="package://wubble_description/meshes/collada/ax12_45_bracket.dae"/>
             </geometry>
         </collision>

Commit message: use dae files in laser urdf

File: arrg/ua_robots/hokuyo_urg_description/urdf/hokuyo_urg.xacro (robot description, xacro)
@@ -20,5 +20,5 @@
                 <origin xyz="0.0 0.0 0.0" rpy="${M_PI/2} 0 ${M_PI/2}" />
                 <geometry>
-                    <mesh filename="package://hokuyo_urg_description/meshes/hokuyo_urg.stl"/>
+                    <mesh filename="package://hokuyo_urg_description/meshes/collada/hokuyo_urg.dae"/>
                 </geometry>
                 <material name="Black" />
