Commit message: Fixed some bad tags.

File: arrg/ua_robots/erratic_description/urdf/erratic_wheel.xacro (robot description, xacro)
@@ -28,5 +28,5 @@
             </visual>
             <collision>
-                <origin xyz="$0 ${reflect*0.0125} 0" rpy="{M_PI/2} 0 0" />
+                <origin xyz="0 ${reflect*0.0125} 0" rpy="${M_PI/2} 0 0" />
                 <geometry>
                     <cylinder radius="0.0127" length="0.025" />
@@ -59,5 +59,5 @@
             </visual>
             <collision>
-                <origin xyz="0 0 0" rpy="$0 0 ${M_PI/2}" />
+                <origin xyz="0 0 0" rpy="0 0 ${M_PI/2}" />
                 <geometry>
                     <mesh filename="package://erratic_description/meshes/erratic_wheel.stl"/>

File: arrg/ua_robots/videre_stoc_description/urdf/videre_stoc.xacro (robot description, xacro)
@@ -57,5 +57,5 @@
                 <origin xyz="0 0 0" rpy="0 0 0" />
                 <geometry>
-                    <sphere radius="$0.001" />
+                    <sphere radius="0.001" />
                 </geometry>
             </visual>
@@ -63,5 +63,5 @@
                 <origin xyz="0 0 0" rpy="0 0 0" />
                 <geometry>
-                    <sphere radius="$0.001" />
+                    <sphere radius="0.001" />
                 </geometry>
             </collision>
