Commit message: Ignore and delete generated stl decompositions. Fix all urdfs to point to new packages for stl files.

File: arrg/ua_robots/erratic_description/urdf/erratic_base.xacro (robot description, xacro)
@@ -92,5 +92,5 @@
                 <origin xyz="0.0 0.0 0.0" rpy="0 0 0" />
                 <geometry>
-                    <mesh filename="package://wubble_robots/meshes/erratic_top_origin.stl"/>
+                    <mesh filename="package://erratic_description/meshes/erratic_top.stl"/>
                 </geometry>
                 <material name="Blue" />
@@ -99,5 +99,5 @@
                 <origin xyz="0.0 0.0 0.0" rpy="0 0 0" />
                 <geometry>
-                    <mesh filename="package://wubble_robots/meshes/erratic_top_origin.stl"/>
+                    <mesh filename="package://erratic_description/meshes/erratic_top.stl"/>
                 </geometry>
             </collision>

File: arrg/ua_robots/erratic_description/urdf/erratic_wheel.xacro (robot description, xacro)
@@ -6,7 +6,4 @@
     <!-- Properties (Constants) -->
     <property name="M_PI" value="3.14159"/>
-    <property name="wheel_radius" value="0.0762" />
-    <property name="wheel_length" value="0.02" />
-    <property name="caster_wheel_offset_y" value="0.17" />
     <property name="wheel_offset_z" value="${-base_size_z/2 + 0.0236}" />
     <macro name="erratic_wheel" params="suffix parent reflect">
@@ -57,5 +54,5 @@
                 <origin xyz="0 0 0" rpy="0 0 ${M_PI/2}" />
                 <geometry>
-                    <mesh filename="package://wubble_robots/meshes/erratic_wheel.stl"/>
+                    <mesh filename="package://erratic_description/meshes/erratic_wheel.stl"/>
                 </geometry>
                 <material name="Black" />
@@ -64,6 +61,5 @@
                 <origin xyz="0 0 0" rpy="$0 0 ${M_PI/2}" />
                 <geometry>
-                    <mesh filename="package://wubble_robots/meshes/erratic_wheel.stl"/>
-<!--                    <cylinder radius="${wheel_radius}" length="${wheel_length}" />-->
+                    <mesh filename="package://erratic_description/meshes/erratic_wheel.stl"/>
                 </geometry>
             </collision>

File: arrg/ua_robots/hokuyo_urg_description/urdf/hokuyo_urg.xacro (robot description, xacro)
@@ -15,5 +15,5 @@
                 <origin xyz="0.0 0.0 0.0" rpy="${M_PI/2} 0 ${M_PI/2}" />
                 <geometry>
-                    <mesh filename="package://wubble_robots/meshes/hokuyo_urg.stl"/>
+                    <mesh filename="package://hokuyo_urg_description/meshes/hokuyo_urg.stl"/>
                 </geometry>
             </visual>
@@ -21,5 +21,5 @@
                 <origin xyz="0.0 0.0 0.0" rpy="${M_PI/2} 0 ${M_PI/2}" />
                 <geometry>
-                    <mesh filename="package://wubble_robots/meshes/hokuyo_urg.stl"/>
+                    <mesh filename="package://hokuyo_urg_description/meshes/hokuyo_urg.stl"/>
                 </geometry>
             </collision>

File: arrg/ua_robots/smart_arm_description/urdf/smart_arm.xacro (robot description, xacro)
@@ -4,7 +4,7 @@
     xmlns:controller="http://playerstage.sourceforge.net/gazebo/xmlschema/#controller"
     xmlns:interface="http://playerstage.sourceforge.net/gazebo/xmlschema/#interface">
-    <macro name="smart_arm" params="parent">
+    <macro name="smart_arm" params="parent *origin">
         <joint name="arm_base_joint" type="fixed">
-            <origin xyz="${top_size_x/2 - 0.0575} 0 ${top_size_z/2 + 0.025}"/>
+            <insert_block name="origin" />
             <parent link="${parent}"/>
             <child link="arm_base_link"/>
@@ -21,12 +21,11 @@
                 <origin xyz="0.0 0.0 0.0" rpy="0 0 0" />
                 <geometry>
-<!--                    <box size="${0.0575*2} ${0.0575*2} ${0.025*2}" />-->
-                    <mesh filename="package://wubble_robots/meshes/arm_base.stl"/>
-                </geometry>
-            </visual>
-            <collision>
-                <origin xyz="0.0 0.0 0.0" rpy="0 0 0" />
-                <geometry>
-                    <box size="${0.0575*2} ${0.0575*2} ${0.025*2}" />
+                    <mesh filename="package://smart_arm_description/meshes/arm_base.stl"/>
+                </geometry>
+            </visual>
+            <collision>
+                <origin xyz="0.0 0.0 0.0" rpy="0 0 0" />
+                <geometry>
+                    <mesh filename="package://smart_arm_description/meshes/arm_base.stl"/>
                 </geometry>
             </collision>
@@ -59,11 +58,11 @@
                 <origin xyz="0.0 0.0 0.005" rpy="0 0 0" />
                 <geometry>
-                    <mesh filename="package://wubble_robots/meshes/arm_shoulder.stl"/>
-                </geometry>
-            </visual>
-            <collision>
-                <origin xyz="0.0 0.0 0.0" rpy="0 0 0" />
-                <geometry>
-                    <mesh filename="package://wubble_robots/meshes/arm_shoulder.stl"/>
+                    <mesh filename="package://smart_arm_description/meshes/arm_shoulder_pan.stl"/>
+                </geometry>
+            </visual>
+            <collision>
+                <origin xyz="0.0 0.0 0.0" rpy="0 0 0" />
+                <geometry>
+                    <mesh filename="package://smart_arm_description/meshes/arm_shoulder_pan.stl"/>
                 </geometry>
             </collision>
@@ -91,16 +90,16 @@
                 <origin xyz="0.0 0.0 0.0" rpy="0 0 0" />
                 <geometry>
-                    <mesh filename="package://wubble_robots/meshes/arm_shoulder_tilt.stl"/>
-                </geometry>
-            </visual>
-            <collision>
-                <origin xyz="0.0 0.0 0.0" rpy="0 0 0" />
-                <geometry>
-                    <mesh filename="package://wubble_robots/meshes/arm_shoulder_tilt.stl"/>
-                </geometry>
-            </collision>
-        </link>
-        <transmission type="SimpleTransmission" name="arm_base_shoulder_tilt_trans">
-            <actuator name="arm_base_shoulder_tilt_motor" />
+                    <mesh filename="package://smart_arm_description/meshes/arm_shoulder_tilt.stl"/>
+                </geometry>
+            </visual>
+            <collision>
+                <origin xyz="0.0 0.0 0.0" rpy="0 0 0" />
+                <geometry>
+                    <mesh filename="package://smart_arm_description/meshes/arm_shoulder_tilt.stl"/>
+                </geometry>
+            </collision>
+        </link>
+        <transmission type="SimpleTransmission" name="shoulder_tilt_trans">
+            <actuator name="shoulder_tilt_motor" />
             <joint name="shoulder_tilt_joint" />
             <mechanicalReduction>1.0</mechanicalReduction>
@@ -129,16 +128,16 @@
                 <origin xyz="0.0 0.0 0.0" rpy="0 0 0" />
                 <geometry>
-                    <mesh filename="package://wubble_robots/meshes/arm_elbow_tilt.stl"/>
-                </geometry>
-            </visual>
-            <collision>
-                <origin xyz="0.0 0.0 0.0" rpy="0 0 0" />
-                <geometry>
-                    <mesh filename="package://wubble_robots/meshes/arm_elbow_tilt.stl"/>
-                </geometry>
-            </collision>
-        </link>
-        <transmission type="SimpleTransmission" name="arm_elbow_tilt_trans">
-            <actuator name="arm_elbow_tilt_motor" />
+                    <mesh filename="package://smart_arm_description/meshes/arm_elbow_tilt.stl"/>
+                </geometry>
+            </visual>
+            <collision>
+                <origin xyz="0.0 0.0 0.0" rpy="0 0 0" />
+                <geometry>
+                    <mesh filename="package://smart_arm_description/meshes/arm_elbow_tilt.stl"/>
+                </geometry>
+            </collision>
+        </link>
+        <transmission type="SimpleTransmission" name="elbow_tilt_trans">
+            <actuator name="elbow_tilt_motor" />
             <joint name="elbow_tilt_joint" />
             <mechanicalReduction>1.0</mechanicalReduction>
@@ -167,16 +166,16 @@
                 <origin xyz="0.0 0.0 0.0" rpy="0 0 0" />
                 <geometry>
-                    <mesh filename="package://wubble_robots/meshes/arm_wrist_rotate.stl"/>
-                </geometry>
-            </visual>
-            <collision>
-                <origin xyz="0.0 0.0 0.0" rpy="0 0 0" />
-                <geometry>
-                    <mesh filename="package://wubble_robots/meshes/arm_wrist_rotate.stl"/>
-                </geometry>
-            </collision>
-        </link>
-        <transmission type="SimpleTransmission" name="arm_wrist_rotate_trans">
-            <actuator name="arm_wrist_rotate_motor" />
+                    <mesh filename="package://smart_arm_description/meshes/arm_wrist_rotate.stl"/>
+                </geometry>
+            </visual>
+            <collision>
+                <origin xyz="0.0 0.0 0.0" rpy="0 0 0" />
+                <geometry>
+                    <mesh filename="package://smart_arm_description/meshes/arm_wrist_rotate.stl"/>
+                </geometry>
+            </collision>
+        </link>
+        <transmission type="SimpleTransmission" name="wrist_rotate_trans">
+            <actuator name="wrist_rotate_motor" />
             <joint name="wrist_rotate_joint" />
             <mechanicalReduction>1.0</mechanicalReduction>
@@ -205,16 +204,16 @@
                 <origin xyz="0.0 0.0 0.0" rpy="0 0 0" />
                 <geometry>
-                    <mesh filename="package://wubble_robots/meshes/arm_right_finger.stl"/>
-                </geometry>
-            </visual>
-            <collision>
-                <origin xyz="0.0 0.0 0.0" rpy="0 0 0" />
-                <geometry>
-                    <mesh filename="package://wubble_robots/meshes/arm_right_finger.stl"/>
-                </geometry>
-            </collision>
-        </link>
-        <transmission type="SimpleTransmission" name="arm_right_finger_trans">
-            <actuator name="arm_right_finger_motor" />
+                    <mesh filename="package://smart_arm_description/meshes/arm_right_finger.stl"/>
+                </geometry>
+            </visual>
+            <collision>
+                <origin xyz="0.0 0.0 0.0" rpy="0 0 0" />
+                <geometry>
+                    <mesh filename="package://smart_arm_description/meshes/arm_right_finger.stl"/>
+                </geometry>
+            </collision>
+        </link>
+        <transmission type="SimpleTransmission" name="finger_right_trans">
+            <actuator name="finger_right_motor" />
             <joint name="finger_right_joint" />
             <mechanicalReduction>1.0</mechanicalReduction>
@@ -243,16 +242,16 @@
                 <origin xyz="0.0 0.0 0.0" rpy="0 0 0" />
                 <geometry>
-                    <mesh filename="package://wubble_robots/meshes/arm_left_finger.stl"/>
-                </geometry>
-            </visual>
-            <collision>
-                <origin xyz="0.0 0.0 0.0" rpy="0 0 0" />
-                <geometry>
-                    <mesh filename="package://wubble_robots/meshes/arm_left_finger.stl"/>
-                </geometry>
-            </collision>
-        </link>
-        <transmission type="SimpleTransmission" name="arm_left_finger_trans">
-            <actuator name="arm_left_finger_motor" />
+                    <mesh filename="package://smart_arm_description/meshes/arm_left_finger.stl"/>
+                </geometry>
+            </visual>
+            <collision>
+                <origin xyz="0.0 0.0 0.0" rpy="0 0 0" />
+                <geometry>
+                    <mesh filename="package://smart_arm_description/meshes/arm_left_finger.stl"/>
+                </geometry>
+            </collision>
+        </link>
+        <transmission type="SimpleTransmission" name="finger_left_trans">
+            <actuator name="finger_left_motor" />
             <joint name="finger_left_joint" />
             <mechanicalReduction>1.0</mechanicalReduction>

File: arrg/ua_robots/wubble_description/urdf/wubble.urdf.xacro (robot description, xacro)
@@ -17,5 +17,11 @@
     <!-- MACRO INSTANTIATION -->
     <erratic />
-    <smart_arm parent="base_top_link" />
+    <smart_arm parent="base_top_link" >
+        <origin xyz="${top_size_x/2 - 0.0575} 0 ${top_size_z/2 + 0.025}"/>
+    </smart_arm>
+    <tilting_hokuyo parent="base_top_link">
+        <origin xyz="0.15 0 ${-top_size_z - 0.05}" rpy="${M_PI} 0 0" />
+    </tilting_hokuyo>
+    <stoc_camera name="stoc" parent="head_pan_link" />
 <!--    <joint name="laser_test_joint" type="fixed">-->
 <!--        <origin xyz="0.5 0.0 0.5" />-->
@@ -23,8 +29,4 @@
 <!--        <child link="hokuyo_link" />-->
 <!--    </joint>-->
-    <tilting_hokuyo parent="base_top_link">
-        <origin xyz="0.15 0 ${-top_size_z - 0.05}" rpy="${M_PI} 0 0" />
-    </tilting_hokuyo>
-    <stoc_camera name="stoc" parent="head_pan_link" />
     <!-- Special Links -->
     <joint name="head_support_joint" type="fixed">
@@ -89,5 +91,5 @@
         </collision>
     </link>
-    <!--        <joint name="stoc_camera_joint" type="fixed">
+<!--        <joint name="stoc_camera_joint" type="fixed">
             <origin xyz="0 0 ${(stoc_height/2)+0.0254}" rpy="0 0 0" />
             <parent link="${parent}" />

Commit message: Added a computer box to erratic platform. Minor tweaks to size and locatin of head support.

File: arrg/ua_robots/erratic_description/urdf/erratic_base.xacro (robot description, xacro)
@@ -5,4 +5,5 @@
     xmlns:interface="http://playerstage.sourceforge.net/gazebo/xmlschema/#interface">
     <!-- Included URDF Files -->
+    <include filename="$(find erratic_description)/urdf/erratic_computer.xacro" />
     <include filename="$(find erratic_description)/urdf/erratic_wheel.xacro" />
     <include filename="$(find pr2_defs)/defs/materials.urdf.xacro" />
@@ -208,4 +209,5 @@
         </gazebo>
         <!-- MACRO INSTANTIATION -->
+        <erratic_computer parent="base_top_link"/>
         <erratic_wheel suffix="left" parent="base_link" reflect="1"/>
         <erratic_wheel suffix="right" parent="base_link" reflect="-1"/>

File: arrg/ua_robots/wubble_description/urdf/wubble.urdf.xacro (robot description, xacro)
@@ -13,6 +13,6 @@
     <!-- Properties (Constants) -->
     <property name="M_PI" value="3.14159"/>
-    <property name="support_radius" value="0.01" />
-    <property name="support_height" value="0.7578" />
+    <property name="support_radius" value="0.0065" />
+    <property name="support_height" value="0.7556" />
     <!-- MACRO INSTANTIATION -->
     <erratic />
@@ -24,5 +24,5 @@
     </tilting_hokuyo>
     <joint name="head_support_joint" type="fixed">
-        <origin xyz="0.0254 0 ${top_size_z/2}" />
+        <origin xyz="${top_size_x/2 - 0.16} 0 ${top_size_z/2}" />
         <parent link="base_top_link" />
         <child link="head_support_link" />
@@ -31,5 +31,5 @@
         <inertial>
             <mass value="0.1"/>
-            <origin xyz="0.0 0.0 0.0" rpy="0 0 0" />
+            <origin xyz="0.0 0.0 ${support_height/2}" rpy="0 0 0" />
             <inertia    ixx="0.1" ixy="0" ixz="0"
                         iyy="0.1" iyz="0"

Commit message: Add controllers for the arm joints. The arm is controllable now, yippee.

File: arrg/ua_robots/erratic_description/urdf/erratic_base.xacro (robot description, xacro)
@@ -26,15 +26,14 @@
         <link name="base_footprint">
             <inertial>
-                <mass value="1.0" />
+                <mass value="0.0001" />
                 <origin xyz="0 0 0" />
-                <inertia ixx="0.01" ixy="0.0" ixz="0.0"
-                         iyy="0.01" iyz="0.0"
-                         izz="0.01" />
-            </inertial>
-            <visual>
-                <!-- Hiding the base_footprint at the center of the body -->
+                <inertia ixx="0.0001" ixy="0.0" ixz="0.0"
+                         iyy="0.0001" iyz="0.0"
+                         izz="0.0001" />
+            </inertial>
+            <visual>
                 <origin xyz="0 0 0" rpy="0 0 0" />
                 <geometry>
-                    <box size="0.01 0.01 0.01" />
+                    <box size="0.001 0.001 0.001" />
                 </geometry>
                 <material name="Green" />

File: arrg/ua_robots/smart_arm_description/urdf/smart_arm.xacro (robot description, xacro)
@@ -10,4 +10,5 @@
             <child link="arm_base_link"/>
         </joint>
+        <!-- Arm's base link -->
         <link name="arm_base_link">
             <inertial>
@@ -37,8 +38,7 @@
             <child link="arm_shoulder_pan_link"/>
             <axis xyz="0 0 1"/>
-            <limit  lower="-1.22"
-                    upper="1.22"
-                    effort="100"
-                    velocity="2.33" />
+            <limit  lower="-1.22" upper="1.22" effort="100" velocity="1.17" />
+            <safety_controller k_position="100" k_velocity="15.0" soft_lower_limit="${-1.22+0.1}" soft_upper_limit="${1.22-0.1}" />
+            <dynamics damping="50" friction="1"/>
         </joint>
         <transmission type="SimpleTransmission" name="shoulder_pan_trans">
@@ -73,9 +73,8 @@
             <parent link="arm_shoulder_pan_link"/>
             <child link="arm_shoulder_tilt_link" />
-            <axis xyz="0 1 0"/>
-            <limit  lower="-1.972222"
-                    upper="1.04719755"
-                    effort="100"
-                    velocity="2.33" />
+            <axis xyz="0 -1 0"/>    <!-- not sure why I need negative number here to get proper z-direction -->
+            <limit  lower="-1.04719755" upper="1.972222" effort="100" velocity="1.17" />
+            <safety_controller k_position="100" k_velocity="15.0" soft_lower_limit="${-1.04719755+0.1}" soft_upper_limit="${1.972222-0.1}" />
+            <dynamics damping="50" friction="1"/>
         </joint>
         <link name="arm_shoulder_tilt_link">
@@ -110,10 +109,9 @@
             <parent link="arm_shoulder_tilt_link"/>
             <child link="arm_elbow_tilt_link" />
-            <axis xyz="0 1 0"/>
+            <axis xyz="0 -1 0"/>
             <!-- From -113 to 108 degrees -->
-            <limit  lower="-1.972222"
-                    upper="1.8849556"
-                    effort="100"
-                    velocity="2.33" />
+            <limit  lower="-1.972222" upper="1.8849556" effort="100" velocity="1.17" />
+            <dynamics damping="50" friction="1"/>
+            <safety_controller k_position="100" k_velocity="15.0" soft_lower_limit="${-1.972222+0.1}" soft_upper_limit="${1.8849556-0.1}" />
         </joint>
         <link name="arm_elbow_tilt_link">
@@ -148,10 +146,9 @@
             <parent link="arm_elbow_tilt_link"/>
             <child link="arm_wrist_rotate_link" />
-            <axis xyz="1 0 0"/>
+            <axis xyz="-1 0 0"/>
             <!-- From -150 to 150 degrees -->
-            <limit  lower="-2.6179939"
-                    upper="2.6179939"
-                    effort="100"
-                    velocity="2.33" />
+            <limit  lower="-2.6179939" upper="2.6179939" effort="100" velocity="1.17" />
+            <dynamics damping="50" friction="1"/>
+            <safety_controller k_position="100" k_velocity="15.0" soft_lower_limit="${-2.6179939+0.1}" soft_upper_limit="${2.6179939-0.1}" />
         </joint>
         <link name="arm_wrist_rotate_link">
@@ -188,8 +185,7 @@
             <axis xyz="0 0 1"/>
             <!-- From -20 to 20 degrees -->
-            <limit  lower="-0.3490658"
-                    upper="0.3490658"
-                    effort="100"
-                    velocity="2.33" />
+            <limit  lower="-0.3490658" upper="0.3490658" effort="100" velocity="1.17" />
+            <dynamics damping="50" friction="1"/>
+            <safety_controller k_position="100" k_velocity="15.0" soft_lower_limit="${-0.3490658+0.1}" soft_upper_limit="${0.3490658-0.1}" />
         </joint>
         <link name="arm_right_finger_link">
@@ -226,8 +222,7 @@
             <axis xyz="0 0 1"/>
             <!-- From -20 to 20 degrees -->
-            <limit  lower="-0.3490658"
-                    upper="0.3490658"
-                    effort="100"
-                    velocity="2.33" />
+            <limit  lower="-0.3490658" upper="0.3490658" effort="100" velocity="1.17" />
+            <dynamics damping="50" friction="1"/>
+            <safety_controller k_position="100" k_velocity="15.0" soft_lower_limit="${-0.3490658+0.1}" soft_upper_limit="${0.3490658-0.1}" />
         </joint>
         <link name="arm_left_finger_link">

File: arrg/ua_robots/wubble_description/urdf/wubble.urdf.xacro (robot description, xacro)
@@ -18,5 +18,5 @@
     <!-- CRUST CRAWLER SMART ARM ATTACHMENT -->
     <smart_arm parent="base_top_link" >
-        <origin xyz="${top_size_x/2 - 0.0575} 0 ${top_size_z/2 + 0.025}"/>
+        <origin xyz="${top_size_x/2 - 0.0575} 0 ${top_size_z/2 + 0.025}" rpy="0 0 0"/>
     </smart_arm>
     <!-- HOKUYO LASER ATTACHMENT -->
@@ -52,6 +52,6 @@
         <child link="hokuyo_mount_link" />
         <axis xyz="0 1 0" />
-        <limit lower="-0.1" upper="${M_PI/2}" effort="100" velocity="12.0" />
-        <safety_controller k_position="100" k_velocity="12.0" soft_lower_limit="${-0.1+0.1}" soft_upper_limit="${M_PI/3}" />-->
+        <limit lower="-0.1" upper="0.785398164" effort="100" velocity="12.0" />
+        <safety_controller k_position="100" k_velocity="15.0" soft_lower_limit="${-0.1+0.1}" soft_upper_limit="${0.785398164-0.1}" />
         <dynamics damping="50" friction="1"/>
     </joint>
@@ -143,6 +143,6 @@
         <child link="head_tilt_link" />
         <axis xyz="0 0 1" />
-        <limit lower="-3" upper="3" effort="100.0" velocity="4.0" />
-        <safety_controller k_position="100" k_velocity="4.0" soft_lower_limit="${-3+0.2}" soft_upper_limit="${3-0.2}" />
+        <limit lower="-1.570796327" upper="1.570796327" effort="100.0" velocity="1.17" />
+        <safety_controller k_position="100" k_velocity="15.0" soft_lower_limit="${-1.570796327+0.1}" soft_upper_limit="${1.570796327-0.1}" />
         <dynamics damping="50" friction="1"/>
     </joint>
@@ -177,7 +177,7 @@
         <parent link="head_tilt_link" />
         <child link="head_mount_link" />
-        <axis xyz="0 1 0" />
-        <limit lower="-1.0" upper="1.0" effort="100.0" velocity="4.0" />
-        <safety_controller k_position="100" k_velocity="4.0" soft_lower_limit="${-1.0+0.1}" soft_upper_limit="${1.0-0.1}" />
+        <axis xyz="0 -1 0" />
+        <limit lower="-1.221730476" upper="0.610865238" effort="100.0" velocity="1.17" />
+        <safety_controller k_position="100" k_velocity="15.0" soft_lower_limit="${-1.221730476+0.1}" soft_upper_limit="${0.610865238-0.1}" />
         <dynamics damping="50" friction="1"/>
     </joint>
