Commit message: Correct overhead_cam principal point and focal length in urdf, and correct tf in launch file.

File: arrg/ua_robots/overhead_cam_description/urdf/overhead_cam.urdf.xacro (robot description, xacro)
@@ -8,7 +8,7 @@
         <origin xyz="0 0 3" rpy="0 ${M_PI/2} 0"/>
         <parent link="world"/>
-        <child link="camera_link"/>
+        <child link="overhead_cam_link"/>
     </joint>
-    <link name="camera_link">
+    <link name="overhead_cam_link">
         <inertial>
           <mass value="0.001" />
@@ -31,9 +31,12 @@
         </collision>
     </link>
-    <gazebo reference="camera_link">
+    <property name="image_width" value="1024"/>
+    <property name="image_height" value="1024"/>
+    <property name="hfov" value="90"/>
+    <gazebo reference="overhead_cam_link">
         <sensor:camera name="overhead_cam_sensor">
-            <imageSize>1024 1024</imageSize>
+            <imageSize>${image_width} ${image_height}</imageSize>
             <imageFormat>PF_B8G8R8</imageFormat>
-            <hfov>90</hfov>
+            <hfov>${hfov}</hfov>
             <nearClip>0.1</nearClip>
             <farClip>100</farClip>
@@ -45,8 +48,9 @@
                 <cameraInfoTopicName>overhead_cam/camera_info</cameraInfoTopicName>
                 <frameName>overhead_cam_link</frameName>
-                <CxPrime>320.5</CxPrime>
-                <Cx>320.5</Cx>
-                <Cy>240.5</Cy>
-                <focal_length>320</focal_length>
+                <CxPrime>${(image_width+1)/2}</CxPrime>
+                <Cx>${(image_width+1)/2}</Cx>
+                <Cy>${(image_height+1)/2}</Cy>
+                <!-- focal_length = image_width / (2*tan(hfov_radian /2)) BUT tan(45 deg) = 1 -->
+                <focal_length>${image_width / 2}</focal_length>
                 <distortion_k1>0</distortion_k1>
                 <distortion_k2>0</distortion_k2>
@@ -58,5 +62,5 @@
         </sensor:camera>
     </gazebo>
-    <gazebo reference="camera_link">
+    <gazebo reference="overhead_cam_link">
         <material>Gazebo/Black</material>
     </gazebo>
