Commit message: Ahh, why not... added some meshes for camera mount, looks more like the real thing now.

File: arrg/ua_robots/smart_arm_description/urdf/smart_arm.xacro (robot description, xacro)
@@ -42,6 +42,6 @@
                     velocity="2.33" />
         </joint>
-        <transmission type="SimpleTransmission" name="arm_base_shoulder_trans">
-            <actuator name="arm_base_shoulder_motor" />
+        <transmission type="SimpleTransmission" name="shoulder_pan_trans">
+            <actuator name="shoulder_pan_motor" />
             <joint name="shoulder_pan_joint" />
             <mechanicalReduction>1.0</mechanicalReduction>

File: arrg/ua_robots/videre_stoc_description/urdf/videre_stoc.xacro (robot description, xacro)
@@ -110,5 +110,5 @@
             </inertial>
             <visual>
-                <origin xyz="0 0 0.03" rpy="0 0 0" />
+                <origin xyz="0 0 0.0215" rpy="0 0 0" />
                 <geometry>
                     <box size="${stoc_depth} ${stoc_width} ${stoc_height}" />
@@ -116,5 +116,5 @@
             </visual>
             <collision>
-                <origin xyz="0 0 0.03" rpy="0 0 0" />
+                <origin xyz="0 0 0.0215" rpy="0 0 0" />
                 <geometry>
                     <box size="${stoc_depth} ${stoc_width} ${stoc_height}" />
@@ -123,5 +123,5 @@
         </link>
         <joint name="stoc_back_joint" type="fixed">
-            <origin xyz="${-(stoc_depth/2)-(back_depth/2)} 0 0.03" rpy="0 0 0" />
+            <origin xyz="${-(stoc_depth/2)-(back_depth/2)} 0 0.0215" rpy="0 0 0" />
             <parent link="stoc_camera_link" />
             <child link="stoc_back_link"/>

File: arrg/ua_robots/wubble_description/urdf/wubble.urdf.xacro (robot description, xacro)
@@ -14,5 +14,5 @@
     <property name="M_PI" value="3.14159"/>
     <property name="support_radius" value="0.01" />
-    <property name="support_height" value="0.8128" />
+    <property name="support_height" value="0.7578" />
     <!-- MACRO INSTANTIATION -->
     <erratic />
@@ -23,11 +23,4 @@
         <origin xyz="0.15 0 ${-top_size_z - 0.05}" rpy="${M_PI} 0 0" />
     </tilting_hokuyo>
-    <stoc_camera name="stoc" parent="head_pan_link" />
-<!--    <joint name="laser_test_joint" type="fixed">-->
-<!--        <origin xyz="0.5 0.0 0.5" />-->
-<!--        <parent link="base_top_link" />-->
-<!--        <child link="hokuyo_link" />-->
-<!--    </joint>-->
-    <!-- Special Links -->
     <joint name="head_support_joint" type="fixed">
         <origin xyz="0.0254 0 ${top_size_z/2}" />
@@ -56,14 +49,37 @@
         </collision>
     </link>
-    <joint name="head_pan_joint" type="revolute">
+    <joint name="head_pan_support_joint" type="fixed">
         <origin xyz="0 0 ${support_height}" />
         <parent link="head_support_link" />
         <child link="head_pan_link" />
+    </joint>
+    <link name="head_pan_link">
+        <inertial>
+            <mass value="0.01"/>
+            <origin xyz="0.0 0.0 0.0" rpy="0 0 0" />
+            <inertia ixx="0.01" ixy="0" ixz="0"
+                     iyy="0.01" iyz="0"
+                     izz="0.01"/>
+        </inertial>
+        <visual>
+            <origin xyz="0 0 0.018" rpy="0 0 0"/>
+            <geometry>
+                <mesh filename="package://wubble_description/meshes/camera_pan.stl"/>
+            </geometry>
+        </visual>
+        <collision>
+            <origin xyz="0 0 0.018" rpy="0 0 0"/>
+            <geometry>
+                <mesh filename="package://wubble_description/meshes/camera_pan.stl"/>
+            </geometry>
+        </collision>
+    </link>
+    <joint name="head_pan_joint" type="revolute">
+        <origin xyz="0.0135 0 0.058" />
+        <parent link="head_pan_link" />
+        <child link="head_tilt_link" />
         <axis xyz="0 0 1" />
-<!--        <anchor xyz="0 0 0" />-->
-<!--        <limit effort="100" velocity="100" />-->
         <limit lower="0" upper="0" effort="100" velocity="1.0" />
         <dynamics damping="1" friction="1" />
-<!--        <safety_controller k_position="100" k_velocity="0.05" soft_lower_limit="${-0.785+0.0}" soft_upper_limit="${1.57-0.0}" />-->
     </joint>
     <transmission type="SimpleTransmission" name="head_pan_trans">
@@ -72,32 +88,56 @@
         <mechanicalReduction>6.0</mechanicalReduction>
     </transmission>
-    <link name="head_pan_link">
+    <link name="head_tilt_link">
         <inertial>
             <mass value="0.01"/>
             <origin xyz="0.0 0.0 0.0" rpy="0 0 0" />
-            <inertia ixx="0.01" ixy="0" ixz="0" iyy="0.01" iyz="0" izz="0.01"/>
+            <inertia ixx="0.01" ixy="0" ixz="0"
+                     iyy="0.01" iyz="0"
+                     izz="0.01"/>
         </inertial>
         <visual>
-            <origin xyz="0 0 0.0127" rpy="0 0 0"/>
+            <origin xyz="0 0 0" rpy="0 0 0"/>
             <geometry>
-                <box size="${2*support_radius} ${2*support_radius} 0.0254" />
+                <mesh filename="package://wubble_description/meshes/camera_tilt.stl"/>
+<!--                <box size="${2*support_radius} ${2*support_radius} 0.0254" />-->
             </geometry>
         </visual>
         <collision>
-            <origin xyz="0 0 0.0127" rpy="0 0 0"/>
+            <origin xyz="0 0 0" rpy="0 0 0"/>
             <geometry>
-                <box size="${2*support_radius} ${2*support_radius} 0.0254" />
+                <mesh filename="package://wubble_description/meshes/camera_tilt.stl"/>
+<!--                <box size="${2*support_radius} ${2*support_radius} 0.0254" />-->
             </geometry>
         </collision>
     </link>
-<!--        <joint name="stoc_camera_joint" type="fixed">
-            <origin xyz="0 0 ${(stoc_height/2)+0.0254}" rpy="0 0 0" />
-            <parent link="${parent}" />
-            <child link="stoc_camera_link"/>
-        </joint>
--->
+    <joint name="head_mount_joint" type="fixed">
+        <origin xyz="-0.019 0 0.043" />
+        <parent link="head_tilt_link" />
+        <child link="head_mount_link" />
+    </joint>
+    <link name="head_mount_link">
+        <inertial>
+            <mass value="0.01"/>
+            <origin xyz="0.0 0.0 0.0" rpy="0 0 0" />
+            <inertia ixx="0.01" ixy="0" ixz="0"
+                     iyy="0.01" iyz="0"
+                     izz="0.01"/>
+        </inertial>
+        <visual>
+            <origin xyz="0 0 0" rpy="0 0 0"/>
+            <geometry>
+                <mesh filename="package://wubble_description/meshes/camera_mount.stl"/>
+            </geometry>
+        </visual>
+        <collision>
+            <origin xyz="0 0 0" rpy="0 0 0"/>
+            <geometry>
+                <mesh filename="package://wubble_description/meshes/camera_mount.stl"/>
+            </geometry>
+        </collision>
+    </link>
     <joint name="head_tilt_joint" type="revolute">
-        <origin xyz="0 0 ${0.0254}" rpy="0 0 0" />
-        <parent link="head_pan_link"/>
+        <origin xyz="0 0 0.023" rpy="0 0 0" />
+        <parent link="head_mount_link"/>
         <child link="stoc_camera_link"/>
         <axis xyz="0 1 0" />
@@ -113,8 +153,6 @@
         <mechanicalReduction>3.0</mechanicalReduction>
     </transmission>
+    <stoc_camera name="stoc" parent="head_mount_link" />
     <!-- GAZEBO MATERIALS -->
-<!--    <gazebo reference="base_laser_link">-->
-<!--        <material>PR2/Red</material>-->
-<!--    </gazebo>-->
     <gazebo reference="head_support_link">
         <material>Wubble/BrassScratched</material>
@@ -123,3 +161,9 @@
         <material>PR2/Black</material>
     </gazebo>
+    <gazebo reference="head_tilt_link">
+        <material>PR2/Black</material>
+    </gazebo>
+    <gazebo reference="head_mount_link">
+        <material>PR2/White</material>
+    </gazebo>
 </robot>

Commit message: Make simulated arm's gripper joint limits exactly the same as the real arm.

File: arrg/ua_robots/smart_arm_description/urdf/smart_arm.xacro (robot description, xacro)
@@ -61,7 +61,7 @@
             <axis xyz="0 0 1"/>
             <!-- From 14 to -45 degrees -->
-            <limit  lower="-0.785398163" upper="0.244346095" effort="300" velocity="1.17" />
-            <dynamics damping="50" friction="1"/>
-            <safety_controller k_position="100" k_velocity="15.0" soft_lower_limit="${-0.785398163+0.1}" soft_upper_limit="${0.244346095-0.1}" />
+            <limit  lower="-0.838576116" upper="0.245436912" effort="300" velocity="1.17" />
+            <dynamics damping="50" friction="1"/>
+            <safety_controller k_position="100" k_velocity="15.0" soft_lower_limit="${-0.838576116+0.1}" soft_upper_limit="${0.245436912-0.1}" />
         </joint>
         <!-- Gripper left finger joint -->
@@ -72,7 +72,7 @@
             <axis xyz="0 0 1"/>
             <!-- From -14 to 45 degrees -->
-            <limit  lower="-0.244346095" upper="0.785398163" effort="300" velocity="1.17" />
-            <dynamics damping="50" friction="1"/>
-            <safety_controller k_position="100" k_velocity="15.0" soft_lower_limit="${-0.244346095+0.1}" soft_upper_limit="${0.785398163-0.1}" />
+            <limit  lower="-0.240323643" upper="0.843689385" effort="300" velocity="1.17" />
+            <dynamics damping="50" friction="1"/>
+            <safety_controller k_position="100" k_velocity="15.0" soft_lower_limit="${-0.240323643+0.1}" soft_upper_limit="${0.843689385-0.1}" />
         </joint>
         <!-- ****** LINK DEFINITIONS ****** -->
