Commit message: Fix head tilt joint

File: arrg/ua_robots/wubble_description/urdf/wubble.urdf.xacro (robot description, xacro)
@@ -100,5 +100,4 @@
             <geometry>
                 <mesh filename="package://wubble_description/meshes/camera_tilt.stl"/>
-<!--                <box size="${2*support_radius} ${2*support_radius} 0.0254" />-->
             </geometry>
         </visual>
@@ -107,13 +106,23 @@
             <geometry>
                 <mesh filename="package://wubble_description/meshes/camera_tilt.stl"/>
-<!--                <box size="${2*support_radius} ${2*support_radius} 0.0254" />-->
             </geometry>
         </collision>
     </link>
-    <joint name="head_mount_joint" type="fixed">
+    <joint name="head_tilt_joint" type="revolute">
         <origin xyz="-0.019 0 0.043" />
         <parent link="head_tilt_link" />
         <child link="head_mount_link" />
+        <axis xyz="0 1 0" />
+        <limit lower="-0.5" upper="1.00" effort="100" velocity="2.00" />
+        <safety_controller k_position="100" k_velocity="0.05" soft_lower_limit="${-0.785+0.0}" soft_upper_limit="${1.57-0.0}" />
+        <!-- hold both reference_position and upper/lower for tick-tock, remove reference_positiion after verifying upper/lower works with calibration controllers.  if search velocity in pr2_calibration_controllers.yaml is +, the reference_position is rising, if - then it is falling -->
+        <calibration reference_position="-.35" falling="-.35" />
+        <dynamics damping="0.008" />
     </joint>
+    <transmission type="SimpleTransmission" name="head_tilt_trans">
+        <actuator name="head_tilt_motor" />
+        <joint name="head_tilt_joint" />
+        <mechanicalReduction>3.0</mechanicalReduction>
+    </transmission>
     <link name="head_mount_link">
         <inertial>
@@ -137,20 +146,9 @@
         </collision>
     </link>
-    <joint name="head_tilt_joint" type="revolute">
+    <joint name="head_mount_joint" type="fixed">
         <origin xyz="0 0 0.023" rpy="0 0 0" />
         <parent link="head_mount_link"/>
         <child link="stoc_camera_link"/>
-        <axis xyz="0 1 0" />
-        <limit lower="-0.5" upper="1.00" effort="100" velocity="2.00" />
-        <safety_controller k_position="100" k_velocity="0.05" soft_lower_limit="${-0.785+0.0}" soft_upper_limit="${1.57-0.0}" />
-        <!-- hold both reference_position and upper/lower for tick-tock, remove reference_positiion after verifying upper/lower works with calibration controllers.  if search velocity in pr2_calibration_controllers.yaml is +, the reference_position is rising, if - then it is falling -->
-        <calibration reference_position="-.35" falling="-.35" />
-        <dynamics damping="0.008" />
     </joint>
-    <transmission type="SimpleTransmission" name="head_tilt_trans">
-        <actuator name="head_tilt_motor" />
-        <joint name="head_tilt_joint" />
-        <mechanicalReduction>3.0</mechanicalReduction>
-    </transmission>
     <stoc_camera name="stoc" parent="head_mount_link" />
     <!-- GAZEBO MATERIALS -->

Commit message: Created new wubble_teleop in ua_apps package (named after pr2_apps). Also, adjusted controllers for head so they are close to serviceable.

File: arrg/ua_robots/wubble_description/urdf/wubble.urdf.xacro (robot description, xacro)
@@ -79,11 +79,12 @@
         <child link="head_tilt_link" />
         <axis xyz="0 0 1" />
-        <limit lower="0" upper="0" effort="100" velocity="1.0" />
-        <dynamics damping="1" friction="1" />
+        <limit lower="-3" upper="3" effort="100.0" velocity="3.0" />
+        <safety_controller k_position="100" k_velocity="1.5" soft_lower_limit="${-3+0.2}" soft_upper_limit="${3-0.2}" />
+        <dynamics damping="100" friction="100"/>
     </joint>
     <transmission type="SimpleTransmission" name="head_pan_trans">
         <actuator name="head_pan_motor" />
         <joint name="head_pan_joint" />
-        <mechanicalReduction>6.0</mechanicalReduction>
+        <mechanicalReduction>1.0</mechanicalReduction>
     </transmission>
     <link name="head_tilt_link">
@@ -113,14 +114,14 @@
         <child link="head_mount_link" />
         <axis xyz="0 1 0" />
-        <limit lower="-0.5" upper="1.00" effort="100" velocity="2.00" />
-        <safety_controller k_position="100" k_velocity="0.05" soft_lower_limit="${-0.785+0.0}" soft_upper_limit="${1.57-0.0}" />
+        <limit lower="-0.5" upper="1.00" effort="100.0" velocity="2.0" />
+        <safety_controller k_position="100" k_velocity="1.5" soft_lower_limit="${-0.5+0.1}" soft_upper_limit="${1.0-0.1}" />
         <!-- hold both reference_position and upper/lower for tick-tock, remove reference_positiion after verifying upper/lower works with calibration controllers.  if search velocity in pr2_calibration_controllers.yaml is +, the reference_position is rising, if - then it is falling -->
         <calibration reference_position="-.35" falling="-.35" />
-        <dynamics damping="0.008" />
+        <dynamics damping="100" friction="100"/>
     </joint>
     <transmission type="SimpleTransmission" name="head_tilt_trans">
         <actuator name="head_tilt_motor" />
         <joint name="head_tilt_joint" />
-        <mechanicalReduction>3.0</mechanicalReduction>
+        <mechanicalReduction>1.0</mechanicalReduction>
     </transmission>
     <link name="head_mount_link">
@@ -132,4 +133,11 @@
                      izz="0.01"/>
         </inertial>
+<!--         <inertial>-->
+<!--        <mass value="1.749727" />-->
+<!--        <origin xyz="0.041935 0.003569 0.028143" rpy="0 0 0" />-->
+<!--        <inertia ixx="0.010602303435"  ixy="-0.000408814235"  ixz="0.00198303894"-->
+<!--                 iyy="0.011874383747"  iyz="0.000197908779"-->
+<!--                 izz="0.005516790626" />-->
+<!--      </inertial>-->
         <visual>
             <origin xyz="0 0 0" rpy="0 0 0"/>

Commit message: Somewhat faster pan/tilt controller.

File: arrg/ua_robots/wubble_description/urdf/wubble.urdf.xacro (robot description, xacro)
@@ -79,7 +79,7 @@
         <child link="head_tilt_link" />
         <axis xyz="0 0 1" />
-        <limit lower="-3" upper="3" effort="100.0" velocity="3.0" />
-        <safety_controller k_position="100" k_velocity="1.5" soft_lower_limit="${-3+0.2}" soft_upper_limit="${3-0.2}" />
-        <dynamics damping="100" friction="100"/>
+        <limit lower="-3" upper="3" effort="100.0" velocity="4.0" />
+        <safety_controller k_position="100" k_velocity="4.0" soft_lower_limit="${-3+0.2}" soft_upper_limit="${3-0.2}" />
+        <dynamics damping="50" friction="1"/>
     </joint>
     <transmission type="SimpleTransmission" name="head_pan_trans">
@@ -114,9 +114,7 @@
         <child link="head_mount_link" />
         <axis xyz="0 1 0" />
-        <limit lower="-0.5" upper="1.00" effort="100.0" velocity="2.0" />
-        <safety_controller k_position="100" k_velocity="1.5" soft_lower_limit="${-0.5+0.1}" soft_upper_limit="${1.0-0.1}" />
-        <!-- hold both reference_position and upper/lower for tick-tock, remove reference_positiion after verifying upper/lower works with calibration controllers.  if search velocity in pr2_calibration_controllers.yaml is +, the reference_position is rising, if - then it is falling -->
-        <calibration reference_position="-.35" falling="-.35" />
-        <dynamics damping="100" friction="100"/>
+        <limit lower="-1.0" upper="1.0" effort="100.0" velocity="4.0" />
+        <safety_controller k_position="100" k_velocity="4.0" soft_lower_limit="${-1.0+0.1}" soft_upper_limit="${1.0-0.1}" />
+        <dynamics damping="50" friction="1"/>
     </joint>
     <transmission type="SimpleTransmission" name="head_tilt_trans">
@@ -133,11 +131,4 @@
                      izz="0.01"/>
         </inertial>
-<!--         <inertial>-->
-<!--        <mass value="1.749727" />-->
-<!--        <origin xyz="0.041935 0.003569 0.028143" rpy="0 0 0" />-->
-<!--        <inertia ixx="0.010602303435"  ixy="-0.000408814235"  ixz="0.00198303894"-->
-<!--                 iyy="0.011874383747"  iyz="0.000197908779"-->
-<!--                 izz="0.005516790626" />-->
-<!--      </inertial>-->
         <visual>
             <origin xyz="0 0 0" rpy="0 0 0"/>

Commit message: various bits and pieces from the robot. Tweaked the position of the laser and camera in URDF

File: arrg/ua_robots/wubble_description/urdf/wubble.urdf.xacro (robot description, xacro)
@@ -21,5 +21,5 @@
     <!-- HOKUYO LASER ATTACHMENT -->
     <joint name="laser_support_joint" type="fixed">
-        <origin xyz="${top_size_x/2 - 0.016} 0 -${top_size_z/2}" rpy="${M_PI} 0 0" />
+        <origin xyz="${top_size_x/2 - 0.016} 0.02 -${top_size_z/2}" rpy="${M_PI} 0 0" />
         <parent link="base_top_link"/>
         <child link="hokuyo_tilt_link"/>
@@ -86,5 +86,5 @@
     <!-- VIDERE STOC STEREO CAMERA ATTACHMENT -->
     <joint name="head_support_joint" type="fixed">
-        <origin xyz="${top_size_x/2 - 0.16} 0 ${top_size_z/2}" />
+        <origin xyz="${top_size_x/2 - 0.17} 0 ${top_size_z/2}" />
         <parent link="base_top_link" />
         <child link="head_support_link" />

Commit message: Added IMU to the Wubble robot model.

File: arrg/ua_robots/wubble_description/urdf/wubble.urdf.xacro (robot description, xacro)
@@ -9,4 +9,5 @@
     <include filename="$(find hokuyo_urg_description)/urdf/hokuyo_urg.xacro" />
     <include filename="$(find videre_stoc_description)/urdf/videre_stoc.xacro" />
+    <include filename="$(find chr_6dm_imu_description)/urdf/chrobotics_chr_6dm_imu.urdf.xacro" />
     <!-- Properties (Constants) -->
     <property name="M_PI" value="3.14159"/>
@@ -19,4 +20,8 @@
         <origin xyz="${top_size_x/2 - 0.0575} 0 ${top_size_z/2 + 0.025}" rpy="0 0 0"/>
     </smart_arm>
+    <!-- CHR-6dm IMU ATTACHMENT -->
+    <chrobotics_chr_6dm_imu name="imu" parent="base_top_link" imu_topic="imu/data" update_rate="100.0" stdev="0.00017" >
+        <origin xyz="0.0 0.1 ${top_size_z/2}" rpy="0 0 0" />
+    </chrobotics_chr_6dm_imu>
     <!-- HOKUYO LASER ATTACHMENT -->
     <joint name="laser_support_joint" type="fixed">
