Commit message: Added all params necessary to run arm navigation on wubble robot and example launch file.

File: arrg/ua_robots/wubble_description/urdf/wubble2.urdf.xacro (robot description, xacro)
@@ -156,6 +156,6 @@
         <child link="neck_tilt_link"/>
         <axis xyz="0 1 0" />
-        <limit lower="0" upper="1.57" effort="100" velocity="12.0" />
-        <safety_controller k_position="100" k_velocity="15.0" soft_lower_limit="${0}" soft_upper_limit="${1.57}" />
+        <limit lower="-1.57" upper="1.57" effort="100" velocity="12.0" />
+        <safety_controller k_position="100" k_velocity="15.0" soft_lower_limit="${-1.57}" soft_upper_limit="${1.57}" />
         <dynamics damping="50" friction="1"/>
     </joint>
@@ -210,68 +210,7 @@
         <origin xyz="0.01148 0 0.02635" rpy="0 0 0" />
     </hokuyo_urg>
-    <!-- HOKUYO LASER ATTACHMENT -->
-    <joint name="laser_support_joint" type="fixed">
-        <origin xyz="${top_size_x/2 - 0.016} 0 -${top_size_z/2}" rpy="${M_PI} 0 0" />
-        <parent link="base_top_link"/>
-        <child link="hokuyo_tilt_link"/>
-    </joint>
-    <link name="hokuyo_tilt_link">
-        <inertial>
-            <mass value="0.1"/>
-            <origin xyz="0 0 0" rpy="0 0 0" />
-            <inertia ixx="0.01" ixy="0" ixz="0"
-                     iyy="0.01" iyz="0"
-                     izz="0.01"/>
-        </inertial>
-        <visual>
-            <origin xyz="0 0 0" rpy="0 0 0"/>
-            <geometry>
-                <mesh filename="package://wubble_description/meshes/camera_tilt.stl"/>
-            </geometry>
-        </visual>
-        <collision>
-            <origin xyz="0 0 0" rpy="0 0 0"/>
-            <geometry>
-                <mesh filename="package://wubble_description/meshes/camera_tilt.stl"/>
-            </geometry>
-        </collision>
-    </link>
-    <joint name="hokuyo_tilt_joint" type="revolute">
-        <origin xyz="-0.019 0 0.043" />
-        <parent link="hokuyo_tilt_link" />
-        <child link="hokuyo_mount_link" />
-        <axis xyz="0 1 0" />
-        <limit lower="-0.6" upper="0.785398164" effort="100" velocity="12.0" />
-        <safety_controller k_position="100" k_velocity="15.0" soft_lower_limit="${-0.6+0.1}" soft_upper_limit="${0.785398164-0.1}" />
-        <dynamics damping="50" friction="1"/>
-    </joint>
-    <transmission type="pr2_mechanism_model/SimpleTransmission" name="hokuyo_tilt_trans">
-        <actuator name="hokuyo_tilt_motor" />
-        <joint name="hokuyo_tilt_joint" />
-        <mechanicalReduction>1.0</mechanicalReduction>
-    </transmission>
-    <link name="hokuyo_mount_link">
-        <inertial>
-            <mass value="0.01"/>
-            <origin xyz="0 0 0" rpy="0 0 0" />
-            <inertia ixx="0.01" ixy="0" ixz="0"
-                     iyy="0.01" iyz="0"
-                     izz="0.01"/>
-        </inertial>
-        <visual>
-            <origin xyz="0 0 0" rpy="0 0 0"/>
-            <geometry>
-                <mesh filename="package://wubble_description/meshes/camera_mount.stl"/>
-            </geometry>
-        </visual>
-        <collision>
-            <origin xyz="0 0 0" rpy="0 0 0"/>
-            <geometry>
-                <mesh filename="package://wubble_description/meshes/camera_mount.stl"/>
-            </geometry>
-        </collision>
-    </link>
-    <hokuyo_urg name="base_scan" parent="hokuyo_mount_link">
-        <origin xyz="0 0 0.023" rpy="0 0 0" />
+    <!-- BASE LASER ATTACHMENT -->
+    <hokuyo_urg name="base_scan" parent="base_top_link">
+        <origin xyz="${top_size_x/2 - 0.01 - 0.04} 0 -${top_size_z/2}" rpy="${M_PI} 0 0" />
     </hokuyo_urg>
     <!-- GAZEBO MATERIALS -->
@@ -291,10 +230,4 @@
         <material>SmartArm/GunMetalBrushedAluminum</material>
     </gazebo>
-    <gazebo reference="hokuyo_tilt_link">
-        <material>Erratic/Black</material>
-    </gazebo>
-    <gazebo reference="hokuyo_mount_link">
-        <material>SmartArm/GunMetalBrushedAluminum</material>
-    </gazebo>
     <gazebo reference="platform_link">
         <material>Erratic/White</material>

Commit message: Move laser to proper position.

File: arrg/ua_robots/wubble_description/urdf/wubble2.urdf.xacro (robot description, xacro)
@@ -214,5 +214,5 @@
     </transmission>
     <hokuyo_urg name="neck_scan" parent="neck_tilt_link">
-        <origin xyz="0.01148 0 0.02635" rpy="0 0 0" />
+        <origin xyz="0 -0.0056 0.02635" rpy="0 0 0" />
     </hokuyo_urg>
     <!-- BASE LASER ATTACHMENT -->

Commit message: Move laser up to where it actually is on the robot, change velocity limits for trajectories, faster is smoother.

File: arrg/ua_robots/wubble_description/urdf/wubble2.urdf.xacro (robot description, xacro)
@@ -151,5 +151,5 @@
     <!-- NECK TILTING LASER ATTACHMENT -->
     <joint name="neck_support_joint" type="fixed">
-        <origin xyz="0.0254 0 0.6001" rpy="0 0 0" />
+        <origin xyz="0.0254 0 0.6411" rpy="0 0 0" />
         <parent link="platform_link"/>
         <child link="neck_support_link"/>

Commit message: Add swissranger models and urdf and use it on the wubble model.

File: arrg/ua_robots/wubble_description/urdf/wubble2.urdf.xacro (robot description, xacro)
@@ -8,4 +8,5 @@
     <include filename="$(find hokuyo_urg_description)/urdf/hokuyo_urg.xacro" />
     <include filename="$(find wubble_arm_description)/urdf/wubble_arm.xacro" />
+    <include filename="$(find swissranger_camera_description)/urdf/swissranger_camera.xacro" />
     <include filename="$(find videre_stoc_description)/urdf/videre_stereo_6cm.xacro" />
     <!-- Properties (Constants) -->
@@ -43,10 +44,10 @@
     <!-- WUBBLE HEAD ATTACHMENT -->
     <joint name="head_base_joint" type="fixed">
-        <origin xyz="0.0254 0 0.8001" rpy="0 0 0" />
+        <origin xyz="0.0254 0 ${0.8001-0.019}" rpy="0 0 0" />
         <parent link="platform_link"/>
         <child link="head_base_link"/>
     </joint>
     <joint name="head_pan_joint" type="revolute">
-        <origin xyz="0.0415 0 0.004" rpy="0 0 0" />
+        <origin xyz="0.0545 0 0.026" rpy="0 0 0" />
         <parent link="head_base_link"/>
         <child link="head_pan_link"/>
@@ -57,5 +58,5 @@
     </joint>
     <joint name="head_tilt_joint" type="revolute">
-        <origin xyz="0 0 0.0415" rpy="0 0 0" />
+        <origin xyz="0.06506 0 0.06147" rpy="0 0 0" />
         <parent link="head_pan_link"/>
         <child link="head_tilt_link"/>
@@ -141,7 +142,11 @@
         <mechanicalReduction>1.0</mechanicalReduction>
     </transmission>
+    <!-- SWISSRANGER CAMERA ATTACHMENT -->
+    <swissranger_camera name="swissranger" parent="head_tilt_link">
+        <origin xyz="0.0125 0 0.036" rpy="${M_PI} 0 0" />
+    </swissranger_camera>
     <!-- VIDERE STEREO CAMERA ATTACHMENT -->
     <videre_stereo_6cm name="stoc" parent="head_tilt_link" >
-        <origin xyz="0.01148 0 0.02635" rpy="0 0 0" />
+        <origin xyz="0.01148 0 0.037" rpy="0 0 0" />
     </videre_stereo_6cm>
     <!-- WUBBLE ARM ATTACHMENT -->
@@ -197,12 +202,12 @@
             <origin xyz="0 0 0" rpy="0 0 0"/>
             <geometry>
-                <mesh filename="package://wubble_description/meshes/head_tilt_link.stl"/>
-            </geometry>
-            <material name="GunMetalBrushedAluminum" />
-        </visual>
-        <collision>
-            <origin xyz="0 0 0" rpy="0 0 0"/>
-            <geometry>
-                <mesh filename="package://wubble_description/meshes/head_tilt_link.stl"/>
+                <mesh filename="package://wubble_description/meshes/ax12_45_bracket.stl"/>
+            </geometry>
+            <material name="GunMetalBrushedAluminum" />
+        </visual>
+        <collision>
+            <origin xyz="0 0 0" rpy="0 0 0"/>
+            <geometry>
+                <mesh filename="package://wubble_description/meshes/ax12_45_bracket.stl"/>
             </geometry>
         </collision>

Commit message: Position stereo camera correctly.

File: arrg/ua_robots/wubble_description/urdf/wubble2.urdf.xacro (robot description, xacro)
@@ -148,5 +148,5 @@
     <!-- VIDERE STEREO CAMERA ATTACHMENT -->
     <videre_stereo_6cm name="stoc" parent="head_tilt_link" >
-        <origin xyz="0.01148 0 0.037" rpy="0 0 0" />
+        <origin xyz="0.03 0 ${0.036 + 0.016}" rpy="0 0 0" />
     </videre_stereo_6cm>
     <!-- WUBBLE ARM ATTACHMENT -->

Commit message: Move neck laser down a bit, was sitting too high in the model.

File: arrg/ua_robots/wubble_description/urdf/wubble2.urdf.xacro (robot description, xacro)
@@ -156,5 +156,5 @@
     <!-- NECK TILTING LASER ATTACHMENT -->
     <joint name="neck_support_joint" type="fixed">
-        <origin xyz="0.0254 0 0.6411" rpy="0 0 0" />
+        <origin xyz="0.0254 0 0.628" rpy="0 0 0" />
         <parent link="platform_link"/>
         <child link="neck_support_link"/>

Commit message: point to stl models instead of dae

File: arrg/ua_robots/wubble_description/urdf/wubble2.urdf.xacro (robot description, xacro)
@@ -31,5 +31,5 @@
             <origin xyz="0 0 0" rpy="0 0 0"/>
             <geometry>
-                <mesh filename="package://wubble_description/meshes/collada/wubble2_platform.dae"/>
+                <mesh filename="package://wubble_description/meshes/wubble2_platform.stl"/>
             </geometry>
             <material name="White" />
@@ -38,5 +38,5 @@
             <origin xyz="0 0 0" rpy="0 0 0"/>
             <geometry>
-                <mesh filename="package://wubble_description/meshes/collada/wubble2_platform.dae"/>
+                <mesh filename="package://wubble_description/meshes/wubble2_platform.stl"/>
             </geometry>
         </collision>
@@ -77,12 +77,12 @@
             <origin xyz="0 0 0" rpy="0 0 0"/>
             <geometry>
-                <mesh filename="package://wubble_description/meshes/collada/head_base_link.dae"/>
-            </geometry>
-            <material name="GunMetalBrushedAluminum" />
-        </visual>
-        <collision>
-            <origin xyz="0 0 0" rpy="0 0 0"/>
-            <geometry>
-                <mesh filename="package://wubble_description/meshes/collada/head_base_link.dae"/>
+                <mesh filename="package://wubble_description/meshes/head_base_link.stl"/>
+            </geometry>
+            <material name="GunMetalBrushedAluminum" />
+        </visual>
+        <collision>
+            <origin xyz="0 0 0" rpy="0 0 0"/>
+            <geometry>
+                <mesh filename="package://wubble_description/meshes/head_base_link.stl"/>
             </geometry>
         </collision>
@@ -99,12 +99,12 @@
             <origin xyz="0 0 0" rpy="0 0 0"/>
             <geometry>
-                <mesh filename="package://wubble_description/meshes/collada/head_pan_link.dae"/>
-            </geometry>
-            <material name="GunMetalBrushedAluminum" />
-        </visual>
-        <collision>
-            <origin xyz="0 0 0" rpy="0 0 0"/>
-            <geometry>
-                <mesh filename="package://wubble_description/meshes/collada/head_pan_link.dae"/>
+                <mesh filename="package://wubble_description/meshes/head_pan_link.stl"/>
+            </geometry>
+            <material name="GunMetalBrushedAluminum" />
+        </visual>
+        <collision>
+            <origin xyz="0 0 0" rpy="0 0 0"/>
+            <geometry>
+                <mesh filename="package://wubble_description/meshes/head_pan_link.stl"/>
             </geometry>
         </collision>
@@ -121,12 +121,12 @@
             <origin xyz="0 0 0" rpy="0 0 0"/>
             <geometry>
-                <mesh filename="package://wubble_description/meshes/collada/head_tilt_link.dae"/>
-            </geometry>
-            <material name="GunMetalBrushedAluminum" />
-        </visual>
-        <collision>
-            <origin xyz="0 0 0" rpy="0 0 0"/>
-            <geometry>
-                <mesh filename="package://wubble_description/meshes/collada/head_tilt_link.dae"/>
+                <mesh filename="package://wubble_description/meshes/head_tilt_link.stl"/>
+            </geometry>
+            <material name="GunMetalBrushedAluminum" />
+        </visual>
+        <collision>
+            <origin xyz="0 0 0" rpy="0 0 0"/>
+            <geometry>
+                <mesh filename="package://wubble_description/meshes/head_tilt_link.stl"/>
             </geometry>
         </collision>
@@ -180,12 +180,12 @@
             <origin xyz="0 0 0" rpy="0 0 0"/>
             <geometry>
-                <mesh filename="package://wubble_description/meshes/collada/neck_laser_support_link.dae"/>
-            </geometry>
-            <material name="GunMetalBrushedAluminum" />
-        </visual>
-        <collision>
-            <origin xyz="0 0 0" rpy="0 0 0"/>
-            <geometry>
-                <mesh filename="package://wubble_description/meshes/collada/neck_laser_support_link.dae"/>
+                <mesh filename="package://wubble_description/meshes/neck_laser_support_link.stl"/>
+            </geometry>
+            <material name="GunMetalBrushedAluminum" />
+        </visual>
+        <collision>
+            <origin xyz="0 0 0" rpy="0 0 0"/>
+            <geometry>
+                <mesh filename="package://wubble_description/meshes/neck_laser_support_link.stl"/>
             </geometry>
         </collision>
@@ -202,12 +202,12 @@
             <origin xyz="0 0 0" rpy="0 0 0"/>
             <geometry>
-                <mesh filename="package://wubble_description/meshes/collada/ax12_45_bracket.dae"/>
-            </geometry>
-            <material name="GunMetalBrushedAluminum" />
-        </visual>
-        <collision>
-            <origin xyz="0 0 0" rpy="0 0 0"/>
-            <geometry>
-                <mesh filename="package://wubble_description/meshes/collada/ax12_45_bracket.dae"/>
+                <mesh filename="package://wubble_description/meshes/ax12_45_bracket.stl"/>
+            </geometry>
+            <material name="GunMetalBrushedAluminum" />
+        </visual>
+        <collision>
+            <origin xyz="0 0 0" rpy="0 0 0"/>
+            <geometry>
+                <mesh filename="package://wubble_description/meshes/ax12_45_bracket.stl"/>
             </geometry>
         </collision>

Commit message: Modify velocity limits for all arm joints, tweak neck laser z position, add IMU to Wubble2 urdf, move Swissranger back by 1.95cm

File: arrg/ua_robots/wubble_description/urdf/wubble2.urdf.xacro (robot description, xacro)
@@ -10,4 +10,5 @@
     <include filename="$(find swissranger_camera_description)/urdf/swissranger_camera.xacro" />
     <include filename="$(find videre_stoc_description)/urdf/videre_stereo_6cm.xacro" />
+    <include filename="$(find chr_6dm_imu_description)/urdf/chrobotics_chr_6dm_imu.urdf.xacro" />
     <!-- Properties (Constants) -->
     <property name="M_PI" value="3.14159"/>
@@ -42,4 +43,8 @@
         </collision>
     </link>
+    <!-- CHR-6dm IMU ATTACHMENT -->
+    <chrobotics_chr_6dm_imu name="imu" parent="platform_link" imu_topic="imu/data" update_rate="120.0" stdev="0.00017" >
+        <origin xyz="0 0 1.0" rpy="0 0 0" />
+    </chrobotics_chr_6dm_imu>
     <!-- WUBBLE HEAD ATTACHMENT -->
     <joint name="head_base_joint" type="fixed">
@@ -144,5 +149,5 @@
     <!-- SWISSRANGER CAMERA ATTACHMENT -->
     <swissranger_camera name="swissranger" parent="head_tilt_link">
-        <origin xyz="0.0195 -0.004 0.1235" rpy="${M_PI} 0 0" />
+        <origin xyz="0.0 -0.004 0.1235" rpy="${M_PI} 0 0" />
     </swissranger_camera>
     <!-- VIDERE STEREO CAMERA ATTACHMENT -->
@@ -156,5 +161,5 @@
     <!-- NECK TILTING LASER ATTACHMENT -->
     <joint name="neck_support_joint" type="fixed">
-        <origin xyz="0.0254 0 0.628" rpy="0 0 0" />
+        <origin xyz="0.0254 0 0.61" rpy="0 0 0" />
         <parent link="platform_link"/>
         <child link="neck_support_link"/>

Commit message: update wubble2 model with new neck_tilt assembly

File: arrg/ua_robots/wubble_description/urdf/wubble2.urdf.xacro (robot description, xacro)
@@ -161,10 +161,10 @@
     <!-- NECK TILTING LASER ATTACHMENT -->
     <joint name="neck_support_joint" type="fixed">
-        <origin xyz="0.0254 0 0.61" rpy="0 0 0" />
+        <origin xyz="0.0254 0 0.655" rpy="0 0 0" />
         <parent link="platform_link"/>
         <child link="neck_support_link"/>
     </joint>
     <joint name="neck_tilt_joint" type="revolute">
-        <origin xyz="0.0415 0 0.016" rpy="0 0 0" />
+        <origin xyz="0.0316 0 0" rpy="0 0 0" />
         <parent link="neck_support_link"/>
         <child link="neck_tilt_link"/>
@@ -207,12 +207,12 @@
             <origin xyz="0 0 0" rpy="0 0 0"/>
             <geometry>
-                <mesh filename="package://wubble_description/meshes/ax12_45_bracket.stl"/>
-            </geometry>
-            <material name="GunMetalBrushedAluminum" />
-        </visual>
-        <collision>
-            <origin xyz="0 0 0" rpy="0 0 0"/>
-            <geometry>
-                <mesh filename="package://wubble_description/meshes/collada/ax12_45_bracket.dae"/>
+                <mesh filename="package://wubble_description/meshes/neck_tilt_link.stl"/>
+            </geometry>
+            <material name="GunMetalBrushedAluminum" />
+        </visual>
+        <collision>
+            <origin xyz="0 0 0" rpy="0 0 0"/>
+            <geometry>
+                <mesh filename="package://wubble_description/meshes/collada/neck_tilt_link.dae"/>
             </geometry>
         </collision>
@@ -224,5 +224,5 @@
     </transmission>
     <hokuyo_urg name="neck_scan" parent="neck_tilt_link">
-        <origin xyz="0 -0.0056 0.02635" rpy="0 0 0" />
+        <origin xyz="0.00478 0.00334 0.021" rpy="0 0 0" />
     </hokuyo_urg>
     <!-- BASE LASER ATTACHMENT -->

Commit message: update wubble head meshes

File: arrg/ua_robots/wubble_description/urdf/wubble2.urdf.xacro (robot description, xacro)
@@ -147,16 +147,91 @@
         <mechanicalReduction>1.0</mechanicalReduction>
     </transmission>
-    <!-- SWISSRANGER CAMERA ATTACHMENT -->
-    <swissranger_camera name="swissranger" parent="head_tilt_link">
-        <origin xyz="0.0 -0.004 0.1235" rpy="${M_PI} 0 0" />
-    </swissranger_camera>
-    <!-- VIDERE STEREO CAMERA ATTACHMENT -->
-    <videre_stereo_6cm name="stoc" parent="head_tilt_link" >
-        <origin xyz="0.0375 0 0.142" rpy="0 0 0" />
-    </videre_stereo_6cm>
     <!-- WUBBLE ARM ATTACHMENT -->
     <wubble_arm parent="base_top_link" >
         <origin xyz="0.16281 0.0825 ${top_size_z/2 + 0.109}" rpy="0 0 0"/>
     </wubble_arm>
+    <!-- KINECT ATTACHMENT -->
+    <joint name="base_kinect_joint" type="fixed">
+        <origin xyz="0.04 0 0.08173" rpy="0 0 0" />
+        <parent link="neck_support_link"/>
+        <child link="kinect_link"/>
+    </joint>
+    <link name="kinect_link">
+        <inertial>
+            <mass value="0.00001" />
+            <origin xyz="0 0 0" />
+            <inertia ixx="1.0" ixy="0.0" ixz="0.0"
+                     iyy="1.0" iyz="0.0"
+                     izz="1.0" />
+        </inertial>
+        <visual>
+            <origin xyz=" 0 0 0 " rpy="0 0 0" />
+            <geometry>
+                <mesh filename="package://wubble_description/meshes/kinect.stl"/>
+            </geometry>
+        </visual>
+        <collision>
+            <origin xyz="0.0 0.0 0.0" rpy="0 0 0" />
+            <geometry>
+                <mesh filename="package://wubble_description/meshes/collada/kinect.dae"/>
+            </geometry>
+        </collision>
+    </link>
+    <joint name="kinect_depth_joint" type="fixed">
+        <origin xyz="0 0.018 0" rpy="0 0 0" />
+        <parent link="kinect_link" />
+        <child link="kinect_depth_frame" />
+    </joint>
+    <link name="kinect_depth_frame">
+        <inertial>
+            <mass value="0.000001" />
+            <origin xyz="0 0 0" />
+            <inertia ixx="0.0001" ixy="0.0" ixz="0.0"
+                     iyy="0.0001" iyz="0.0"
+                     izz="0.0001" />
+        </inertial>
+    </link>
+    <joint name="kinect_depth_optical_joint" type="fixed">
+        <origin xyz="0 0 0" rpy="${-M_PI/2} 0 ${-M_PI/2}" />
+        <parent link="kinect_depth_frame" />
+        <child link="kinect_depth_optical_frame" />
+    </joint>
+    <link name="kinect_depth_optical_frame">
+        <inertial>
+            <mass value="0.000001" />
+            <origin xyz="0 0 0" />
+            <inertia ixx="0.0001" ixy="0.0" ixz="0.0"
+                     iyy="0.0001" iyz="0.0"
+                     izz="0.0001" />
+        </inertial>
+    </link>
+    <joint name="kinect_rgb_joint" type="fixed">
+        <origin xyz="0 -0.005 0" rpy="0 0 0" />
+        <parent link="kinect_link" />
+        <child link="kinect_rgb_frame" />
+    </joint>
+    <link name="kinect_rgb_frame">
+        <inertial>
+            <mass value="0.000001" />
+            <origin xyz="0 0 0" />
+            <inertia ixx="0.0001" ixy="0.0" ixz="0.0"
+                     iyy="0.0001" iyz="0.0"
+                     izz="0.0001" />
+        </inertial>
+    </link>
+    <joint name="kinect_rgb_optical_joint" type="fixed">
+        <origin xyz="0 0 0" rpy="${-M_PI/2} 0 ${-M_PI/2}" />
+        <parent link="kinect_rgb_frame" />
+        <child link="kinect_rgb_optical_frame" />
+    </joint>
+    <link name="kinect_rgb_optical_frame">
+        <inertial>
+            <mass value="0.000001" />
+            <origin xyz="0 0 0" />
+            <inertia ixx="0.0001" ixy="0.0" ixz="0.0"
+                     iyy="0.0001" iyz="0.0"
+                     izz="0.0001" />
+        </inertial>
+    </link>
     <!-- NECK TILTING LASER ATTACHMENT -->
     <joint name="neck_support_joint" type="fixed">

Commit message: fix wrong parent link for kinect

File: arrg/ua_robots/wubble_description/urdf/wubble2.urdf.xacro (robot description, xacro)
@@ -154,5 +154,5 @@
     <joint name="base_kinect_joint" type="fixed">
         <origin xyz="0.04 0 0.08173" rpy="0 0 0" />
-        <parent link="neck_support_link"/>
+        <parent link="head_tilt_link"/>
         <child link="kinect_link"/>
     </joint>

Commit message: change kinect's color to black

File: arrg/ua_robots/wubble_description/urdf/wubble2.urdf.xacro (robot description, xacro)
@@ -170,4 +170,5 @@
                 <mesh filename="package://wubble_description/meshes/kinect.stl"/>
             </geometry>
+            <material name="Black" />
         </visual>
         <collision>
