Commit message: update wubble2 urdf to accomodate erratic changes

File: arrg/ua_robots/wubble_description/urdf/wubble2.urdf.xacro (robot description, xacro)
@@ -17,6 +17,6 @@
     <!-- WUBBLE PLATFORM ATTACHMENT -->
     <joint name="platform_support_joint" type="fixed">
-        <origin xyz="0 0 0" rpy="0 0 0" />
-        <parent link="base_top_link"/>
+        <origin xyz="0 0 ${base_link_to_top}" rpy="0 0 0" />
+        <parent link="base_link"/>
         <child link="platform_link"/>
     </joint>
@@ -32,5 +32,5 @@
             <origin xyz="0 0 0" rpy="0 0 0"/>
             <geometry>
-                <mesh filename="package://wubble_description/meshes/wubble2_platform.stl"/>
+                <mesh filename="package://wubble_description/meshes/collada/wubble2_platform.dae"/>
             </geometry>
             <material name="White" />
@@ -82,13 +82,13 @@
             <origin xyz="0 0 0" rpy="0 0 0"/>
             <geometry>
-                <mesh filename="package://wubble_description/meshes/head_base_link.stl"/>
-            </geometry>
-            <material name="GunMetalBrushedAluminum" />
-        </visual>
-        <collision>
-            <origin xyz="0 0 0" rpy="0 0 0"/>
-            <geometry>
                 <mesh filename="package://wubble_description/meshes/collada/head_base_link.dae"/>
             </geometry>
+            <material name="GunMetalBrushedAluminum" />
+        </visual>
+        <collision>
+            <origin xyz="0 0 0" rpy="0 0 0"/>
+            <geometry>
+                <mesh filename="package://wubble_description/meshes/collada/head_base_link.dae"/>
+            </geometry>
         </collision>
     </link>
@@ -104,13 +104,13 @@
             <origin xyz="0 0 0" rpy="0 0 0"/>
             <geometry>
-                <mesh filename="package://wubble_description/meshes/head_pan_link.stl"/>
-            </geometry>
-            <material name="GunMetalBrushedAluminum" />
-        </visual>
-        <collision>
-            <origin xyz="0 0 0" rpy="0 0 0"/>
-            <geometry>
                 <mesh filename="package://wubble_description/meshes/collada/head_pan_link.dae"/>
             </geometry>
+            <material name="GunMetalBrushedAluminum" />
+        </visual>
+        <collision>
+            <origin xyz="0 0 0" rpy="0 0 0"/>
+            <geometry>
+                <mesh filename="package://wubble_description/meshes/collada/head_pan_link.dae"/>
+            </geometry>
         </collision>
     </link>
@@ -126,5 +126,5 @@
             <origin xyz="0 0 0" rpy="0 0 0"/>
             <geometry>
-                <mesh filename="package://wubble_description/meshes/head_tilt_link.stl"/>
+                <mesh filename="package://wubble_description/meshes/collada/head_tilt_link.dae"/>
             </geometry>
             <material name="GunMetalBrushedAluminum" />
@@ -148,6 +148,6 @@
     </transmission>
     <!-- WUBBLE ARM ATTACHMENT -->
-    <wubble_arm parent="base_top_link" >
-        <origin xyz="0.16281 0.0825 ${top_size_z/2 + 0.109}" rpy="0 0 0"/>
+    <wubble_arm parent="base_link" >
+        <origin xyz="0.16281 0.0825 0.1885" rpy="0 0 0"/>
     </wubble_arm>
     <!-- KINECT ATTACHMENT -->
@@ -168,5 +168,5 @@
             <origin xyz=" 0 0 0 " rpy="0 0 0" />
             <geometry>
-                <mesh filename="package://wubble_description/meshes/kinect.stl"/>
+                <mesh filename="package://wubble_description/meshes/collada/kinect.dae"/>
             </geometry>
             <material name="Black" />
@@ -261,13 +261,13 @@
             <origin xyz="0 0 0" rpy="0 0 0"/>
             <geometry>
-                <mesh filename="package://wubble_description/meshes/neck_laser_support_link.stl"/>
-            </geometry>
-            <material name="GunMetalBrushedAluminum" />
-        </visual>
-        <collision>
-            <origin xyz="0 0 0" rpy="0 0 0"/>
-            <geometry>
                 <mesh filename="package://wubble_description/meshes/collada/neck_laser_support_link.dae"/>
             </geometry>
+            <material name="GunMetalBrushedAluminum" />
+        </visual>
+        <collision>
+            <origin xyz="0 0 0" rpy="0 0 0"/>
+            <geometry>
+                <mesh filename="package://wubble_description/meshes/collada/neck_laser_support_link.dae"/>
+            </geometry>
         </collision>
     </link>
@@ -283,5 +283,5 @@
             <origin xyz="0 0 0" rpy="0 0 0"/>
             <geometry>
-                <mesh filename="package://wubble_description/meshes/neck_tilt_link.stl"/>
+                <mesh filename="package://wubble_description/meshes/collada/neck_tilt_link.dae"/>
             </geometry>
             <material name="GunMetalBrushedAluminum" />
@@ -303,6 +303,6 @@
     </hokuyo_urg>
     <!-- BASE LASER ATTACHMENT -->
-    <hokuyo_urg name="base_scan" parent="base_top_link">
-        <origin xyz="${top_size_x/2 - 0.01 - 0.04} 0 -${top_size_z/2}" rpy="${M_PI} 0 0" />
+    <hokuyo_urg name="base_scan" parent="base_link">
+        <origin xyz="0.16025 -0.0025 0.0775" rpy="${M_PI} 0 0" />
     </hokuyo_urg>
     <!-- GAZEBO MATERIALS -->

Commit message: updated wubble2 urdf

File: arrg/ua_robots/wubble_description/urdf/wubble2.urdf.xacro (robot description, xacro)
@@ -10,5 +10,6 @@
     <include filename="$(find swissranger_camera_description)/urdf/swissranger_camera.xacro" />
     <include filename="$(find videre_stoc_description)/urdf/videre_stereo_6cm.xacro" />
-    <include filename="$(find chr_6dm_imu_description)/urdf/chrobotics_chr_6dm_imu.urdf.xacro" />
+    <include filename="$(find wubble_description)/urdf/microstrain_3dmgx3_imu.urdf.xacro" />
+    <include filename="$(find wubble_description)/urdf/wubble2_calibration.xacro" />
     <!-- Properties (Constants) -->
     <property name="M_PI" value="3.14159"/>
@@ -43,8 +44,8 @@
         </collision>
     </link>
-    <!-- CHR-6dm IMU ATTACHMENT -->
-    <chrobotics_chr_6dm_imu name="imu" parent="platform_link" imu_topic="imu/data" update_rate="120.0" stdev="0.00017" >
-        <origin xyz="0 0 1.0" rpy="0 0 0" />
-    </chrobotics_chr_6dm_imu>
+    <!-- MicroStrain IMU ATTACHMENT -->
+    <microstrain_3dmgx3_imu_v0 name="imu" parent="platform_link" imu_topic="imu/data" update_rate="100.0" stdev="0.00017" >
+        <origin xyz="0 0 0.80514" rpy="0 ${M_PI} 0" />
+    </microstrain_3dmgx3_imu_v0>
     <!-- WUBBLE HEAD ATTACHMENT -->
     <joint name="head_base_joint" type="fixed">
@@ -153,6 +154,7 @@
     <!-- KINECT ATTACHMENT -->
     <joint name="base_kinect_joint" type="fixed">
-        <origin xyz="0.04 0 0.08173" rpy="0 0 0" />
-        <parent link="head_tilt_link"/>
+        <origin xyz="${wubble2_calib_cam_x} ${wubble2_calib_cam_y} ${wubble2_calib_cam_z}"
+                rpy="${wubble2_calib_cam_rr} ${wubble2_calib_cam_rp} ${wubble2_calib_cam_ry}" />
+        <parent link="${wubble2_kinect_frame_name}" />
         <child link="kinect_link"/>
     </joint>
@@ -237,5 +239,5 @@
     <!-- NECK TILTING LASER ATTACHMENT -->
     <joint name="neck_support_joint" type="fixed">
-        <origin xyz="0.0254 0 0.655" rpy="0 0 0" />
+        <origin xyz="0.0254 0 0.645" rpy="0 0 0" />
         <parent link="platform_link"/>
         <child link="neck_support_link"/>
@@ -300,9 +302,11 @@
     </transmission>
     <hokuyo_urg name="neck_scan" parent="neck_tilt_link">
-        <origin xyz="0.00478 0.00334 0.021" rpy="0 0 0" />
+        <origin xyz="${calib_tilt_laser_x} ${calib_tilt_laser_y} ${calib_tilt_laser_z}"
+                rpy="${calib_tilt_laser_rr} ${calib_tilt_laser_rp} ${calib_tilt_laser_ry}" />
     </hokuyo_urg>
     <!-- BASE LASER ATTACHMENT -->
     <hokuyo_urg name="base_scan" parent="base_link">
-        <origin xyz="0.16025 -0.0025 0.0775" rpy="${M_PI} 0 0" />
+        <origin xyz="${calib_base_laser_x} ${calib_base_laser_y} ${calib_base_laser_z}"
+                rpy="${calib_base_laser_rr} ${calib_base_laser_rp} ${calib_base_laser_ry}" />
     </hokuyo_urg>
     <!-- GAZEBO MATERIALS -->
