Commit message: Move erratic related packages into separate stack.

File: arrg/videre_erratic/erratic_description/urdf/materials.urdf.xacro (robot description, xacro)
@@ -22,3 +22,6 @@
         <color rgba="1.0 1.0 1.0 1.0"/>
     </material>
+    <material name="GunMetalBrushedAluminum">
+        <texture filename="package://smart_arm_description/Media/materials/textures/gun_metal_brushed_aluminum.jpg" />
+    </material>
 </robot>
