Commit message: Change to Z forward orientation for swissranger model, add interpolated_ik launch and test.

File: arrg/ua_robots/swissranger_camera_description/urdf/swissranger_camera.xacro (robot description, xacro)
@@ -31,5 +31,5 @@
         </link>
         <joint name="${name}_joint" type="fixed">
-            <origin xyz="0.02795 0 0.0325" rpy="0 0 0" />
+            <origin xyz="0.02795 0 0.0325" rpy="${-M_PI/2} 0.0 ${-M_PI/2}" />
             <parent link="${name}_mount_link" />
             <child link="${name}_link" />

File: arrg/ua_robots/wubble_description/urdf/wubble2.urdf.xacro (robot description, xacro)
@@ -144,5 +144,5 @@
     <!-- SWISSRANGER CAMERA ATTACHMENT -->
     <swissranger_camera name="swissranger" parent="head_tilt_link">
-        <origin xyz="0.0125 0 0.036" rpy="${M_PI} 0 0" />
+        <origin xyz="0.0125 0 ${0.036-0.003}" rpy="${M_PI} 0 0" />
     </swissranger_camera>
     <!-- VIDERE STEREO CAMERA ATTACHMENT -->

Commit message: move swissranger optical center back a bit

File: arrg/ua_robots/swissranger_camera_description/urdf/swissranger_camera.xacro (robot description, xacro)
@@ -31,5 +31,5 @@
         </link>
         <joint name="${name}_joint" type="fixed">
-            <origin xyz="0.02795 0 0.0325" rpy="${-M_PI/2} 0.0 ${-M_PI/2}" />
+            <origin xyz="-0.03205 0 0.0325" rpy="${-M_PI/2} 0.0 ${-M_PI/2}" />
             <parent link="${name}_mount_link" />
             <child link="${name}_link" />

Commit message: revert swissranger change

File: arrg/ua_robots/swissranger_camera_description/urdf/swissranger_camera.xacro (robot description, xacro)
@@ -31,5 +31,5 @@
         </link>
         <joint name="${name}_joint" type="fixed">
-            <origin xyz="-0.03205 0 0.0325" rpy="${-M_PI/2} 0.0 ${-M_PI/2}" />
+            <origin xyz="0.02795 0 0.0325" rpy="${-M_PI/2} 0.0 ${-M_PI/2}" />
             <parent link="${name}_mount_link" />
             <child link="${name}_link" />
