Commit message: consolidate all crustcrawler smart arm packages into one stack

File: arrg/crustcrawler_smart_arm/smart_arm_description/urdf/smart_arm.xacro (robot description, xacro)
@@ -23,8 +23,8 @@
         </joint>
         <!-- Shoulder tilt joint -->
-        <joint name="shoulder_tilt_joint" type="revolute">
+        <joint name="shoulder_pitch_joint" type="revolute">
             <origin xyz="${0.105 - 0.01 - 0.03085/2} 0 ${0.01 + 0.05 - 0.031/2}" rpy="0 0 0" />
             <parent link="arm_shoulder_pan_link"/>
-            <child link="arm_shoulder_tilt_link" />
+            <child link="arm_shoulder_pitch_link" />
             <axis xyz="0 -1 0"/>
             <limit  lower="-1.04719755" upper="1.972222" effort="300" velocity="1.17" />
@@ -33,8 +33,8 @@
         </joint>
         <!-- Elbow tilt joint -->
-        <joint name="elbow_tilt_joint" type="revolute">
+        <joint name="elbow_flex_joint" type="revolute">
             <origin xyz="${0.04 - 0.01 + 0.0015 + 0.105 + 0.055 - 0.01} 0 0" rpy="0 0 0" />
-            <parent link="arm_shoulder_tilt_link"/>
-            <child link="arm_elbow_tilt_link" />
+            <parent link="arm_shoulder_pitch_link"/>
+            <child link="arm_elbow_flex_link" />
             <axis xyz="0 -1 0"/>
             <!-- From -113 to 108 degrees -->
@@ -44,8 +44,8 @@
         </joint>
         <!-- Wrist rotate joint -->
-        <joint name="wrist_rotate_joint" type="revolute">
+        <joint name="wrist_roll_joint" type="revolute">
             <origin xyz="${0.08 - 0.01} 0 ${0.05 - 0.0115 - 0.0155}" rpy="0 0 0" />
-            <parent link="arm_elbow_tilt_link"/>
-            <child link="arm_wrist_rotate_link" />
+            <parent link="arm_elbow_flex_link"/>
+            <child link="arm_wrist_roll_link" />
             <axis xyz="-1 0 0"/>
             <!-- From -150 to 150 degrees -->
@@ -57,5 +57,5 @@
         <joint name="finger_right_joint" type="revolute">
             <origin xyz="${0.0015 + 0.05 - 0.01} ${-0.035/2} 0" rpy="0 0 0" />
-            <parent link="arm_wrist_rotate_link"/>
+            <parent link="arm_wrist_roll_link"/>
             <child link="arm_right_finger_link" />
             <axis xyz="0 0 1"/>
@@ -68,5 +68,5 @@
         <joint name="finger_left_joint" type="revolute">
             <origin xyz="${0.0015 + 0.05 - 0.01} ${0.035/2} 0" rpy="0 0 0" />
-            <parent link="arm_wrist_rotate_link"/>
+            <parent link="arm_wrist_roll_link"/>
             <child link="arm_left_finger_link" />
             <axis xyz="0 0 1"/>
@@ -119,5 +119,5 @@
             </collision>
         </link>
-        <link name="arm_shoulder_tilt_link">
+        <link name="arm_shoulder_pitch_link">
             <inertial>
                 <mass value="0.18" />
@@ -130,15 +130,15 @@
                 <origin xyz="0.0 0.0 0.0" rpy="0 0 0" />
                 <geometry>
-                    <mesh filename="package://smart_arm_description/meshes/arm_shoulder_tilt.stl"/>
-                </geometry>
-            </visual>
-            <collision>
-                <origin xyz="0.0 0.0 0.0" rpy="0 0 0" />
-                <geometry>
-                    <mesh filename="package://smart_arm_description/meshes/convex/arm_shoulder_tilt_convex.stlb"/>
-                </geometry>
-            </collision>
-        </link>
-        <link name="arm_elbow_tilt_link">
+                    <mesh filename="package://smart_arm_description/meshes/arm_shoulder_pitch.stl"/>
+                </geometry>
+            </visual>
+            <collision>
+                <origin xyz="0.0 0.0 0.0" rpy="0 0 0" />
+                <geometry>
+                    <mesh filename="package://smart_arm_description/meshes/convex/arm_shoulder_pitch_convex.stlb"/>
+                </geometry>
+            </collision>
+        </link>
+        <link name="arm_elbow_flex_link">
             <inertial>
                 <mass value="0.12" />
@@ -151,15 +151,15 @@
                 <origin xyz="0.0 0.0 0.0" rpy="0 0 0" />
                 <geometry>
-                    <mesh filename="package://smart_arm_description/meshes/arm_elbow_tilt.stl"/>
-                </geometry>
-            </visual>
-            <collision>
-                <origin xyz="0.0 0.0 0.0" rpy="0 0 0" />
-                <geometry>
-                    <mesh filename="package://smart_arm_description/meshes/convex/arm_elbow_tilt_convex.stlb"/>
-                </geometry>
-            </collision>
-        </link>
-        <link name="arm_wrist_rotate_link">
+                    <mesh filename="package://smart_arm_description/meshes/arm_elbow_flex.stl"/>
+                </geometry>
+            </visual>
+            <collision>
+                <origin xyz="0.0 0.0 0.0" rpy="0 0 0" />
+                <geometry>
+                    <mesh filename="package://smart_arm_description/meshes/convex/arm_elbow_flex_convex.stlb"/>
+                </geometry>
+            </collision>
+        </link>
+        <link name="arm_wrist_roll_link">
             <inertial>
                 <mass value="0.13" />
@@ -172,11 +172,11 @@
                 <origin xyz="0.0 0.0 0.0" rpy="0 0 0" />
                 <geometry>
-                    <mesh filename="package://smart_arm_description/meshes/arm_wrist_rotate.stl"/>
-                </geometry>
-            </visual>
-            <collision>
-                <origin xyz="0.0 0.0 0.0" rpy="0 0 0" />
-                <geometry>
-                    <mesh filename="package://smart_arm_description/meshes/convex/arm_wrist_rotate_convex.stlb"/>
+                    <mesh filename="package://smart_arm_description/meshes/arm_wrist_roll.stl"/>
+                </geometry>
+            </visual>
+            <collision>
+                <origin xyz="0.0 0.0 0.0" rpy="0 0 0" />
+                <geometry>
+                    <mesh filename="package://smart_arm_description/meshes/convex/arm_wrist_roll_convex.stlb"/>
                 </geometry>
             </collision>
@@ -230,17 +230,17 @@
             <mechanicalReduction>1.0</mechanicalReduction>
         </transmission>
-        <transmission type="pr2_mechanism_model/SimpleTransmission" name="shoulder_tilt_trans">
-            <actuator name="shoulder_tilt_motor" />
-            <joint name="shoulder_tilt_joint" />
-            <mechanicalReduction>1.0</mechanicalReduction>
-        </transmission>
-        <transmission type="pr2_mechanism_model/SimpleTransmission" name="elbow_tilt_trans">
-            <actuator name="elbow_tilt_motor" />
-            <joint name="elbow_tilt_joint" />
-            <mechanicalReduction>1.0</mechanicalReduction>
-        </transmission>
-        <transmission type="pr2_mechanism_model/SimpleTransmission" name="wrist_rotate_trans">
-            <actuator name="wrist_rotate_motor" />
-            <joint name="wrist_rotate_joint" />
+        <transmission type="pr2_mechanism_model/SimpleTransmission" name="shoulder_pitch_trans">
+            <actuator name="shoulder_pitch_motor" />
+            <joint name="shoulder_pitch_joint" />
+            <mechanicalReduction>1.0</mechanicalReduction>
+        </transmission>
+        <transmission type="pr2_mechanism_model/SimpleTransmission" name="elbow_flex_trans">
+            <actuator name="elbow_flex_motor" />
+            <joint name="elbow_flex_joint" />
+            <mechanicalReduction>1.0</mechanicalReduction>
+        </transmission>
+        <transmission type="pr2_mechanism_model/SimpleTransmission" name="wrist_roll_trans">
+            <actuator name="wrist_roll_motor" />
+            <joint name="wrist_roll_joint" />
             <mechanicalReduction>1.0</mechanicalReduction>
         </transmission>
@@ -264,13 +264,13 @@
             <turnGravityOff>true</turnGravityOff>
         </gazebo>
-        <gazebo reference="arm_shoulder_tilt_link">
-            <material>SmartArm/GunMetalBrushedAluminum</material>
-            <turnGravityOff>true</turnGravityOff>
-        </gazebo>
-        <gazebo reference="arm_elbow_tilt_link">
-            <material>SmartArm/GunMetalBrushedAluminum</material>
-            <turnGravityOff>true</turnGravityOff>
-        </gazebo>
-        <gazebo reference="arm_wrist_rotate_link">
+        <gazebo reference="arm_shoulder_pitch_link">
+            <material>SmartArm/GunMetalBrushedAluminum</material>
+            <turnGravityOff>true</turnGravityOff>
+        </gazebo>
+        <gazebo reference="arm_elbow_flex_link">
+            <material>SmartArm/GunMetalBrushedAluminum</material>
+            <turnGravityOff>true</turnGravityOff>
+        </gazebo>
+        <gazebo reference="arm_wrist_roll_link">
             <material>SmartArm/GunMetalBrushedAluminum</material>
             <turnGravityOff>true</turnGravityOff>
@@ -297,15 +297,15 @@
             <fudgeFactor value="0.5" />
         </gazebo>
-        <gazebo reference="shoulder_tilt_joint">
+        <gazebo reference="shoulder_pitch_joint">
             <stopKd value="1.0" />
             <stopKp value="1000000.0" />
             <fudgeFactor value="0.5" />
         </gazebo>
-        <gazebo reference="elbow_tilt_joint">
+        <gazebo reference="elbow_flex_joint">
             <stopKd value="1.0" />
             <stopKp value="1000000.0" />
             <fudgeFactor value="0.5" />
         </gazebo>
-        <gazebo reference="wrist_rotate_joint">
+        <gazebo reference="wrist_roll_joint">
             <stopKd value="1.0" />
             <stopKp value="1000000.0" />

Commit message: add collada models for each smart arm joint, generate collada description for openrave, regenerate ik

File: arrg/crustcrawler_smart_arm/smart_arm_description/urdf/smart_arm.xacro (robot description, xacro)
@@ -55,5 +55,5 @@
         </joint>
         <!-- Gripper right finger joint -->
-        <joint name="finger_right_joint" type="revolute">
+        <joint name="right_finger_joint" type="revolute">
             <origin xyz="${0.0015 + 0.05 - 0.01} ${-0.035/2} 0" rpy="0 0 0" />
             <parent link="arm_wrist_roll_link"/>
@@ -66,5 +66,5 @@
         </joint>
         <!-- Gripper left finger joint -->
-        <joint name="finger_left_joint" type="revolute">
+        <joint name="left_finger_joint" type="revolute">
             <origin xyz="${0.0015 + 0.05 - 0.01} ${0.035/2} 0" rpy="0 0 0" />
             <parent link="arm_wrist_roll_link"/>
@@ -88,11 +88,11 @@
                 <origin xyz="0.0 0.0 0.0" rpy="0 0 0" />
                 <geometry>
-                    <mesh filename="package://smart_arm_description/meshes/arm_base.stl"/>
-                </geometry>
-            </visual>
-            <collision>
-                <origin xyz="0.0 0.0 0.0" rpy="0 0 0" />
-                <geometry>
-                    <mesh filename="package://smart_arm_description/meshes/convex/arm_base_convex.stlb"/>
+                    <mesh filename="package://smart_arm_description/meshes/collada/arm_base.dae"/>
+                </geometry>
+            </visual>
+            <collision>
+                <origin xyz="0.0 0.0 0.0" rpy="0 0 0" />
+                <geometry>
+                    <mesh filename="package://smart_arm_description/meshes/collada/arm_base.dae"/>
                 </geometry>
             </collision>
@@ -109,11 +109,11 @@
                 <origin xyz="0.0 0.0 0.005" rpy="0 0 0" />
                 <geometry>
-                    <mesh filename="package://smart_arm_description/meshes/arm_shoulder_pan.stl"/>
-                </geometry>
-            </visual>
-            <collision>
-                <origin xyz="0.0 0.0 0.0" rpy="0 0 0" />
-                <geometry>
-                    <mesh filename="package://smart_arm_description/meshes/convex/arm_shoulder_pan_convex.stlb"/>
+                    <mesh filename="package://smart_arm_description/meshes/collada/arm_shoulder_pan.dae"/>
+                </geometry>
+            </visual>
+            <collision>
+                <origin xyz="0.0 0.0 0.0" rpy="0 0 0" />
+                <geometry>
+                    <mesh filename="package://smart_arm_description/meshes/collada/arm_shoulder_pan.dae"/>
                 </geometry>
             </collision>
@@ -130,11 +130,11 @@
                 <origin xyz="0.0 0.0 0.0" rpy="0 0 0" />
                 <geometry>
-                    <mesh filename="package://smart_arm_description/meshes/arm_shoulder_pitch.stl"/>
-                </geometry>
-            </visual>
-            <collision>
-                <origin xyz="0.0 0.0 0.0" rpy="0 0 0" />
-                <geometry>
-                    <mesh filename="package://smart_arm_description/meshes/convex/arm_shoulder_pitch_convex.stlb"/>
+                    <mesh filename="package://smart_arm_description/meshes/collada/arm_shoulder_pitch.dae"/>
+                </geometry>
+            </visual>
+            <collision>
+                <origin xyz="0.0 0.0 0.0" rpy="0 0 0" />
+                <geometry>
+                    <mesh filename="package://smart_arm_description/meshes/collada/arm_shoulder_pitch.dae"/>
                 </geometry>
             </collision>
@@ -151,11 +151,11 @@
                 <origin xyz="0.0 0.0 0.0" rpy="0 0 0" />
                 <geometry>
-                    <mesh filename="package://smart_arm_description/meshes/arm_elbow_flex.stl"/>
-                </geometry>
-            </visual>
-            <collision>
-                <origin xyz="0.0 0.0 0.0" rpy="0 0 0" />
-                <geometry>
-                    <mesh filename="package://smart_arm_description/meshes/convex/arm_elbow_flex_convex.stlb"/>
+                    <mesh filename="package://smart_arm_description/meshes/collada/arm_elbow_flex.dae"/>
+                </geometry>
+            </visual>
+            <collision>
+                <origin xyz="0.0 0.0 0.0" rpy="0 0 0" />
+                <geometry>
+                    <mesh filename="package://smart_arm_description/meshes/collada/arm_elbow_flex.dae"/>
                 </geometry>
             </collision>
@@ -172,11 +172,11 @@
                 <origin xyz="0.0 0.0 0.0" rpy="0 0 0" />
                 <geometry>
-                    <mesh filename="package://smart_arm_description/meshes/arm_wrist_roll.stl"/>
-                </geometry>
-            </visual>
-            <collision>
-                <origin xyz="0.0 0.0 0.0" rpy="0 0 0" />
-                <geometry>
-                    <mesh filename="package://smart_arm_description/meshes/convex/arm_wrist_roll_convex.stlb"/>
+                    <mesh filename="package://smart_arm_description/meshes/collada/arm_wrist_roll.dae"/>
+                </geometry>
+            </visual>
+            <collision>
+                <origin xyz="0.0 0.0 0.0" rpy="0 0 0" />
+                <geometry>
+                    <mesh filename="package://smart_arm_description/meshes/collada/arm_wrist_roll.dae"/>
                 </geometry>
             </collision>
@@ -193,11 +193,11 @@
                 <origin xyz="0.0 0.0 0.0" rpy="0 0 0" />
                 <geometry>
-                    <mesh filename="package://smart_arm_description/meshes/arm_right_finger.stl"/>
-                </geometry>
-            </visual>
-            <collision>
-                <origin xyz="0.0 0.0 0.0" rpy="0 0 0" />
-                <geometry>
-                    <mesh filename="package://smart_arm_description/meshes/convex/arm_right_finger_convex.stlb"/>
+                    <mesh filename="package://smart_arm_description/meshes/collada/arm_right_finger.dae"/>
+                </geometry>
+            </visual>
+            <collision>
+                <origin xyz="0.0 0.0 0.0" rpy="0 0 0" />
+                <geometry>
+                    <mesh filename="package://smart_arm_description/meshes/collada/arm_right_finger.dae"/>
                 </geometry>
             </collision>
@@ -214,11 +214,11 @@
                 <origin xyz="0.0 0.0 0.0" rpy="0 0 0" />
                 <geometry>
-                    <mesh filename="package://smart_arm_description/meshes/arm_left_finger.stl"/>
-                </geometry>
-            </visual>
-            <collision>
-                <origin xyz="0.0 0.0 0.0" rpy="0 0 0" />
-                <geometry>
-                    <mesh filename="package://smart_arm_description/meshes/convex/arm_left_finger_convex.stlb"/>
+                    <mesh filename="package://smart_arm_description/meshes/collada/arm_left_finger.dae"/>
+                </geometry>
+            </visual>
+            <collision>
+                <origin xyz="0.0 0.0 0.0" rpy="0 0 0" />
+                <geometry>
+                    <mesh filename="package://smart_arm_description/meshes/collada/arm_left_finger.dae"/>
                 </geometry>
             </collision>
@@ -245,12 +245,12 @@
             <mechanicalReduction>1.0</mechanicalReduction>
         </transmission>
-        <transmission type="pr2_mechanism_model/SimpleTransmission" name="finger_right_trans">
-            <actuator name="finger_right_motor" />
-            <joint name="finger_right_joint" />
-            <mechanicalReduction>1.0</mechanicalReduction>
-        </transmission>
-        <transmission type="pr2_mechanism_model/SimpleTransmission" name="finger_left_trans">
-            <actuator name="finger_left_motor" />
-            <joint name="finger_left_joint" />
+        <transmission type="pr2_mechanism_model/SimpleTransmission" name="right_finger_trans">
+            <actuator name="right_finger_motor" />
+            <joint name="right_finger_joint" />
+            <mechanicalReduction>1.0</mechanicalReduction>
+        </transmission>
+        <transmission type="pr2_mechanism_model/SimpleTransmission" name="left_finger_trans">
+            <actuator name="left_finger_motor" />
+            <joint name="left_finger_joint" />
             <mechanicalReduction>1.0</mechanicalReduction>
         </transmission>
@@ -312,10 +312,10 @@
             <fudgeFactor value="0.5" />
         </gazebo>
-        <gazebo reference="finger_right_joint">
+        <gazebo reference="right_finger_joint">
             <stopKd value="1.0" />
             <stopKp value="1000000.0" />
             <fudgeFactor value="1.0" />
         </gazebo>
-        <gazebo reference="finger_left_joint">
+        <gazebo reference="left_finger_joint">
             <stopKd value="1.0" />
             <stopKp value="1000000.0" />

Commit message: update smart arm openrave model

File: arrg/crustcrawler_smart_arm/smart_arm_description/urdf/smart_arm.xacro (robot description, xacro)
@@ -1,7 +1,41 @@
 <?xml version="1.0"?>
+<!--
+* Software License Agreement (BSD License)
+*
+* Copyright (c) 2010, Antons Rebguns. All rights reserved.
+*
+* Redistribution and use in source and binary forms, with or without
+* modification, are permitted provided that the following conditions
+* are met:
+*
+*  * Redistributions of source code must retain the above copyright
+*    notice, this list of conditions and the following disclaimer.
+*  * Redistributions in binary form must reproduce the above
+*    copyright notice, this list of conditions and the following
+*    disclaimer in the documentation and/or other materials provided
+*    with the distribution.
+*  * Neither the name of University of Arizona nor the names of its
+*    contributors may be used to endorse or promote products derived
+*    from this software without specific prior written permission.
+*
+* THIS SOFTWARE IS PROVIDED BY THE COPYRIGHT HOLDERS AND CONTRIBUTORS
+* "AS IS" AND ANY EXPRESS OR IMPLIED WARRANTIES, INCLUDING, BUT NOT
+* LIMITED TO, THE IMPLIED WARRANTIES OF MERCHANTABILITY AND FITNESS
+* FOR A PARTICULAR PURPOSE ARE DISCLAIMED. IN NO EVENT SHALL THE
+* COPYRIGHT OWNER OR CONTRIBUTORS BE LIABLE FOR ANY DIRECT, INDIRECT,
+* INCIDENTAL, SPECIAL, EXEMPLARY, OR CONSEQUENTIAL DAMAGES (INCLUDING,
+* BUT NOT LIMITED TO, PROCUREMENT OF SUBSTITUTE GOODS OR SERVICES;
+* LOSS OF USE, DATA, OR PROFITS; OR BUSINESS INTERRUPTION) HOWEVER
+* CAUSED AND ON ANY THEORY OF LIABILITY, WHETHER IN CONTRACT, STRICT
+* LIABILITY, OR TORT (INCLUDING NEGLIGENCE OR OTHERWISE) ARISING IN
+* ANY WAY OUT OF THE USE OF THIS SOFTWARE, EVEN IF ADVISED OF THE
+* POSSIBILITY OF SUCH DAMAGE.
+* Author: Antons Rebguns
+-->
 <robot
     xmlns:sensor="http://playerstage.sourceforge.net/gazebo/xmlschema/#sensor"
     xmlns:controller="http://playerstage.sourceforge.net/gazebo/xmlschema/#controller"
     xmlns:interface="http://playerstage.sourceforge.net/gazebo/xmlschema/#interface">
+    <include filename="$(find smart_arm_description)/urdf/materials.urdf.xacro" />
     <macro name="smart_arm" params="parent *origin">
         <!-- ****** JOINT DEFINITIONS ****** -->
@@ -90,4 +124,5 @@
                     <mesh filename="package://smart_arm_description/meshes/collada/arm_base.dae"/>
                 </geometry>
+                <material name="Green" />
             </visual>
             <collision>
@@ -111,4 +146,5 @@
                     <mesh filename="package://smart_arm_description/meshes/collada/arm_shoulder_pan.dae"/>
                 </geometry>
+                <material name="Grey" />
             </visual>
             <collision>
@@ -132,4 +168,5 @@
                     <mesh filename="package://smart_arm_description/meshes/collada/arm_shoulder_pitch.dae"/>
                 </geometry>
+                <material name="Blue" />
             </visual>
             <collision>
@@ -153,4 +190,5 @@
                     <mesh filename="package://smart_arm_description/meshes/collada/arm_elbow_flex.dae"/>
                 </geometry>
+                <material name="Green" />
             </visual>
             <collision>
@@ -174,4 +212,5 @@
                     <mesh filename="package://smart_arm_description/meshes/collada/arm_wrist_roll.dae"/>
                 </geometry>
+                <material name="Grey" />
             </visual>
             <collision>
@@ -195,4 +234,5 @@
                     <mesh filename="package://smart_arm_description/meshes/collada/arm_right_finger.dae"/>
                 </geometry>
+                <material name="Blue" />
             </visual>
             <collision>
@@ -216,4 +256,5 @@
                     <mesh filename="package://smart_arm_description/meshes/collada/arm_left_finger.dae"/>
                 </geometry>
+                <material name="Green" />
             </visual>
             <collision>
