Commit message: Modify limits on all arm joints in urdf to match hardware limits.

File: arrg/ua_robots/wubble_arm_description/urdf/wubble_arm.xacro (robot description, xacro)
@@ -51,6 +51,6 @@
             <child link="L1_shoulder_pitch_link"/>
             <axis xyz="0 1 0"/>
-            <limit  lower="-1.22" upper="1.22" effort="300" velocity="1.17" />
-            <safety_controller k_position="100" k_velocity="15.0" soft_lower_limit="${-1.22+0.1}" soft_upper_limit="${1.22-0.1}" />
+            <limit  lower="-2.13" upper="1.39" effort="300" velocity="1.17" />
+            <safety_controller k_position="100" k_velocity="15.0" soft_lower_limit="${-2.13}" soft_upper_limit="${1.39}" />
             <dynamics damping="50" friction="1"/>
         </joint>
@@ -61,6 +61,6 @@
             <child link="L2_shoulder_yaw_link"/>
             <axis xyz="0 0 1"/>
-            <limit  lower="-1.22" upper="1.22" effort="300" velocity="1.17" />
-            <safety_controller k_position="100" k_velocity="15.0" soft_lower_limit="${-1.22+0.1}" soft_upper_limit="${1.22-0.1}" />
+            <limit  lower="-1.90" upper="1.90" effort="300" velocity="1.17" />
+            <safety_controller k_position="100" k_velocity="15.0" soft_lower_limit="${-1.90}" soft_upper_limit="${1.90}" />
             <dynamics damping="50" friction="1"/>
         </joint>
@@ -71,6 +71,6 @@
             <child link="L3_shoulder_roll_link"/>
             <axis xyz="0 1 0"/>
-            <limit  lower="-1.22" upper="1.22" effort="300" velocity="1.17" />
-            <safety_controller k_position="100" k_velocity="15.0" soft_lower_limit="${-1.22+0.1}" soft_upper_limit="${1.22-0.1}" />
+            <limit  lower="-2.18" upper="2.18" effort="300" velocity="1.17" />
+            <safety_controller k_position="100" k_velocity="15.0" soft_lower_limit="${-2.18}" soft_upper_limit="${2.18}" />
             <dynamics damping="50" friction="1"/>
         </joint>
@@ -81,6 +81,6 @@
             <child link="L4_elbow_pitch_link"/>
             <axis xyz="0 0 1"/>
-            <limit  lower="-1.22" upper="1.22" effort="300" velocity="1.17" />
-            <safety_controller k_position="100" k_velocity="15.0" soft_lower_limit="${-1.22+0.1}" soft_upper_limit="${1.22-0.1}" />
+            <limit  lower="-1.53" upper="1.80" effort="300" velocity="1.17" />
+            <safety_controller k_position="100" k_velocity="15.0" soft_lower_limit="${-1.53}" soft_upper_limit="${1.80}" />
             <dynamics damping="50" friction="1"/>
         </joint>
@@ -91,6 +91,6 @@
             <child link="L5_wrist_roll_link"/>
             <axis xyz="1 0 0"/>
-            <limit  lower="-1.22" upper="1.22" effort="300" velocity="1.17" />
-            <safety_controller k_position="100" k_velocity="15.0" soft_lower_limit="${-1.22+0.1}" soft_upper_limit="${1.22-0.1}" />
+            <limit  lower="-2.61" upper="2.61" effort="300" velocity="1.17" />
+            <safety_controller k_position="100" k_velocity="15.0" soft_lower_limit="${-2.61}" soft_upper_limit="${2.61}" />
             <dynamics damping="50" friction="1"/>
         </joint>
@@ -101,6 +101,6 @@
             <child link="L6_wrist_pitch_link"/>
             <axis xyz="0 1 0"/>
-            <limit  lower="-1.22" upper="1.22" effort="300" velocity="1.17" />
-            <safety_controller k_position="100" k_velocity="15.0" soft_lower_limit="${-1.22+0.1}" soft_upper_limit="${1.22-0.1}" />
+            <limit  lower="-0.61" upper="2.27" effort="300" velocity="1.17" />
+            <safety_controller k_position="100" k_velocity="15.0" soft_lower_limit="${-0.61}" soft_upper_limit="${2.27}" />
             <dynamics damping="50" friction="1"/>
         </joint>
@@ -111,6 +111,6 @@
             <child link="L7_wrist_yaw_link"/>
             <axis xyz="0 0 1"/>
-            <limit  lower="-1.22" upper="1.22" effort="300" velocity="1.17" />
-            <safety_controller k_position="100" k_velocity="15.0" soft_lower_limit="${-1.22+0.1}" soft_upper_limit="${1.22-0.1}" />
+            <limit  lower="-1.66" upper="1.62" effort="300" velocity="1.17" />
+            <safety_controller k_position="100" k_velocity="15.0" soft_lower_limit="${-1.66}" soft_upper_limit="${1.62}" />
             <dynamics damping="50" friction="1"/>
         </joint>
@@ -121,6 +121,6 @@
             <child link="L8_left_finger_link"/>
             <axis xyz="0 0 1"/>
-            <limit  lower="-1.22" upper="1.22" effort="300" velocity="1.17" />
-            <safety_controller k_position="100" k_velocity="15.0" soft_lower_limit="${-1.22+0.1}" soft_upper_limit="${1.22-0.1}" />
+            <limit  lower="-0.28" upper="0.785" effort="300" velocity="1.17" />
+            <safety_controller k_position="100" k_velocity="15.0" soft_lower_limit="${-0.28}" soft_upper_limit="${0.785}" />
             <dynamics damping="50" friction="1"/>
         </joint>
@@ -131,6 +131,6 @@
             <child link="L9_right_finger_link"/>
             <axis xyz="0 0 1"/>
-            <limit  lower="-1.22" upper="1.22" effort="300" velocity="1.17" />
-            <safety_controller k_position="100" k_velocity="15.0" soft_lower_limit="${-1.22+0.1}" soft_upper_limit="${1.22-0.1}" />
+            <limit  lower="-0.785" upper="0.28" effort="300" velocity="1.17" />
+            <safety_controller k_position="100" k_velocity="15.0" soft_lower_limit="${-0.785}" soft_upper_limit="${0.28}" />
             <dynamics damping="50" friction="1"/>
         </joint>

Commit message: wubble arm model updates

File: arrg/ua_robots/wubble_arm_description/urdf/wubble_arm.xacro (robot description, xacro)
@@ -153,5 +153,5 @@
                 <origin xyz="0.0 0.0 0.0" rpy="0 0 0" />
                 <geometry>
-                    <mesh filename="package://wubble_arm_description/meshes/convex/L0_base_link_convex.stlb"/>
+                    <mesh filename="package://wubble_arm_description/meshes/L0_base_link.stl"/>
                 </geometry>
             </collision>
@@ -174,5 +174,5 @@
                 <origin xyz="0.0 0.0 0.0" rpy="0 0 0" />
                 <geometry>
-                    <mesh filename="package://wubble_arm_description/meshes/convex/L1_shoulder_pitch_link_convex.stlb"/>
+                    <mesh filename="package://wubble_arm_description/meshes/L1_shoulder_pitch_link.stl"/>
                 </geometry>
             </collision>
@@ -195,5 +195,5 @@
                 <origin xyz="0.0 0.0545 0.0" rpy="0 0 0" />
                 <geometry>
-                    <mesh filename="package://wubble_arm_description/meshes/convex/L2_shoulder_yaw_link_convex.stlb"/>
+                    <mesh filename="package://wubble_arm_description/meshes/L2_shoulder_yaw_link.stl"/>
                 </geometry>
             </collision>
@@ -216,5 +216,5 @@
                 <origin xyz="0.0 0.0 0.0" rpy="0 0 0" />
                 <geometry>
-                    <mesh filename="package://wubble_arm_description/meshes/convex/L3_shoulder_roll_link_convex.stlb"/>
+                    <mesh filename="package://wubble_arm_description/meshes/L3_shoulder_roll_link.stl"/>
                 </geometry>
             </collision>
@@ -237,5 +237,5 @@
                 <origin xyz="0.03458 0.04399 0.026" rpy="0 0 0" />
                 <geometry>
-                    <mesh filename="package://wubble_arm_description/meshes/convex/L4_elbow_pitch_link_convex.stlb"/>
+                    <mesh filename="package://wubble_arm_description/meshes/L4_elbow_pitch_link.stl"/>
                 </geometry>
             </collision>
@@ -258,5 +258,5 @@
                 <origin xyz="0.025 0.0 0.0" rpy="0 0 0" />
                 <geometry>
-                    <mesh filename="package://wubble_arm_description/meshes/convex/L5_wrist_roll_link_convex.stlb"/>
+                    <mesh filename="package://wubble_arm_description/meshes/L5_wrist_roll_link.stl"/>
                 </geometry>
             </collision>
@@ -279,5 +279,5 @@
                 <origin xyz="0.0 0.0 0.0" rpy="0 0 0" />
                 <geometry>
-                    <mesh filename="package://wubble_arm_description/meshes/convex/L6_wrist_pitch_link_convex.stlb"/>
+                    <mesh filename="package://wubble_arm_description/meshes/L6_wrist_pitch_link.stl"/>
                 </geometry>
             </collision>
@@ -300,5 +300,5 @@
                 <origin xyz="0.0751 0 -0.002" rpy="0 0 0" />
                 <geometry>
-                    <mesh filename="package://wubble_arm_description/meshes/convex/L7_wrist_yaw_link_convex.stlb"/>
+                    <mesh filename="package://wubble_arm_description/meshes/L7_wrist_yaw_link.stl"/>
                 </geometry>
             </collision>
@@ -321,5 +321,5 @@
                 <origin xyz="0 0 0" rpy="0 0 0" />
                 <geometry>
-                    <mesh filename="package://wubble_arm_description/meshes/convex/L8_gripper_left_finger_convex.stlb"/>
+                    <mesh filename="package://wubble_arm_description/meshes/L8_gripper_left_finger.stl"/>
                 </geometry>
             </collision>
@@ -342,5 +342,5 @@
                 <origin xyz="0 0 0" rpy="0 0 0" />
                 <geometry>
-                    <mesh filename="package://wubble_arm_description/meshes/convex/L9_gripper_right_finger_convex.stlb"/>
+                    <mesh filename="package://wubble_arm_description/meshes/L9_gripper_right_finger.stl"/>
                 </geometry>
             </collision>

Commit message: Wubble2 model updates.

File: arrg/ua_robots/wubble_arm_description/urdf/wubble_arm.xacro (robot description, xacro)
@@ -149,4 +149,5 @@
                     <mesh filename="package://wubble_arm_description/meshes/L0_base_link.stl"/>
                 </geometry>
+                <material name="GunMetalBrushedAluminum" />
             </visual>
             <collision>
@@ -170,4 +171,5 @@
                     <mesh filename="package://wubble_arm_description/meshes/L1_shoulder_pitch_link.stl"/>
                 </geometry>
+                <material name="GunMetalBrushedAluminum" />
             </visual>
             <collision>
@@ -191,4 +193,5 @@
                     <mesh filename="package://wubble_arm_description/meshes/L2_shoulder_yaw_link.stl"/>
                 </geometry>
+                <material name="GunMetalBrushedAluminum" />
             </visual>
             <collision>
@@ -212,4 +215,5 @@
                     <mesh filename="package://wubble_arm_description/meshes/L3_shoulder_roll_link.stl"/>
                 </geometry>
+                <material name="GunMetalBrushedAluminum" />
             </visual>
             <collision>
@@ -233,4 +237,5 @@
                     <mesh filename="package://wubble_arm_description/meshes/L4_elbow_pitch_link.stl"/>
                 </geometry>
+                <material name="GunMetalBrushedAluminum" />
             </visual>
             <collision>
@@ -254,4 +259,5 @@
                     <mesh filename="package://wubble_arm_description/meshes/L5_wrist_roll_link.stl"/>
                 </geometry>
+                <material name="GunMetalBrushedAluminum" />
             </visual>
             <collision>
@@ -275,4 +281,5 @@
                     <mesh filename="package://wubble_arm_description/meshes/L6_wrist_pitch_link.stl"/>
                 </geometry>
+                <material name="GunMetalBrushedAluminum" />
             </visual>
             <collision>
@@ -296,4 +303,5 @@
                     <mesh filename="package://wubble_arm_description/meshes/L7_wrist_yaw_link.stl"/>
                 </geometry>
+                <material name="GunMetalBrushedAluminum" />
             </visual>
             <collision>
@@ -317,4 +325,5 @@
                     <mesh filename="package://wubble_arm_description/meshes/L8_gripper_left_finger.stl"/>
                 </geometry>
+                <material name="GunMetalBrushedAluminum" />
             </visual>
             <collision>
@@ -338,4 +347,5 @@
                     <mesh filename="package://wubble_arm_description/meshes/L9_gripper_right_finger.stl"/>
                 </geometry>
+                <material name="GunMetalBrushedAluminum" />
             </visual>
             <collision>

File: arrg/ua_robots/wubble_description/urdf/wubble2.urdf.xacro (robot description, xacro)
@@ -32,4 +32,5 @@
                 <mesh filename="package://wubble_description/meshes/wubble2_platform.stl"/>
             </geometry>
+            <material name="White" />
         </visual>
         <collision>
@@ -77,4 +78,5 @@
                 <mesh filename="package://wubble_description/meshes/head_base_link.stl"/>
             </geometry>
+            <material name="GunMetalBrushedAluminum" />
         </visual>
         <collision>
@@ -98,4 +100,5 @@
                 <mesh filename="package://wubble_description/meshes/head_pan_link.stl"/>
             </geometry>
+            <material name="GunMetalBrushedAluminum" />
         </visual>
         <collision>
@@ -119,4 +122,5 @@
                 <mesh filename="package://wubble_description/meshes/head_tilt_link.stl"/>
             </geometry>
+            <material name="GunMetalBrushedAluminum" />
         </visual>
         <collision>
@@ -173,4 +177,5 @@
                 <mesh filename="package://wubble_description/meshes/neck_laser_support_link.stl"/>
             </geometry>
+            <material name="GunMetalBrushedAluminum" />
         </visual>
         <collision>
@@ -194,4 +199,5 @@
                 <mesh filename="package://wubble_description/meshes/head_tilt_link.stl"/>
             </geometry>
+            <material name="GunMetalBrushedAluminum" />
         </visual>
         <collision>

Commit message: Replace shoulder yaw link. Modify joint limits on wubble arm.

File: arrg/ua_robots/wubble_arm_description/urdf/wubble_arm.xacro (robot description, xacro)
@@ -51,16 +51,16 @@
             <child link="L1_shoulder_pitch_link"/>
             <axis xyz="0 1 0"/>
-            <limit  lower="-2.13" upper="1.39" effort="300" velocity="1.17" />
-            <safety_controller k_position="100" k_velocity="15.0" soft_lower_limit="${-2.13}" soft_upper_limit="${1.39}" />
+            <limit  lower="-2.13" upper="1.40" effort="300" velocity="1.17" />
+            <safety_controller k_position="100" k_velocity="15.0" soft_lower_limit="${-2.13}" soft_upper_limit="${1.40}" />
             <dynamics damping="50" friction="1"/>
         </joint>
         <!-- Shoulder yaw joint -->
         <joint name="shoulder_yaw_joint" type="revolute" >
-            <origin xyz="0 0.064 0" rpy="0 0 0" />
+            <origin xyz="0.02899 0.06312 0" rpy="0 0 0" />
             <parent link="L1_shoulder_pitch_link" />
             <child link="L2_shoulder_yaw_link"/>
             <axis xyz="0 0 1"/>
-            <limit  lower="-1.90" upper="1.90" effort="300" velocity="1.17" />
-            <safety_controller k_position="100" k_velocity="15.0" soft_lower_limit="${-1.90}" soft_upper_limit="${1.90}" />
+            <limit  lower="-1.84" upper="1.58" effort="300" velocity="1.17" />
+            <safety_controller k_position="100" k_velocity="15.0" soft_lower_limit="${-1.84}" soft_upper_limit="${1.58}" />
             <dynamics damping="50" friction="1"/>
         </joint>
@@ -71,6 +71,6 @@
             <child link="L3_shoulder_roll_link"/>
             <axis xyz="0 1 0"/>
-            <limit  lower="-2.18" upper="2.18" effort="300" velocity="1.17" />
-            <safety_controller k_position="100" k_velocity="15.0" soft_lower_limit="${-2.18}" soft_upper_limit="${2.18}" />
+            <limit  lower="-1.99" upper="2.39" effort="300" velocity="1.17" />
+            <safety_controller k_position="100" k_velocity="15.0" soft_lower_limit="${-1.99}" soft_upper_limit="${2.39}" />
             <dynamics damping="50" friction="1"/>
         </joint>

Commit message: Goes with previous yaml changes.

File: arrg/ua_robots/wubble_arm_description/urdf/wubble_arm.xacro (robot description, xacro)
@@ -71,6 +71,6 @@
             <child link="L3_shoulder_roll_link"/>
             <axis xyz="0 1 0"/>
-            <limit  lower="-1.99" upper="2.39" effort="300" velocity="1.17" />
-            <safety_controller k_position="100" k_velocity="15.0" soft_lower_limit="${-1.99}" soft_upper_limit="${2.39}" />
+            <limit  lower="-2.19" upper="2.19" effort="300" velocity="1.17" />
+            <safety_controller k_position="100" k_velocity="15.0" soft_lower_limit="${-2.19}" soft_upper_limit="${2.19}" />
             <dynamics damping="50" friction="1"/>
         </joint>
