Commit message: Updated arm urdf and wrist stl

File: arrg/ua_robots/wubble_arm_description/urdf/wubble_arm.xacro (robot description, xacro)
@@ -57,5 +57,5 @@
         <!-- Shoulder yaw joint -->
         <joint name="shoulder_yaw_joint" type="revolute" >
-            <origin xyz="0.02899 0.06312 0" rpy="0 0 0" />
+            <origin xyz="0.029 0.063 0" rpy="0 0 0" />
             <parent link="L1_shoulder_pitch_link" />
             <child link="L2_shoulder_yaw_link"/>
@@ -67,5 +67,5 @@
         <!-- Shoulder roll joint -->
         <joint name="shoulder_roll_joint" type="revolute" >
-            <origin xyz="0 0.10582 0" rpy="0 0 0" />
+            <origin xyz="0 0.106 0" rpy="0 0 0" />
             <parent link="L2_shoulder_yaw_link" />
             <child link="L3_shoulder_roll_link"/>
@@ -87,5 +87,5 @@
         <!-- Wrist roll joint -->
         <joint name="wrist_roll_joint" type="revolute" >
-            <origin xyz="0.03308 0.02899 0" rpy="0 0 0" />
+            <origin xyz="0.033 0.029 0" rpy="0 0 0" />
             <parent link="L4_elbow_pitch_link" />
             <child link="L5_wrist_roll_link"/>
@@ -107,5 +107,5 @@
         <!-- Wrist yaw joint -->
         <joint name="wrist_yaw_joint" type="revolute" >
-            <origin xyz="0 0 0" rpy="0 0 0" />
+            <origin xyz="0.091 0 -0.002" rpy="0 0 0" />
             <parent link="L6_wrist_pitch_link" />
             <child link="L7_wrist_yaw_link"/>
@@ -117,5 +117,5 @@
         <!-- Left finger joint -->
         <joint name="left_finger_joint" type="revolute" >
-            <origin xyz="0.0791 0.021 -0.002" rpy="0 0 0" />
+            <origin xyz="-0.012 0.021 0" rpy="0 0 0" />
             <parent link="L7_wrist_yaw_link" />
             <child link="L8_left_finger_link"/>
@@ -127,5 +127,5 @@
         <!-- Right finger joint -->
         <joint name="right_finger_joint" type="revolute" >
-            <origin xyz="0.0791 -0.021 -0.002" rpy="0 0 0" />
+            <origin xyz="-0.012 -0.021 0" rpy="0 0 0" />
             <parent link="L7_wrist_yaw_link" />
             <child link="L9_right_finger_link"/>
@@ -140,10 +140,10 @@
                 <mass value="0.325" />
                 <origin xyz="0 0 0" rpy="0 0 0" />
-                <inertia ixx="1.0" ixy="0.0" ixz="0.0"
-                         iyy="1.0" iyz="0.0"
-                         izz="1.0" />
-            </inertial>
-            <visual>
-                <origin xyz="0.0 0.0 0.0" rpy="0 0 0" />
+                <inertia ixx="1.0" ixy="0" ixz="0"
+                         iyy="1.0" iyz="0"
+                         izz="1.0" />
+            </inertial>
+            <visual>
+                <origin xyz="0 0 0" rpy="0 0 0" />
                 <geometry>
                     <mesh filename="package://wubble_arm_description/meshes/L0_base_link.stl"/>
@@ -152,5 +152,5 @@
             </visual>
             <collision>
-                <origin xyz="0.0 0.0 0.0" rpy="0 0 0" />
+                <origin xyz="0 0 0" rpy="0 0 0" />
                 <geometry>
                     <mesh filename="package://wubble_arm_description/meshes/L0_base_link.stl"/>
@@ -162,10 +162,10 @@
                 <mass value="0.030" />
                 <origin xyz="0 0 0" rpy="0 0 0" />
-                <inertia ixx="1.0" ixy="0.0" ixz="0.0"
-                         iyy="1.0" iyz="0.0"
-                         izz="1.0" />
-            </inertial>
-            <visual>
-                <origin xyz="0.0 0.0 0.0" rpy="0 0 0" />
+                <inertia ixx="1.0" ixy="0" ixz="0"
+                         iyy="1.0" iyz="0"
+                         izz="1.0" />
+            </inertial>
+            <visual>
+                <origin xyz="0 0 0" rpy="0 0 0" />
                 <geometry>
                     <mesh filename="package://wubble_arm_description/meshes/L1_shoulder_pitch_link.stl"/>
@@ -174,5 +174,5 @@
             </visual>
             <collision>
-                <origin xyz="0.0 0.0 0.0" rpy="0 0 0" />
+                <origin xyz="0 0 0" rpy="0 0 0" />
                 <geometry>
                     <mesh filename="package://wubble_arm_description/meshes/L1_shoulder_pitch_link.stl"/>
@@ -184,10 +184,10 @@
                 <mass value="0.030" />
                 <origin xyz="0 0 0" rpy="0 0 0" />
-                <inertia ixx="1.0" ixy="0.0" ixz="0.0"
-                         iyy="1.0" iyz="0.0"
-                         izz="1.0" />
-            </inertial>
-            <visual>
-                <origin xyz="0.0 0.0545 0.0" rpy="0 0 0" />
+                <inertia ixx="1.0" ixy="0" ixz="0"
+                         iyy="1.0" iyz="0"
+                         izz="1.0" />
+            </inertial>
+            <visual>
+                <origin xyz="0 0.055 0" rpy="0 0 0" />
                 <geometry>
                     <mesh filename="package://wubble_arm_description/meshes/L2_shoulder_yaw_link.stl"/>
@@ -196,5 +196,5 @@
             </visual>
             <collision>
-                <origin xyz="0.0 0.0545 0.0" rpy="0 0 0" />
+                <origin xyz="0 0.0545 0" rpy="0 0 0" />
                 <geometry>
                     <mesh filename="package://wubble_arm_description/meshes/L2_shoulder_yaw_link.stl"/>
@@ -206,10 +206,10 @@
                 <mass value="0.030" />
                 <origin xyz="0 0 0" rpy="0 0 0" />
-                <inertia ixx="1.0" ixy="0.0" ixz="0.0"
-                         iyy="1.0" iyz="0.0"
-                         izz="1.0" />
-            </inertial>
-            <visual>
-                <origin xyz="0.0 0.0 0.0" rpy="0 0 0" />
+                <inertia ixx="1.0" ixy="0" ixz="0"
+                         iyy="1.0" iyz="0"
+                         izz="1.0" />
+            </inertial>
+            <visual>
+                <origin xyz="0 0 0" rpy="0 0 0" />
                 <geometry>
                     <mesh filename="package://wubble_arm_description/meshes/L3_shoulder_roll_link.stl"/>
@@ -218,5 +218,5 @@
             </visual>
             <collision>
-                <origin xyz="0.0 0.0 0.0" rpy="0 0 0" />
+                <origin xyz="0 0 0" rpy="0 0 0" />
                 <geometry>
                     <mesh filename="package://wubble_arm_description/meshes/L3_shoulder_roll_link.stl"/>
@@ -228,10 +228,10 @@
                 <mass value="0.030" />
                 <origin xyz="0 0 0" rpy="0 0 0" />
-                <inertia ixx="1.0" ixy="0.0" ixz="0.0"
-                         iyy="1.0" iyz="0.0"
-                         izz="1.0" />
-            </inertial>
-            <visual>
-                <origin xyz="0.03458 0.04399 0.026" rpy="0 0 0" />
+                <inertia ixx="1.0" ixy="0" ixz="0"
+                         iyy="1.0" iyz="0"
+                         izz="1.0" />
+            </inertial>
+            <visual>
+                <origin xyz="0.035 0.044 0.026" rpy="0 0 0" />
                 <geometry>
                     <mesh filename="package://wubble_arm_description/meshes/L4_elbow_pitch_link.stl"/>
@@ -240,5 +240,5 @@
             </visual>
             <collision>
-                <origin xyz="0.03458 0.04399 0.026" rpy="0 0 0" />
+                <origin xyz="0.035 0.044 0.026" rpy="0 0 0" />
                 <geometry>
                     <mesh filename="package://wubble_arm_description/meshes/L4_elbow_pitch_link.stl"/>
@@ -250,10 +250,10 @@
                 <mass value="0.030" />
                 <origin xyz="0 0 0" rpy="0 0 0" />
-                <inertia ixx="1.0" ixy="0.0" ixz="0.0"
-                         iyy="1.0" iyz="0.0"
-                         izz="1.0" />
-            </inertial>
-            <visual>
-                <origin xyz="0.025 0.0 0.0" rpy="0 0 0" />
+                <inertia ixx="1.0" ixy="0" ixz="0"
+                         iyy="1.0" iyz="0"
+                         izz="1.0" />
+            </inertial>
+            <visual>
+                <origin xyz="0.025 0 0" rpy="0 0 0" />
                 <geometry>
                     <mesh filename="package://wubble_arm_description/meshes/L5_wrist_roll_link.stl"/>
@@ -262,5 +262,5 @@
             </visual>
             <collision>
-                <origin xyz="0.025 0.0 0.0" rpy="0 0 0" />
+                <origin xyz="0.025 0 0" rpy="0 0 0" />
                 <geometry>
                     <mesh filename="package://wubble_arm_description/meshes/L5_wrist_roll_link.stl"/>
@@ -272,10 +272,10 @@
                 <mass value="0.030" />
                 <origin xyz="0 0 0" rpy="0 0 0" />
-                <inertia ixx="1.0" ixy="0.0" ixz="0.0"
-                         iyy="1.0" iyz="0.0"
-                         izz="1.0" />
-            </inertial>
-            <visual>
-                <origin xyz="0.0 0.0 0.0" rpy="0 0 0" />
+                <inertia ixx="1.0" ixy="0" ixz="0"
+                         iyy="1.0" iyz="0"
+                         izz="1.0" />
+            </inertial>
+            <visual>
+                <origin xyz="0 0 0" rpy="0 0 0" />
                 <geometry>
                     <mesh filename="package://wubble_arm_description/meshes/L6_wrist_pitch_link.stl"/>
@@ -284,5 +284,5 @@
             </visual>
             <collision>
-                <origin xyz="0.0 0.0 0.0" rpy="0 0 0" />
+                <origin xyz="0 0 0" rpy="0 0 0" />
                 <geometry>
                     <mesh filename="package://wubble_arm_description/meshes/L6_wrist_pitch_link.stl"/>
@@ -294,10 +294,10 @@
                 <mass value="0.030" />
                 <origin xyz="0 0 0" rpy="0 0 0" />
-                <inertia ixx="1.0" ixy="0.0" ixz="0.0"
-                         iyy="1.0" iyz="0.0"
-                         izz="1.0" />
-            </inertial>
-            <visual>
-                <origin xyz="0.0751 0 -0.002" rpy="0 0 0" />
+                <inertia ixx="1.0" ixy="0" ixz="0"
+                         iyy="1.0" iyz="0"
+                         izz="1.0" />
+            </inertial>
+            <visual>
+                <origin xyz="0 0 0" rpy="0 0 0" />
                 <geometry>
                     <mesh filename="package://wubble_arm_description/meshes/L7_wrist_yaw_link.stl"/>
@@ -306,5 +306,5 @@
             </visual>
             <collision>
-                <origin xyz="0.0751 0 -0.002" rpy="0 0 0" />
+                <origin xyz="0 0 0" rpy="0 0 0" />
                 <geometry>
                     <mesh filename="package://wubble_arm_description/meshes/L7_wrist_yaw_link.stl"/>
@@ -316,6 +316,6 @@
                 <mass value="0.030" />
                 <origin xyz="0 0 0" rpy="0 0 0" />
-                <inertia ixx="1.0" ixy="0.0" ixz="0.0"
-                         iyy="1.0" iyz="0.0"
+                <inertia ixx="1.0" ixy="0" ixz="0"
+                         iyy="1.0" iyz="0"
                          izz="1.0" />
             </inertial>
@@ -338,6 +338,6 @@
                 <mass value="0.030" />
                 <origin xyz="0 0 0" rpy="0 0 0" />
-                <inertia ixx="1.0" ixy="0.0" ixz="0.0"
-                         iyy="1.0" iyz="0.0"
+                <inertia ixx="1.0" ixy="0" ixz="0"
+                         iyy="1.0" iyz="0"
                          izz="1.0" />
             </inertial>

Commit message: fix urdf

File: arrg/ua_robots/wubble_arm_description/urdf/wubble_arm.xacro (robot description, xacro)
@@ -107,5 +107,5 @@
         <!-- Wrist yaw joint -->
         <joint name="wrist_yaw_joint" type="revolute" >
-            <origin xyz="0.091 0 -0.002" rpy="0 0 0" />
+            <origin xyz="0 0 -0.002" rpy="0 0 0" />
             <parent link="L6_wrist_pitch_link" />
             <child link="L7_wrist_yaw_link"/>
@@ -117,5 +117,5 @@
         <!-- Left finger joint -->
         <joint name="left_finger_joint" type="revolute" >
-            <origin xyz="-0.012 0.021 0" rpy="0 0 0" />
+            <origin xyz="${0.091-0.012} 0.021 0" rpy="0 0 0" />
             <parent link="L7_wrist_yaw_link" />
             <child link="L8_left_finger_link"/>
@@ -127,5 +127,5 @@
         <!-- Right finger joint -->
         <joint name="right_finger_joint" type="revolute" >
-            <origin xyz="-0.012 -0.021 0" rpy="0 0 0" />
+            <origin xyz="${0.091-0.012} -0.021 0" rpy="0 0 0" />
             <parent link="L7_wrist_yaw_link" />
             <child link="L9_right_finger_link"/>
@@ -299,5 +299,5 @@
             </inertial>
             <visual>
-                <origin xyz="0 0 0" rpy="0 0 0" />
+                <origin xyz="0.091 0 0" rpy="0 0 0" />
                 <geometry>
                     <mesh filename="package://wubble_arm_description/meshes/L7_wrist_yaw_link.stl"/>
@@ -306,5 +306,5 @@
             </visual>
             <collision>
-                <origin xyz="0 0 0" rpy="0 0 0" />
+                <origin xyz="0.091 0 0" rpy="0 0 0" />
                 <geometry>
                     <mesh filename="package://wubble_arm_description/meshes/L7_wrist_yaw_link.stl"/>
