Commit message: New arm design is in, urdf points to stl models for now, dae models are not very well supported in cturtle

File: arrg/ua_robots/wubble_arm_description/urdf/wubble_arm.xacro (robot description, xacro)
@@ -51,25 +51,25 @@
             <child link="L1_shoulder_pitch_link"/>
             <axis xyz="0 1 0"/>
-            <limit  lower="-2.13" upper="1.40" effort="300" velocity="1.17" />
-            <safety_controller k_position="100" k_velocity="15.0" soft_lower_limit="${-2.13}" soft_upper_limit="${1.40}" />
+            <limit  lower="-2.595" upper="1.025" effort="300" velocity="1.17" />
+            <safety_controller k_position="100" k_velocity="15.0" soft_lower_limit="${-2.595}" soft_upper_limit="${1.025}" />
             <dynamics damping="50" friction="1"/>
         </joint>
         <!-- Shoulder yaw joint -->
         <joint name="shoulder_yaw_joint" type="revolute" >
-            <origin xyz="0.029 0.063 0" rpy="0 0 0" />
+            <origin xyz="0.069 0.029 -0.029" rpy="0 0 0" />
             <parent link="L1_shoulder_pitch_link" />
             <child link="L2_shoulder_yaw_link"/>
             <axis xyz="0 0 1"/>
-            <limit  lower="-1.84" upper="1.58" effort="300" velocity="1.17" />
-            <safety_controller k_position="100" k_velocity="15.0" soft_lower_limit="${-1.84}" soft_upper_limit="${1.58}" />
+            <limit  lower="-3.24" upper="1.03" effort="300" velocity="1.17" />
+            <safety_controller k_position="100" k_velocity="15.0" soft_lower_limit="${-3.24}" soft_upper_limit="${1.03}" />
             <dynamics damping="50" friction="1"/>
         </joint>
         <!-- Shoulder roll joint -->
         <joint name="shoulder_roll_joint" type="revolute" >
-            <origin xyz="0 0.106 0" rpy="0 0 0" />
+            <origin xyz="0 0.1074 0" rpy="0 0 0" />
             <parent link="L2_shoulder_yaw_link" />
             <child link="L3_shoulder_roll_link"/>
             <axis xyz="0 1 0"/>
-            <limit  lower="-2.19" upper="2.19" effort="300" velocity="1.17" />
+            <limit  lower="-0.61" upper="3.77" effort="300" velocity="1.17" />
             <safety_controller k_position="100" k_velocity="15.0" soft_lower_limit="${-2.19}" soft_upper_limit="${2.19}" />
             <dynamics damping="50" friction="1"/>
@@ -77,5 +77,5 @@
         <!-- Elbow pitch joint -->
         <joint name="elbow_pitch_joint" type="revolute" >
-            <origin xyz="0.029 0.184 0" rpy="0 0 0" />
+            <origin xyz="0.029 0.132 0" rpy="0 0 0" />
             <parent link="L3_shoulder_roll_link" />
             <child link="L4_elbow_pitch_link"/>
@@ -87,5 +87,5 @@
         <!-- Wrist roll joint -->
         <joint name="wrist_roll_joint" type="revolute" >
-            <origin xyz="0.033 0.029 0" rpy="0 0 0" />
+            <origin xyz="0.034 0.029 0" rpy="0 0 0" />
             <parent link="L4_elbow_pitch_link" />
             <child link="L5_wrist_roll_link"/>
@@ -97,9 +97,9 @@
         <!-- Wrist pitch joint -->
         <joint name="wrist_pitch_joint" type="revolute" >
-            <origin xyz="0.228 0 0" rpy="0 0 0" />
+            <origin xyz="0.119 0 0" rpy="0 0 0" />
             <parent link="L5_wrist_roll_link" />
             <child link="L6_wrist_pitch_link"/>
             <axis xyz="0 1 0"/>
-            <limit  lower="-0.61" upper="2.27" effort="300" velocity="1.17" />
+            <limit  lower="-2.115" upper="2.61" effort="300" velocity="1.17" />
             <safety_controller k_position="100" k_velocity="15.0" soft_lower_limit="${-0.61}" soft_upper_limit="${2.27}" />
             <dynamics damping="50" friction="1"/>
@@ -107,9 +107,9 @@
         <!-- Wrist yaw joint -->
         <joint name="wrist_yaw_joint" type="revolute" >
-            <origin xyz="0 0 -0.002" rpy="0 0 0" />
+            <origin xyz="0.0925 0 0" rpy="0 0 0" />
             <parent link="L6_wrist_pitch_link" />
             <child link="L7_wrist_yaw_link"/>
-            <axis xyz="0 0 1"/>
-            <limit  lower="-1.66" upper="1.62" effort="300" velocity="1.17" />
+            <axis xyz="1 0 0"/>
+            <limit  lower="-2.61" upper="2.61" effort="300" velocity="1.17" />
             <safety_controller k_position="100" k_velocity="15.0" soft_lower_limit="${-1.66}" soft_upper_limit="${1.62}" />
             <dynamics damping="50" friction="1"/>
@@ -117,5 +117,5 @@
         <!-- Left finger joint -->
         <joint name="left_finger_joint" type="revolute" >
-            <origin xyz="${0.091-0.012} 0.021 0" rpy="0 0 0" />
+            <origin xyz="0.0421 0.021 0" rpy="0 0 0" />
             <parent link="L7_wrist_yaw_link" />
             <child link="L8_left_finger_link"/>
@@ -127,5 +127,5 @@
         <!-- Right finger joint -->
         <joint name="right_finger_joint" type="revolute" >
-            <origin xyz="${0.091-0.012} -0.021 0" rpy="0 0 0" />
+            <origin xyz="0.0421 -0.021 0" rpy="0 0 0" />
             <parent link="L7_wrist_yaw_link" />
             <child link="L9_right_finger_link"/>
@@ -147,12 +147,12 @@
                 <origin xyz="0 0 0" rpy="0 0 0" />
                 <geometry>
-                    <mesh filename="package://wubble_arm_description/meshes/collada/L0_base_link.dae"/>
-                </geometry>
-                <material name="GunMetalBrushedAluminum" />
-            </visual>
-            <collision>
-                <origin xyz="0 0 0" rpy="0 0 0" />
-                <geometry>
-                    <mesh filename="package://wubble_arm_description/meshes/collada/L0_base_link.dae"/>
+                    <mesh filename="package://wubble_arm_description/meshes/L0_base_link.stl"/>
+                </geometry>
+                <material name="Green" />
+            </visual>
+            <collision>
+                <origin xyz="0 0 0" rpy="0 0 0" />
+                <geometry>
+                    <mesh filename="package://wubble_arm_description/meshes/L0_base_link.stl"/>
                 </geometry>
             </collision>
@@ -169,12 +169,12 @@
                 <origin xyz="0 0 0" rpy="0 0 0" />
                 <geometry>
-                    <mesh filename="package://wubble_arm_description/meshes/collada/L1_shoulder_pitch_link.dae"/>
-                </geometry>
-                <material name="GunMetalBrushedAluminum" />
-            </visual>
-            <collision>
-                <origin xyz="0 0 0" rpy="0 0 0" />
-                <geometry>
-                    <mesh filename="package://wubble_arm_description/meshes/collada/L1_shoulder_pitch_link.dae"/>
+                    <mesh filename="package://wubble_arm_description/meshes/L1_shoulder_pitch_link.stl"/>
+                </geometry>
+                <material name="Grey" />
+            </visual>
+            <collision>
+                <origin xyz="0 0 0" rpy="0 0 0" />
+                <geometry>
+                    <mesh filename="package://wubble_arm_description/meshes/L1_shoulder_pitch_link.stl"/>
                 </geometry>
             </collision>
@@ -191,12 +191,12 @@
                 <origin xyz="0 0.055 0" rpy="0 0 0" />
                 <geometry>
-                    <mesh filename="package://wubble_arm_description/meshes/collada/L2_shoulder_yaw_link.dae"/>
-                </geometry>
-                <material name="GunMetalBrushedAluminum" />
+                    <mesh filename="package://wubble_arm_description/meshes/L2_shoulder_yaw_link.stl"/>
+                </geometry>
+                <material name="Blue" />
             </visual>
             <collision>
                 <origin xyz="0 0.0545 0" rpy="0 0 0" />
                 <geometry>
-                    <mesh filename="package://wubble_arm_description/meshes/collada/L2_shoulder_yaw_link.dae"/>
+                    <mesh filename="package://wubble_arm_description/meshes/L2_shoulder_yaw_link.stl"/>
                 </geometry>
             </collision>
@@ -213,12 +213,12 @@
                 <origin xyz="0 0 0" rpy="0 0 0" />
                 <geometry>
-                    <mesh filename="package://wubble_arm_description/meshes/collada/L3_shoulder_roll_link.dae"/>
-                </geometry>
-                <material name="GunMetalBrushedAluminum" />
-            </visual>
-            <collision>
-                <origin xyz="0 0 0" rpy="0 0 0" />
-                <geometry>
-                    <mesh filename="package://wubble_arm_description/meshes/collada/L3_shoulder_roll_link.dae"/>
+                    <mesh filename="package://wubble_arm_description/meshes/L3_shoulder_roll_link.stl"/>
+                </geometry>
+                <material name="Green" />
+            </visual>
+            <collision>
+                <origin xyz="0 0 0" rpy="0 0 0" />
+                <geometry>
+                    <mesh filename="package://wubble_arm_description/meshes/L3_shoulder_roll_link.stl"/>
                 </geometry>
             </collision>
@@ -235,12 +235,12 @@
                 <origin xyz="0.035 0.044 0.026" rpy="0 0 0" />
                 <geometry>
-                    <mesh filename="package://wubble_arm_description/meshes/collada/L4_elbow_pitch_link.dae"/>
-                </geometry>
-                <material name="GunMetalBrushedAluminum" />
+                    <mesh filename="package://wubble_arm_description/meshes/L4_elbow_pitch_link.stl"/>
+                </geometry>
+                <material name="Grey" />
             </visual>
             <collision>
                 <origin xyz="0.035 0.044 0.026" rpy="0 0 0" />
                 <geometry>
-                    <mesh filename="package://wubble_arm_description/meshes/collada/L4_elbow_pitch_link.dae"/>
+                    <mesh filename="package://wubble_arm_description/meshes/L4_elbow_pitch_link.stl"/>
                 </geometry>
             </collision>
@@ -257,12 +257,12 @@
                 <origin xyz="0.025 0 0" rpy="0 0 0" />
                 <geometry>
-                    <mesh filename="package://wubble_arm_description/meshes/collada/L5_wrist_roll_link.dae"/>
-                </geometry>
-                <material name="GunMetalBrushedAluminum" />
+                    <mesh filename="package://wubble_arm_description/meshes/L5_wrist_roll_link.stl"/>
+                </geometry>
+                <material name="Blue" />
             </visual>
             <collision>
                 <origin xyz="0.025 0 0" rpy="0 0 0" />
                 <geometry>
-                    <mesh filename="package://wubble_arm_description/meshes/collada/L5_wrist_roll_link.dae"/>
+                    <mesh filename="package://wubble_arm_description/meshes/L5_wrist_roll_link.stl"/>
                 </geometry>
             </collision>
@@ -279,12 +279,12 @@
                 <origin xyz="0 0 0" rpy="0 0 0" />
                 <geometry>
-                    <mesh filename="package://wubble_arm_description/meshes/collada/L6_wrist_pitch_link.dae"/>
-                </geometry>
-                <material name="GunMetalBrushedAluminum" />
-            </visual>
-            <collision>
-                <origin xyz="0 0 0" rpy="0 0 0" />
-                <geometry>
-                    <mesh filename="package://wubble_arm_description/meshes/collada/L6_wrist_pitch_link.dae"/>
+                    <mesh filename="package://wubble_arm_description/meshes/L6_wrist_pitch_link.stl"/>
+                </geometry>
+                <material name="Green" />
+            </visual>
+            <collision>
+                <origin xyz="0 0 0" rpy="0 0 0" />
+                <geometry>
+                    <mesh filename="package://wubble_arm_description/meshes/L6_wrist_pitch_link.stl"/>
                 </geometry>
             </collision>
@@ -299,14 +299,14 @@
             </inertial>
             <visual>
-                <origin xyz="0.091 0 0" rpy="0 0 0" />
-                <geometry>
-                    <mesh filename="package://wubble_arm_description/meshes/collada/L7_wrist_yaw_link.dae"/>
-                </geometry>
-                <material name="GunMetalBrushedAluminum" />
-            </visual>
-            <collision>
-                <origin xyz="0.091 0 0" rpy="0 0 0" />
-                <geometry>
-                    <mesh filename="package://wubble_arm_description/meshes/collada/L7_wrist_yaw_link.dae"/>
+                <origin xyz="0.0541 0 0" rpy="0 0 0" />
+                <geometry>
+                    <mesh filename="package://wubble_arm_description/meshes/L7_wrist_yaw_link.stl"/>
+                </geometry>
+                <material name="Grey" />
+            </visual>
+            <collision>
+                <origin xyz="-0.0541 0 0" rpy="0 0 0" />
+                <geometry>
+                    <mesh filename="package://wubble_arm_description/meshes/L7_wrist_yaw_link.stl"/>
                 </geometry>
             </collision>
@@ -323,12 +323,12 @@
                 <origin xyz="0 0 0" rpy="0 0 0" />
                 <geometry>
-                    <mesh filename="package://wubble_arm_description/meshes/collada/L8_gripper_left_finger.dae"/>
-                </geometry>
-                <material name="GunMetalBrushedAluminum" />
-            </visual>
-            <collision>
-                <origin xyz="0 0 0" rpy="0 0 0" />
-                <geometry>
-                    <mesh filename="package://wubble_arm_description/meshes/collada/L8_gripper_left_finger.dae"/>
+                    <mesh filename="package://wubble_arm_description/meshes/L8_gripper_left_finger.stl"/>
+                </geometry>
+                <material name="Blue" />
+            </visual>
+            <collision>
+                <origin xyz="0 0 0" rpy="0 0 0" />
+                <geometry>
+                    <mesh filename="package://wubble_arm_description/meshes/L8_gripper_left_finger.stl"/>
                 </geometry>
             </collision>
@@ -345,12 +345,12 @@
                 <origin xyz="0 0 0" rpy="0 0 0" />
                 <geometry>
-                    <mesh filename="package://wubble_arm_description/meshes/collada/L9_gripper_right_finger.dae"/>
-                </geometry>
-                <material name="GunMetalBrushedAluminum" />
-            </visual>
-            <collision>
-                <origin xyz="0 0 0" rpy="0 0 0" />
-                <geometry>
-                    <mesh filename="package://wubble_arm_description/meshes/collada/L9_gripper_right_finger.dae"/>
+                    <mesh filename="package://wubble_arm_description/meshes/L9_gripper_right_finger.stl"/>
+                </geometry>
+                <material name="Green" />
+            </visual>
+            <collision>
+                <origin xyz="0 0 0" rpy="0 0 0" />
+                <geometry>
+                    <mesh filename="package://wubble_arm_description/meshes/L9_gripper_right_finger.stl"/>
                 </geometry>
             </collision>
