Commit message: Update joint names and all configuration files

File: arrg/ua_robots/wubble_arm_description/urdf/wubble_arm.xacro (robot description, xacro)
@@ -51,46 +51,46 @@
             <child link="L1_shoulder_pitch_link"/>
             <axis xyz="0 1 0"/>
-            <limit  lower="-2.595" upper="1.025" effort="300" velocity="1.17" />
-            <safety_controller k_position="100" k_velocity="15.0" soft_lower_limit="${-2.595}" soft_upper_limit="${1.025}" />
-            <dynamics damping="50" friction="1"/>
-        </joint>
-        <!-- Shoulder yaw joint -->
-        <joint name="shoulder_yaw_joint" type="revolute" >
+            <limit  lower="-2.523" upper="1.048" effort="300" velocity="1.17" />
+            <safety_controller k_position="100" k_velocity="15.0" soft_lower_limit="${-2.523}" soft_upper_limit="${1.048}" />
+            <dynamics damping="50" friction="1"/>
+        </joint>
+        <!-- Shoulder pan joint -->
+        <joint name="shoulder_pan_joint" type="revolute" >
             <origin xyz="0.069 0.029 -0.029" rpy="0 0 0" />
             <parent link="L1_shoulder_pitch_link" />
-            <child link="L2_shoulder_yaw_link"/>
+            <child link="L2_shoulder_pan_link"/>
             <axis xyz="0 0 1"/>
-            <limit  lower="-3.24" upper="1.03" effort="300" velocity="1.17" />
-            <safety_controller k_position="100" k_velocity="15.0" soft_lower_limit="${-3.24}" soft_upper_limit="${1.03}" />
-            <dynamics damping="50" friction="1"/>
-        </joint>
-        <!-- Shoulder roll joint -->
-        <joint name="shoulder_roll_joint" type="revolute" >
+            <limit  lower="-3.351" upper="0.905" effort="300" velocity="1.17" />
+            <safety_controller k_position="100" k_velocity="15.0" soft_lower_limit="${-3.351}" soft_upper_limit="${0.905}" />
+            <dynamics damping="50" friction="1"/>
+        </joint>
+        <!-- Uppperarm roll joint -->
+        <joint name="upperarm_roll_joint" type="revolute" >
             <origin xyz="0 0.1074 0" rpy="0 0 0" />
-            <parent link="L2_shoulder_yaw_link" />
-            <child link="L3_shoulder_roll_link"/>
+            <parent link="L2_shoulder_pan_link" />
+            <child link="L3_upperarm_roll_link"/>
             <axis xyz="0 1 0"/>
-            <limit  lower="-0.61" upper="3.77" effort="300" velocity="1.17" />
-            <safety_controller k_position="100" k_velocity="15.0" soft_lower_limit="${-2.19}" soft_upper_limit="${2.19}" />
-            <dynamics damping="50" friction="1"/>
-        </joint>
-        <!-- Elbow pitch joint -->
-        <joint name="elbow_pitch_joint" type="revolute" >
+            <limit  lower="-0.629" upper="3.75" effort="300" velocity="1.17" />
+            <safety_controller k_position="100" k_velocity="15.0" soft_lower_limit="${-0.629}" soft_upper_limit="${3.75}" />
+            <dynamics damping="50" friction="1"/>
+        </joint>
+        <!-- Elbow flex joint -->
+        <joint name="elbow_flex_joint" type="revolute" >
             <origin xyz="0.029 0.132 0" rpy="0 0 0" />
-            <parent link="L3_shoulder_roll_link" />
-            <child link="L4_elbow_pitch_link"/>
+            <parent link="L3_upperarm_roll_link" />
+            <child link="L4_elbow_flex_link"/>
             <axis xyz="0 0 1"/>
-            <limit  lower="-1.53" upper="1.80" effort="300" velocity="1.17" />
-            <safety_controller k_position="100" k_velocity="15.0" soft_lower_limit="${-1.53}" soft_upper_limit="${1.80}" />
-            <dynamics damping="50" friction="1"/>
-        </joint>
-        <!-- Wrist roll joint -->
-        <joint name="wrist_roll_joint" type="revolute" >
+            <limit  lower="-1.652" upper="1.846" effort="300" velocity="1.17" />
+            <safety_controller k_position="100" k_velocity="15.0" soft_lower_limit="${-1.652}" soft_upper_limit="${1.846}" />
+            <dynamics damping="50" friction="1"/>
+        </joint>
+        <!-- Forearm roll joint -->
+        <joint name="forearm_roll_joint" type="revolute" >
             <origin xyz="0.034 0.029 0" rpy="0 0 0" />
-            <parent link="L4_elbow_pitch_link" />
-            <child link="L5_wrist_roll_link"/>
+            <parent link="L4_elbow_flex_link" />
+            <child link="L5_forearm_roll_link"/>
             <axis xyz="1 0 0"/>
-            <limit  lower="-2.61" upper="2.61" effort="300" velocity="1.17" />
-            <safety_controller k_position="100" k_velocity="15.0" soft_lower_limit="${-2.61}" soft_upper_limit="${2.61}" />
+            <limit  lower="-2.521" upper="2.71" effort="300" velocity="1.17" />
+            <safety_controller k_position="100" k_velocity="15.0" soft_lower_limit="${-2.521}" soft_upper_limit="${2.71}" />
             <dynamics damping="50" friction="1"/>
         </joint>
@@ -98,19 +98,19 @@
         <joint name="wrist_pitch_joint" type="revolute" >
             <origin xyz="0.119 0 0" rpy="0 0 0" />
-            <parent link="L5_wrist_roll_link" />
+            <parent link="L5_forearm_roll_link" />
             <child link="L6_wrist_pitch_link"/>
             <axis xyz="0 1 0"/>
-            <limit  lower="-2.115" upper="2.61" effort="300" velocity="1.17" />
-            <safety_controller k_position="100" k_velocity="15.0" soft_lower_limit="${-0.61}" soft_upper_limit="${2.27}" />
-            <dynamics damping="50" friction="1"/>
-        </joint>
-        <!-- Wrist yaw joint -->
-        <joint name="wrist_yaw_joint" type="revolute" >
+            <limit  lower="-2.158" upper="2.613" effort="300" velocity="1.17" />
+            <safety_controller k_position="100" k_velocity="15.0" soft_lower_limit="${-2.158}" soft_upper_limit="${2.613}" />
+            <dynamics damping="50" friction="1"/>
+        </joint>
+        <!-- Wrist roll joint -->
+        <joint name="wrist_roll_joint" type="revolute" >
             <origin xyz="0.0925 0 0" rpy="0 0 0" />
             <parent link="L6_wrist_pitch_link" />
-            <child link="L7_wrist_yaw_link"/>
+            <child link="L7_wrist_roll_link"/>
             <axis xyz="1 0 0"/>
-            <limit  lower="-2.61" upper="2.61" effort="300" velocity="1.17" />
-            <safety_controller k_position="100" k_velocity="15.0" soft_lower_limit="${-1.66}" soft_upper_limit="${1.62}" />
+            <limit  lower="-2.597" upper="2.633" effort="300" velocity="1.17" />
+            <safety_controller k_position="100" k_velocity="15.0" soft_lower_limit="${-2.597}" soft_upper_limit="${2.633}" />
             <dynamics damping="50" friction="1"/>
         </joint>
@@ -118,5 +118,5 @@
         <joint name="left_finger_joint" type="revolute" >
             <origin xyz="0.0421 0.021 0" rpy="0 0 0" />
-            <parent link="L7_wrist_yaw_link" />
+            <parent link="L7_wrist_roll_link" />
             <child link="L8_left_finger_link"/>
             <axis xyz="0 0 1"/>
@@ -128,5 +128,5 @@
         <joint name="right_finger_joint" type="revolute" >
             <origin xyz="0.0421 -0.021 0" rpy="0 0 0" />
-            <parent link="L7_wrist_yaw_link" />
+            <parent link="L7_wrist_roll_link" />
             <child link="L9_right_finger_link"/>
             <axis xyz="0 0 1"/>
@@ -180,5 +180,5 @@
             </collision>
         </link>
-        <link name="L2_shoulder_yaw_link">
+        <link name="L2_shoulder_pan_link">
             <inertial>
                 <mass value="0.030" />
@@ -191,5 +191,5 @@
                 <origin xyz="0 0.055 0" rpy="0 0 0" />
                 <geometry>
-                    <mesh filename="package://wubble_arm_description/meshes/L2_shoulder_yaw_link.stl"/>
+                    <mesh filename="package://wubble_arm_description/meshes/L2_shoulder_pan_link.stl"/>
                 </geometry>
                 <material name="Blue" />
@@ -198,20 +198,20 @@
                 <origin xyz="0 0.0545 0" rpy="0 0 0" />
                 <geometry>
-                    <mesh filename="package://wubble_arm_description/meshes/L2_shoulder_yaw_link.stl"/>
-                </geometry>
-            </collision>
-        </link>
-        <link name="L3_shoulder_roll_link">
-            <inertial>
-                <mass value="0.030" />
-                <origin xyz="0 0 0" rpy="0 0 0" />
-                <inertia ixx="1.0" ixy="0" ixz="0"
-                         iyy="1.0" iyz="0"
-                         izz="1.0" />
-            </inertial>
-            <visual>
-                <origin xyz="0 0 0" rpy="0 0 0" />
-                <geometry>
-                    <mesh filename="package://wubble_arm_description/meshes/L3_shoulder_roll_link.stl"/>
+                    <mesh filename="package://wubble_arm_description/meshes/L2_shoulder_pan_link.stl"/>
+                </geometry>
+            </collision>
+        </link>
+        <link name="L3_upperarm_roll_link">
+            <inertial>
+                <mass value="0.030" />
+                <origin xyz="0 0 0" rpy="0 0 0" />
+                <inertia ixx="1.0" ixy="0" ixz="0"
+                         iyy="1.0" iyz="0"
+                         izz="1.0" />
+            </inertial>
+            <visual>
+                <origin xyz="0 0 0" rpy="0 0 0" />
+                <geometry>
+                    <mesh filename="package://wubble_arm_description/meshes/L3_upperarm_roll_link.stl"/>
                 </geometry>
                 <material name="Green" />
@@ -220,9 +220,9 @@
                 <origin xyz="0 0 0" rpy="0 0 0" />
                 <geometry>
-                    <mesh filename="package://wubble_arm_description/meshes/L3_shoulder_roll_link.stl"/>
-                </geometry>
-            </collision>
-        </link>
-        <link name="L4_elbow_pitch_link">
+                    <mesh filename="package://wubble_arm_description/meshes/L3_upperarm_roll_link.stl"/>
+                </geometry>
+            </collision>
+        </link>
+        <link name="L4_elbow_flex_link">
             <inertial>
                 <mass value="0.030" />
@@ -235,5 +235,5 @@
                 <origin xyz="0.035 0.044 0.026" rpy="0 0 0" />
                 <geometry>
-                    <mesh filename="package://wubble_arm_description/meshes/L4_elbow_pitch_link.stl"/>
+                    <mesh filename="package://wubble_arm_description/meshes/L4_elbow_flex_link.stl"/>
                 </geometry>
                 <material name="Grey" />
@@ -242,9 +242,9 @@
                 <origin xyz="0.035 0.044 0.026" rpy="0 0 0" />
                 <geometry>
-                    <mesh filename="package://wubble_arm_description/meshes/L4_elbow_pitch_link.stl"/>
-                </geometry>
-            </collision>
-        </link>
-        <link name="L5_wrist_roll_link">
+                    <mesh filename="package://wubble_arm_description/meshes/L4_elbow_flex_link.stl"/>
+                </geometry>
+            </collision>
+        </link>
+        <link name="L5_forearm_roll_link">
             <inertial>
                 <mass value="0.030" />
@@ -257,5 +257,5 @@
                 <origin xyz="0.025 0 0" rpy="0 0 0" />
                 <geometry>
-                    <mesh filename="package://wubble_arm_description/meshes/L5_wrist_roll_link.stl"/>
+                    <mesh filename="package://wubble_arm_description/meshes/L5_forearm_roll_link.stl"/>
                 </geometry>
                 <material name="Blue" />
@@ -264,5 +264,5 @@
                 <origin xyz="0.025 0 0" rpy="0 0 0" />
                 <geometry>
-                    <mesh filename="package://wubble_arm_description/meshes/L5_wrist_roll_link.stl"/>
+                    <mesh filename="package://wubble_arm_description/meshes/L5_forearm_roll_link.stl"/>
                 </geometry>
             </collision>
@@ -290,5 +290,5 @@
             </collision>
         </link>
-        <link name="L7_wrist_yaw_link">
+        <link name="L7_wrist_roll_link">
             <inertial>
                 <mass value="0.030" />
@@ -301,5 +301,5 @@
                 <origin xyz="0.0541 0 0" rpy="0 0 0" />
                 <geometry>
-                    <mesh filename="package://wubble_arm_description/meshes/L7_wrist_yaw_link.stl"/>
+                    <mesh filename="package://wubble_arm_description/meshes/L7_wrist_roll_link.stl"/>
                 </geometry>
                 <material name="Grey" />
@@ -308,5 +308,5 @@
                 <origin xyz="-0.0541 0 0" rpy="0 0 0" />
                 <geometry>
-                    <mesh filename="package://wubble_arm_description/meshes/L7_wrist_yaw_link.stl"/>
+                    <mesh filename="package://wubble_arm_description/meshes/L7_wrist_roll_link.stl"/>
                 </geometry>
             </collision>
@@ -362,17 +362,27 @@
             <mechanicalReduction>1.0</mechanicalReduction>
         </transmission>
-        <transmission type="pr2_mechanism_model/SimpleTransmission" name="shoulder_yaw_trans">
-            <actuator name="shoulder_yaw_motor" />
-            <joint name="shoulder_yaw_joint" />
-            <mechanicalReduction>1.0</mechanicalReduction>
-        </transmission>
-        <transmission type="pr2_mechanism_model/SimpleTransmission" name="shoulder_roll_trans">
-            <actuator name="shoulder_roll_motor" />
-            <joint name="shoulder_roll_joint" />
-            <mechanicalReduction>1.0</mechanicalReduction>
-        </transmission>
-        <transmission type="pr2_mechanism_model/SimpleTransmission" name="elbow_pitch_trans">
-            <actuator name="elbow_pitch_motor" />
-            <joint name="elbow_pitch_joint" />
+        <transmission type="pr2_mechanism_model/SimpleTransmission" name="shoulder_pan_trans">
+            <actuator name="shoulder_pan_motor" />
+            <joint name="shoulder_pan_joint" />
+            <mechanicalReduction>1.0</mechanicalReduction>
+        </transmission>
+        <transmission type="pr2_mechanism_model/SimpleTransmission" name="upperarm_roll_trans">
+            <actuator name="upperarm_roll_motor" />
+            <joint name="upperarm_roll_joint" />
+            <mechanicalReduction>1.0</mechanicalReduction>
+        </transmission>
+        <transmission type="pr2_mechanism_model/SimpleTransmission" name="elbow_flex_trans">
+            <actuator name="elbow_flex_motor" />
+            <joint name="elbow_flex_joint" />
+            <mechanicalReduction>1.0</mechanicalReduction>
+        </transmission>
+        <transmission type="pr2_mechanism_model/SimpleTransmission" name="forearm_roll_trans">
+            <actuator name="forearm_roll_motor" />
+            <joint name="forearm_roll_joint" />
+            <mechanicalReduction>1.0</mechanicalReduction>
+        </transmission>
+        <transmission type="pr2_mechanism_model/SimpleTransmission" name="wrist_pitch_trans">
+            <actuator name="wrist_pitch_motor" />
+            <joint name="wrist_pitch_joint" />
             <mechanicalReduction>1.0</mechanicalReduction>
         </transmission>
@@ -382,14 +392,4 @@
             <mechanicalReduction>1.0</mechanicalReduction>
         </transmission>
-        <transmission type="pr2_mechanism_model/SimpleTransmission" name="wrist_pitch_trans">
-            <actuator name="wrist_pitch_motor" />
-            <joint name="wrist_pitch_joint" />
-            <mechanicalReduction>1.0</mechanicalReduction>
-        </transmission>
-        <transmission type="pr2_mechanism_model/SimpleTransmission" name="wrist_yaw_trans">
-            <actuator name="wrist_yaw_motor" />
-            <joint name="wrist_yaw_joint" />
-            <mechanicalReduction>1.0</mechanicalReduction>
-        </transmission>
         <transmission type="pr2_mechanism_model/SimpleTransmission" name="left_finger_trans">
             <actuator name="left_finger_motor" />
@@ -411,17 +411,17 @@
             <turnGravityOff>true</turnGravityOff>
         </gazebo>
-        <gazebo reference="L2_shoulder_yaw_link">
-            <material>SmartArm/GunMetalBrushedAluminum</material>
-            <turnGravityOff>true</turnGravityOff>
-        </gazebo>
-        <gazebo reference="L3_shoulder_roll_link">
-            <material>SmartArm/GunMetalBrushedAluminum</material>
-            <turnGravityOff>true</turnGravityOff>
-        </gazebo>
-        <gazebo reference="L4_elbow_pitch_link">
-            <material>SmartArm/GunMetalBrushedAluminum</material>
-            <turnGravityOff>true</turnGravityOff>
-        </gazebo>
-        <gazebo reference="L5_wrist_roll_link">
+        <gazebo reference="L2_shoulder_pan_link">
+            <material>SmartArm/GunMetalBrushedAluminum</material>
+            <turnGravityOff>true</turnGravityOff>
+        </gazebo>
+        <gazebo reference="L3_upperarm_roll_link">
+            <material>SmartArm/GunMetalBrushedAluminum</material>
+            <turnGravityOff>true</turnGravityOff>
+        </gazebo>
+        <gazebo reference="L4_elbow_flex_link">
+            <material>SmartArm/GunMetalBrushedAluminum</material>
+            <turnGravityOff>true</turnGravityOff>
+        </gazebo>
+        <gazebo reference="L5_forearm_roll_link">
             <material>SmartArm/GunMetalBrushedAluminum</material>
             <turnGravityOff>true</turnGravityOff>
@@ -431,5 +431,5 @@
             <turnGravityOff>true</turnGravityOff>
         </gazebo>
-        <gazebo reference="L7_wrist_yaw_link">
+        <gazebo reference="L7_wrist_roll_link">
             <material>SmartArm/GunMetalBrushedAluminum</material>
             <turnGravityOff>true</turnGravityOff>
@@ -448,15 +448,25 @@
             <fudgeFactor value="0.5" />
         </gazebo>
-        <gazebo reference="shoulder_yaw_joint">
-            <stopKd value="1.0" />
-            <stopKp value="1000000.0" />
-            <fudgeFactor value="0.5" />
-        </gazebo>
-        <gazebo reference="shoulder_roll_joint">
-            <stopKd value="1.0" />
-            <stopKp value="1000000.0" />
-            <fudgeFactor value="0.5" />
-        </gazebo>
-        <gazebo reference="elbow_pitch_joint">
+        <gazebo reference="shoulder_pan_joint">
+            <stopKd value="1.0" />
+            <stopKp value="1000000.0" />
+            <fudgeFactor value="0.5" />
+        </gazebo>
+        <gazebo reference="upperarm_roll_joint">
+            <stopKd value="1.0" />
+            <stopKp value="1000000.0" />
+            <fudgeFactor value="0.5" />
+        </gazebo>
+        <gazebo reference="elbow_flex_joint">
+            <stopKd value="1.0" />
+            <stopKp value="1000000.0" />
+            <fudgeFactor value="0.5" />
+        </gazebo>
+        <gazebo reference="forearm_roll_joint">
+            <stopKd value="1.0" />
+            <stopKp value="1000000.0" />
+            <fudgeFactor value="0.5" />
+        </gazebo>
+        <gazebo reference="wrist_pitch_joint">
             <stopKd value="1.0" />
             <stopKp value="1000000.0" />
@@ -464,14 +474,4 @@
         </gazebo>
         <gazebo reference="wrist_roll_joint">
-            <stopKd value="1.0" />
-            <stopKp value="1000000.0" />
-            <fudgeFactor value="0.5" />
-        </gazebo>
-        <gazebo reference="wrist_pitch_joint">
-            <stopKd value="1.0" />
-            <stopKp value="1000000.0" />
-            <fudgeFactor value="0.5" />
-        </gazebo>
-        <gazebo reference="wrist_yaw_joint">
             <stopKd value="1.0" />
             <stopKp value="1000000.0" />

Commit message: Fix collision offest

File: arrg/ua_robots/wubble_arm_description/urdf/wubble_arm.xacro (robot description, xacro)
@@ -306,5 +306,5 @@
             </visual>
             <collision>
-                <origin xyz="-0.0541 0 0" rpy="0 0 0" />
+                <origin xyz="0.0541 0 0" rpy="0 0 0" />
                 <geometry>
                     <mesh filename="package://wubble_arm_description/meshes/L7_wrist_roll_link.stl"/>

Commit message: modify joint offsets slightly, update IK

File: arrg/ua_robots/wubble_arm_description/urdf/wubble_arm.xacro (robot description, xacro)
@@ -67,5 +67,5 @@
         <!-- Uppperarm roll joint -->
         <joint name="upperarm_roll_joint" type="revolute" >
-            <origin xyz="0 0.1074 0" rpy="0 0 0" />
+            <origin xyz="0 0.108 0" rpy="0 0 0" />
             <parent link="L2_shoulder_pan_link" />
             <child link="L3_upperarm_roll_link"/>
@@ -77,5 +77,5 @@
         <!-- Elbow flex joint -->
         <joint name="elbow_flex_joint" type="revolute" >
-            <origin xyz="0.029 0.132 0" rpy="0 0 0" />
+            <origin xyz="0.029 0.133 0" rpy="0 0 0" />
             <parent link="L3_upperarm_roll_link" />
             <child link="L4_elbow_flex_link"/>
@@ -87,5 +87,5 @@
         <!-- Forearm roll joint -->
         <joint name="forearm_roll_joint" type="revolute" >
-            <origin xyz="0.034 0.029 0" rpy="0 0 0" />
+            <origin xyz="0.036 0.029 0" rpy="0 0 0" />
             <parent link="L4_elbow_flex_link" />
             <child link="L5_forearm_roll_link"/>
@@ -97,5 +97,5 @@
         <!-- Wrist pitch joint -->
         <joint name="wrist_pitch_joint" type="revolute" >
-            <origin xyz="0.119 0 0" rpy="0 0 0" />
+            <origin xyz="0.120 0 0" rpy="0 0 0" />
             <parent link="L5_forearm_roll_link" />
             <child link="L6_wrist_pitch_link"/>
@@ -107,5 +107,5 @@
         <!-- Wrist roll joint -->
         <joint name="wrist_roll_joint" type="revolute" >
-            <origin xyz="0.0925 0 0" rpy="0 0 0" />
+            <origin xyz="0.093 0 0" rpy="0 0 0" />
             <parent link="L6_wrist_pitch_link" />
             <child link="L7_wrist_roll_link"/>
