Commit message: Add dummy fingertip links for gripper opening calculation

File: arrg/ua_robots/wubble_arm_description/urdf/wubble_arm.xacro (robot description, xacro)
@@ -135,4 +135,16 @@
             <dynamics damping="50" friction="1"/>
         </joint>
+        <!-- Left fingertip dummy joint -->
+        <joint name="left_fingertip_joint" type="fixed" >
+            <origin xyz="0.095 0.005 0" rpy="0 0 0" />
+            <parent link="L8_left_finger_link" />
+            <child link="left_fingertip_link"/>
+        </joint>
+        <!-- Right fingertip dummy joint -->
+        <joint name="right_fingertip_joint" type="fixed" >
+            <origin xyz="0.095 -0.005 0" rpy="0 0 0" />
+            <parent link="L9_right_finger_link" />
+            <child link="right_fingertip_link"/>
+        </joint>
         <!-- ****** LINK DEFINITIONS ****** -->
         <link name="L0_base_link">
@@ -353,4 +365,46 @@
                 <geometry>
                     <mesh filename="package://wubble_arm_description/meshes/L9_gripper_right_finger.stl"/>
+                </geometry>
+            </collision>
+        </link>
+        <link name="left_fingertip_link">
+            <inertial>
+                <mass value="0.001" />
+                <origin xyz="0 0 0" rpy="0 0 0" />
+                <inertia ixx="0.001" ixy="0.0" ixz="0.0"
+                         iyy="0.001" iyz="0.0"
+                         izz="0.001" />
+            </inertial>
+            <visual>
+                <origin xyz="0 0 0" rpy="0 0 0" />
+                <geometry>
+                    <box size="0.001 0.001 0.001" />
+                </geometry>
+            </visual>
+            <collision>
+                <origin xyz="0 0 0" rpy="0 0 0" />
+                <geometry>
+                    <box size="0.001 0.001 0.001" />
+                </geometry>
+            </collision>
+        </link>
+        <link name="right_fingertip_link">
+            <inertial>
+                <mass value="0.001" />
+                <origin xyz="0 0 0" rpy="0 0 0" />
+                <inertia ixx="0.001" ixy="0.0" ixz="0.0"
+                         iyy="0.001" iyz="0.0"
+                         izz="0.001" />
+            </inertial>
+            <visual>
+                <origin xyz="0 0 0" rpy="0 0 0" />
+                <geometry>
+                    <box size="0.001 0.001 0.001" />
+                </geometry>
+            </visual>
+            <collision>
+                <origin xyz="0 0 0" rpy="0 0 0" />
+                <geometry>
+                    <box size="0.001 0.001 0.001" />
                 </geometry>
             </collision>

Commit message: update gripper paddings and fingertip locations

File: arrg/ua_robots/wubble_arm_description/urdf/wubble_arm.xacro (robot description, xacro)
@@ -121,6 +121,6 @@
             <child link="L8_left_finger_link"/>
             <axis xyz="0 0 1"/>
-            <limit  lower="-0.28" upper="0.785" effort="300" velocity="1.17" />
-            <safety_controller k_position="100" k_velocity="15.0" soft_lower_limit="${-0.28}" soft_upper_limit="${0.785}" />
+            <limit  lower="-0.317" upper="0.859" effort="300" velocity="1.17" />
+            <safety_controller k_position="100" k_velocity="15.0" soft_lower_limit="${-0.317}" soft_upper_limit="${0.859}" />
             <dynamics damping="50" friction="1"/>
         </joint>
@@ -131,11 +131,11 @@
             <child link="L9_right_finger_link"/>
             <axis xyz="0 0 1"/>
-            <limit  lower="-0.785" upper="0.28" effort="300" velocity="1.17" />
-            <safety_controller k_position="100" k_velocity="15.0" soft_lower_limit="${-0.785}" soft_upper_limit="${0.28}" />
+            <limit  lower="-0.859" upper="0.317" effort="300" velocity="1.17" />
+            <safety_controller k_position="100" k_velocity="15.0" soft_lower_limit="${-0.859}" soft_upper_limit="${0.317}" />
             <dynamics damping="50" friction="1"/>
         </joint>
         <!-- Left fingertip dummy joint -->
         <joint name="left_fingertip_joint" type="fixed" >
-            <origin xyz="0.095 0.005 0" rpy="0 0 0" />
+            <origin xyz="0.095 -0.002 0" rpy="0 0 0" />
             <parent link="L8_left_finger_link" />
             <child link="left_fingertip_link"/>
@@ -143,5 +143,5 @@
         <!-- Right fingertip dummy joint -->
         <joint name="right_fingertip_joint" type="fixed" >
-            <origin xyz="0.095 -0.005 0" rpy="0 0 0" />
+            <origin xyz="0.095 0.002 0" rpy="0 0 0" />
             <parent link="L9_right_finger_link" />
             <child link="right_fingertip_link"/>

Commit message: new arm model and supporting changes

File: arrg/ua_robots/wubble_arm_description/urdf/wubble_arm.xacro (robot description, xacro)
@@ -57,5 +57,5 @@
         <!-- Shoulder pan joint -->
         <joint name="shoulder_pan_joint" type="revolute" >
-            <origin xyz="0.069 0.029 -0.029" rpy="0 0 0" />
+            <origin xyz="0.0692 0.029 -0.029" rpy="0 0 0" />
             <parent link="L1_shoulder_pitch_link" />
             <child link="L2_shoulder_pan_link"/>
@@ -67,5 +67,5 @@
         <!-- Uppperarm roll joint -->
         <joint name="upperarm_roll_joint" type="revolute" >
-            <origin xyz="0 0.108 0" rpy="0 0 0" />
+            <origin xyz="0 0.1074 0" rpy="0 0 0" />
             <parent link="L2_shoulder_pan_link" />
             <child link="L3_upperarm_roll_link"/>
@@ -77,5 +77,5 @@
         <!-- Elbow flex joint -->
         <joint name="elbow_flex_joint" type="revolute" >
-            <origin xyz="0.029 0.133 0" rpy="0 0 0" />
+            <origin xyz="0.029 0.124 0" rpy="0 0 0" />
             <parent link="L3_upperarm_roll_link" />
             <child link="L4_elbow_flex_link"/>
@@ -87,5 +87,5 @@
         <!-- Forearm roll joint -->
         <joint name="forearm_roll_joint" type="revolute" >
-            <origin xyz="0.036 0.029 0" rpy="0 0 0" />
+            <origin xyz="0.0346 0.029 0" rpy="0 0 0" />
             <parent link="L4_elbow_flex_link" />
             <child link="L5_forearm_roll_link"/>
@@ -97,5 +97,5 @@
         <!-- Wrist pitch joint -->
         <joint name="wrist_pitch_joint" type="revolute" >
-            <origin xyz="0.120 0 0" rpy="0 0 0" />
+            <origin xyz="0.1215 0 0" rpy="0 0 0" />
             <parent link="L5_forearm_roll_link" />
             <child link="L6_wrist_pitch_link"/>
@@ -107,5 +107,5 @@
         <!-- Wrist roll joint -->
         <joint name="wrist_roll_joint" type="revolute" >
-            <origin xyz="0.093 0 0" rpy="0 0 0" />
+            <origin xyz="0.0925 0 0" rpy="0 0 0" />
             <parent link="L6_wrist_pitch_link" />
             <child link="L7_wrist_roll_link"/>
@@ -318,5 +318,5 @@
             </visual>
             <collision>
-                <origin xyz="0.0541 0 0" rpy="0 0 0" />
+                <origin xyz="-0.0541 0 0" rpy="0 0 0" />
                 <geometry>
                     <mesh filename="package://wubble_arm_description/meshes/L7_wrist_roll_link.stl"/>

Commit message: fix a bug in collision offset

File: arrg/ua_robots/wubble_arm_description/urdf/wubble_arm.xacro (robot description, xacro)
@@ -318,5 +318,5 @@
             </visual>
             <collision>
-                <origin xyz="-0.0541 0 0" rpy="0 0 0" />
+                <origin xyz="0.0541 0 0" rpy="0 0 0" />
                 <geometry>
                     <mesh filename="package://wubble_arm_description/meshes/L7_wrist_roll_link.stl"/>

Commit message: update joint limits, extract all limits into a separate file for easy regeneration

File: arrg/ua_robots/wubble_arm_description/urdf/wubble_arm.xacro (robot description, xacro)
@@ -37,4 +37,5 @@
     xmlns:controller="http://playerstage.sourceforge.net/gazebo/xmlschema/#controller"
     xmlns:interface="http://playerstage.sourceforge.net/gazebo/xmlschema/#interface">
+    <include filename="$(find wubble_arm_description)/urdf/joint_limits.urdf" />
     <macro name="wubble_arm" params="parent *origin">
         <!-- ****** JOINT DEFINITIONS ****** -->
@@ -51,6 +52,6 @@
             <child link="L1_shoulder_pitch_link"/>
             <axis xyz="0 1 0"/>
-            <limit  lower="-2.523" upper="1.048" effort="300" velocity="1.17" />
-            <safety_controller k_position="100" k_velocity="15.0" soft_lower_limit="${-2.523}" soft_upper_limit="${1.048}" />
+            <limit  lower="${shoulder_pitch_lower}" upper="${shoulder_pitch_upper}" effort="300" velocity="1.50" />
+            <safety_controller k_position="100" k_velocity="15.0" soft_lower_limit="${shoulder_pitch_lower}" soft_upper_limit="${shoulder_pitch_upper}" />
             <dynamics damping="50" friction="1"/>
         </joint>
@@ -61,6 +62,6 @@
             <child link="L2_shoulder_pan_link"/>
             <axis xyz="0 0 1"/>
-            <limit  lower="-3.351" upper="0.905" effort="300" velocity="1.17" />
-            <safety_controller k_position="100" k_velocity="15.0" soft_lower_limit="${-3.351}" soft_upper_limit="${0.905}" />
+            <limit  lower="${shoulder_pan_lower}" upper="${shoulder_pan_upper}" effort="300" velocity="1.50" />
+            <safety_controller k_position="100" k_velocity="15.0" soft_lower_limit="${shoulder_pan_lower}" soft_upper_limit="${shoulder_pan_upper}" />
             <dynamics damping="50" friction="1"/>
         </joint>
@@ -71,6 +72,6 @@
             <child link="L3_upperarm_roll_link"/>
             <axis xyz="0 1 0"/>
-            <limit  lower="-0.629" upper="3.75" effort="300" velocity="1.17" />
-            <safety_controller k_position="100" k_velocity="15.0" soft_lower_limit="${-0.629}" soft_upper_limit="${3.75}" />
+            <limit  lower="${upperarm_roll_lower}" upper="${upperarm_roll_upper}" effort="300" velocity="1.50" />
+            <safety_controller k_position="100" k_velocity="15.0" soft_lower_limit="${upperarm_roll_lower}" soft_upper_limit="${upperarm_roll_upper}" />
             <dynamics damping="50" friction="1"/>
         </joint>
@@ -81,6 +82,6 @@
             <child link="L4_elbow_flex_link"/>
             <axis xyz="0 0 1"/>
-            <limit  lower="-1.652" upper="1.846" effort="300" velocity="1.17" />
-            <safety_controller k_position="100" k_velocity="15.0" soft_lower_limit="${-1.652}" soft_upper_limit="${1.846}" />
+            <limit  lower="${elbow_flex_lower}" upper="${elbow_flex_upper}" effort="300" velocity="1.50" />
+            <safety_controller k_position="100" k_velocity="15.0" soft_lower_limit="${elbow_flex_lower}" soft_upper_limit="${elbow_flex_upper}" />
             <dynamics damping="50" friction="1"/>
         </joint>
@@ -91,6 +92,6 @@
             <child link="L5_forearm_roll_link"/>
             <axis xyz="1 0 0"/>
-            <limit  lower="-2.521" upper="2.71" effort="300" velocity="1.17" />
-            <safety_controller k_position="100" k_velocity="15.0" soft_lower_limit="${-2.521}" soft_upper_limit="${2.71}" />
+            <limit  lower="${forearm_roll_lower}" upper="${forearm_roll_upper}" effort="300" velocity="2.00" />
+            <safety_controller k_position="100" k_velocity="15.0" soft_lower_limit="${forearm_roll_lower}" soft_upper_limit="${forearm_roll_upper}" />
             <dynamics damping="50" friction="1"/>
         </joint>
@@ -101,6 +102,6 @@
             <child link="L6_wrist_pitch_link"/>
             <axis xyz="0 1 0"/>
-            <limit  lower="-2.158" upper="2.613" effort="300" velocity="1.17" />
-            <safety_controller k_position="100" k_velocity="15.0" soft_lower_limit="${-2.158}" soft_upper_limit="${2.613}" />
+            <limit  lower="${wrist_pitch_lower}" upper="${wrist_pitch_upper}" effort="300" velocity="1.50" />
+            <safety_controller k_position="100" k_velocity="15.0" soft_lower_limit="${wrist_pitch_lower}" soft_upper_limit="${wrist_pitch_upper}" />
             <dynamics damping="50" friction="1"/>
         </joint>
@@ -111,6 +112,6 @@
             <child link="L7_wrist_roll_link"/>
             <axis xyz="1 0 0"/>
-            <limit  lower="-2.597" upper="2.633" effort="300" velocity="1.17" />
-            <safety_controller k_position="100" k_velocity="15.0" soft_lower_limit="${-2.597}" soft_upper_limit="${2.633}" />
+            <limit  lower="${wrist_roll_lower}" upper="${wrist_roll_upper}" effort="300" velocity="2.00" />
+            <safety_controller k_position="100" k_velocity="15.0" soft_lower_limit="${wrist_roll_lower}" soft_upper_limit="${wrist_roll_upper}" />
             <dynamics damping="50" friction="1"/>
         </joint>
@@ -159,5 +160,5 @@
                 <origin xyz="0 0 0" rpy="0 0 0" />
                 <geometry>
-                    <mesh filename="package://wubble_arm_description/meshes/L0_base_link.stl"/>
+                    <mesh filename="package://wubble_arm_description/meshes/collada/L0_base_link.dae"/>
                 </geometry>
                 <material name="Green" />
@@ -181,5 +182,5 @@
                 <origin xyz="0 0 0" rpy="0 0 0" />
                 <geometry>
-                    <mesh filename="package://wubble_arm_description/meshes/L1_shoulder_pitch_link.stl"/>
+                    <mesh filename="package://wubble_arm_description/meshes/collada/L1_shoulder_pitch_link.dae"/>
                 </geometry>
                 <material name="Grey" />
@@ -203,5 +204,5 @@
                 <origin xyz="0 0.055 0" rpy="0 0 0" />
                 <geometry>
-                    <mesh filename="package://wubble_arm_description/meshes/L2_shoulder_pan_link.stl"/>
+                    <mesh filename="package://wubble_arm_description/meshes/collada/L2_shoulder_pan_link.dae"/>
                 </geometry>
                 <material name="Blue" />
@@ -225,5 +226,5 @@
                 <origin xyz="0 0 0" rpy="0 0 0" />
                 <geometry>
-                    <mesh filename="package://wubble_arm_description/meshes/L3_upperarm_roll_link.stl"/>
+                    <mesh filename="package://wubble_arm_description/meshes/collada/L3_upperarm_roll_link.dae"/>
                 </geometry>
                 <material name="Green" />
@@ -247,5 +248,5 @@
                 <origin xyz="0.035 0.044 0.026" rpy="0 0 0" />
                 <geometry>
-                    <mesh filename="package://wubble_arm_description/meshes/L4_elbow_flex_link.stl"/>
+                    <mesh filename="package://wubble_arm_description/meshes/collada/L4_elbow_flex_link.dae"/>
                 </geometry>
                 <material name="Grey" />
@@ -269,5 +270,5 @@
                 <origin xyz="0.025 0 0" rpy="0 0 0" />
                 <geometry>
-                    <mesh filename="package://wubble_arm_description/meshes/L5_forearm_roll_link.stl"/>
+                    <mesh filename="package://wubble_arm_description/meshes/collada/L5_forearm_roll_link.dae"/>
                 </geometry>
                 <material name="Blue" />
@@ -291,5 +292,5 @@
                 <origin xyz="0 0 0" rpy="0 0 0" />
                 <geometry>
-                    <mesh filename="package://wubble_arm_description/meshes/L6_wrist_pitch_link.stl"/>
+                    <mesh filename="package://wubble_arm_description/meshes/collada/L6_wrist_pitch_link.dae"/>
                 </geometry>
                 <material name="Green" />
@@ -313,5 +314,5 @@
                 <origin xyz="0.0541 0 0" rpy="0 0 0" />
                 <geometry>
-                    <mesh filename="package://wubble_arm_description/meshes/L7_wrist_roll_link.stl"/>
+                    <mesh filename="package://wubble_arm_description/meshes/collada/L7_wrist_roll_link.dae"/>
                 </geometry>
                 <material name="Grey" />
@@ -335,5 +336,5 @@
                 <origin xyz="0 0 0" rpy="0 0 0" />
                 <geometry>
-                    <mesh filename="package://wubble_arm_description/meshes/L8_gripper_left_finger.stl"/>
+                    <mesh filename="package://wubble_arm_description/meshes/collada/L8_gripper_left_finger.dae"/>
                 </geometry>
                 <material name="Blue" />
@@ -357,5 +358,5 @@
                 <origin xyz="0 0 0" rpy="0 0 0" />
                 <geometry>
-                    <mesh filename="package://wubble_arm_description/meshes/L9_gripper_right_finger.stl"/>
+                    <mesh filename="package://wubble_arm_description/meshes/collada/L9_gripper_right_finger.dae"/>
                 </geometry>
                 <material name="Green" />
